Commit message: [add] transmission xacro
transmissionの一番単純なマクロを作成した。
尚、このマクロでは、位置制御を行うことを前提としたTransmissionが組まれて
いる。

File: urdf/sia5/body/body.transmission.xacro (robot description, xacro)
@@ -1,12 +1,16 @@
 <?xml version="1.0"?>
 <robot name="sia5" xmlns:xacro="http://ros.org/wiki/xacro">
-  <transmission name="simple_trans">
-	<type>transmission_interface/SimpleTransmission</type>
-	<joint name="foo_joint">
-      <hardwareInterface>EffortJointInterface</hardwareInterface>
-	</joint>
-	<actuator name="foo_motor">
-      <mechanicalReduction>50</mechanicalReduction>
-	</actuator>
-  </transmission>
+  <xacro:macro name="simple_joint_position_trans_v0" params="name
+															 joint_name actuator_name
+															 reduction">
+	<transmission name="${name}">
+	  <type>transmission_interface/SimpleTransmission</type>
+	  <joint name="${joint_name}">
+		<hardwareInterface>JointPositionInterface</hardwareInterface>
+	  </joint>
+	  <actuator name="${actuator_name}">
+		<mechanicalReduction>${reduction}</mechanicalReduction>
+	  </actuator>
+	</transmission>
+  </xacro:macro>
 </robot>

Commit message: [modify] マクロの名前が長かったので変更

File: urdf/sia5/body/body.transmission.xacro (robot description, xacro)
@@ -1,5 +1,5 @@
 <?xml version="1.0"?>
 <robot name="sia5" xmlns:xacro="http://ros.org/wiki/xacro">
-  <xacro:macro name="simple_joint_position_trans_v0" params="name
+  <xacro:macro name="simple_jp_trans_v0" params="name
 															 joint_name actuator_name
 															 reduction">
