Commit message: [modify] gazebo上でlinkの色を追加できるmacroを定義

File: urdf/sia5/body/body.gazebo.xacro (robot description, xacro)
@@ -7,3 +7,8 @@
     </plugin>
   </gazebo>
+  <xacro:macro name="gazebo_link_v0" params="name color">
+	<gazebo reference="${name}">
+      <material>Gazebo/${color}</material>
+	</gazebo>
+  </xacro:macro>
 </robot>

Commit message: [modify] stlファイル名変更に伴う変更とxacroの無駄を削減

File: urdf/sia5/body/body.gazebo.xacro (robot description, xacro)
@@ -4,5 +4,5 @@
     <plugin name="gazebo_ros_control" filename="libgazebo_ros_control.so">
       <robotNamespace>/sia5</robotNamespace>
-      <robotSimType>gazebo_ros_control/DefaultRobotHWSim</robotSimType>
+      <!-- <robotSimType>gazebo_ros_control/DefaultRobotHWSim</robotSimType> -->
     </plugin>
   </gazebo>

File: urdf/sia5/body/body.transmission.xacro (robot description, xacro)
@@ -7,5 +7,5 @@
 	  <type>transmission_interface/SimpleTransmission</type>
 	  <joint name="${joint_name}">
-		<hardwareInterface>JointPositionInterface</hardwareInterface>
+		<hardwareInterface>EffortJointInterface</hardwareInterface>
 	  </joint>
 	  <actuator name="${actuator_name}">

File: urdf/sia5/body/body.urdf.xacro (robot description, xacro)
@@ -1,12 +1,12 @@
 <?xml version="1.0"?>
 <robot name="sia5" xmlns:xacro="http://ros.org/wiki/xacro">
-  <xacro:macro name="base_link_v0" params="color mass
-                                           ixx ixy ixz
-                                           iyy iyz izz">
-    <link name="base_link">
+  <xacro:macro name="link_v1" params="name color mass
+                                      ixx ixy ixz
+                                      iyy iyz izz">
+    <link name="${name}">
       <visual>
         <origin rpy="0 0 0" xyz="0 0 0"/>
         <geometry>
-          <mesh filename="package://motoman_description/meshes/sia5/visual/stl/base.stl"/>
+          <mesh filename="package://motoman_description/meshes/sia5/visual/stl/${name}.stl"/>
         </geometry>
         <material name="${color}"/>
@@ -15,29 +15,5 @@
         <origin rpy="0 0 0" xyz="0 0 0"/>
         <geometry>
-          <mesh filename="package://motoman_description/meshes/sia5/collision/stl/base.stl"/>
-        </geometry>
-      </collision>
-      <inertial>
-        <mass value="${mass}"/>
-        <origin xyz="0 0 0"/>
-        <inertia  ixx="${ixx}" ixy="${ixy}" ixz="${ixz}" iyy="${iyy}" iyz="${iyz}" izz="${izz}"/>
-      </inertial>
-    </link>
-  </xacro:macro>
-  <xacro:macro name="link_v0" params="name color mass
-                                      ixx ixy ixz
-                                      iyy iyz izz">
-    <link name="link_${name}">
-      <visual>
-        <origin rpy="0 0 0" xyz="0 0 0"/>
-        <geometry>
-          <mesh filename="package://motoman_description/meshes/sia5/visual/stl/link_${name}.stl"/>
-        </geometry>
-        <material name="${color}"/>
-      </visual>
-      <collision>
-        <origin rpy="0 0 0" xyz="0 0 0"/>
-        <geometry>
-          <mesh filename="package://motoman_description/meshes/sia5/collision/stl/link_${name}.stl"/>
+          <mesh filename="package://motoman_description/meshes/sia5/collision/stl/${name}.stl"/>
         </geometry>
       </collision>
@@ -49,24 +25,13 @@
     </link>
   </xacro:macro>
-  <xacro:macro name="base_joint_v0" params="ox oy oz ax ay az
-											el ll ul vl
-											skp skv sll sul">
-    <joint name="joint_s" type="revolute">
-      <origin rpy="0 0 0" xyz="${ox} ${oy} ${oz}"/>
-      <parent link="base_link"/>
-      <child link="link_s"/>
-      <axis xyz="${ax} ${ay} ${az}"/>
-      <limit effort="${el}" lower="${ll}" upper="${ul}" velocity="${vl}"/>
-      <safety_controller k_position="${skp}" k_velocity="${skv}" soft_lower_limit="${sll}" soft_upper_limit="${sul}"/>
-    </joint>
-  </xacro:macro>
-  <xacro:macro name="joint_v0" params="parent_name child_name
+  <xacro:macro name="joint_v1" params="joint_name
+									   parent_name child_name
                                        ox oy oz ax ay az
 									   el ll ul vl
 									   skp skv sll sul">
-    <joint name="joint_${child_name}" type="revolute">
+    <joint name="${joint_name}" type="revolute">
       <origin rpy="0 0 0" xyz="${ox} ${oy} ${oz}"/>
-      <parent link="link_${parent_name}"/>
-      <child link="link_${child_name}"/>
+      <parent link="${parent_name}"/>
+      <child link="${child_name}"/>
       <axis xyz="${ax} ${ay} ${az}"/>
       <limit effort="${el}" lower="${ll}" upper="${ul}" velocity="${vl}"/>
