Commit message: [fix] urdfのタグの順番が重要？みたい。
link_sが最初だけ回転するようになった。その後はコントロールを加えても動か
ない...orz

File: gazebo/sia5/sia5.gazebo.xacro (robot description, xacro)
@@ -1,35 +1,31 @@
 <?xml version="1.0"?>
 <robot name="sia5" xmlns:xacro="http://ros.org/wiki/xacro">
+  <xacro:include filename="$(find motoman_description)/urdf/sia5/body.gazebo.xacro"/>
+  <!-- gazebo -->
+  <xacro:gazebo_link_v1 name="base_link"/>
+  <xacro:gazebo_link_v1 name="link_s"/>
+  <xacro:include filename="$(find motoman_description)/urdf/sia5/body.transmission.xacro"/>
   <xacro:include filename="$(find motoman_description)/robots/sia5/sia5.urdf.xacro"/>
-  <xacro:include filename="$(find motoman_description)/urdf/sia5/body.transmission.xacro"/>
-  <xacro:include filename="$(find motoman_description)/urdf/sia5/body.gazebo.xacro"/>
-  <!-- fix base_link to world -->
-  <!-- Used for fixing robot to Gazebo 'base_link' -->
-  <link name="world"/>
-  <joint name="fixed" type="fixed">
-    <parent link="world"/>
-    <child link="base_link"/>
-  </joint>
   <!-- transmission -->
   <xacro:simple_jp_trans_v0 name="transmission_s"
   							joint_name="joint_s" actuator_name="motor_s"
   							reduction="1"/>
-  <xacro:simple_jp_trans_v0 name="transmission_l"
-  							joint_name="joint_l" actuator_name="motor_l"
-  							reduction="1"/>
-  <xacro:simple_jp_trans_v0 name="transmission_e"
-  							joint_name="joint_e" actuator_name="motor_e"
-  							reduction="1"/>
-  <xacro:simple_jp_trans_v0 name="transmission_u"
-  							joint_name="joint_u" actuator_name="motor_u"
-  							reduction="1"/>
-  <xacro:simple_jp_trans_v0 name="transmission_r"
-  							joint_name="joint_r" actuator_name="motor_r"
-  							reduction="1"/>
-  <xacro:simple_jp_trans_v0 name="transmission_b"
-  							joint_name="joint_b" actuator_name="motor_b"
-  							reduction="1"/>
-  <xacro:simple_jp_trans_v0 name="transmission_t"
-  							joint_name="joint_t" actuator_name="motor_t"
-  							reduction="1"/>
+  <!-- <xacro:simple_jp_trans_v0 name="transmission_l" -->
+  <!-- 							joint_name="joint_l" actuator_name="motor_l" -->
+  <!-- 							reduction="1"/> -->
+  <!-- <xacro:simple_jp_trans_v0 name="transmission_e" -->
+  <!-- 							joint_name="joint_e" actuator_name="motor_e" -->
+  <!-- 							reduction="1"/> -->
+  <!-- <xacro:simple_jp_trans_v0 name="transmission_u" -->
+  <!-- 							joint_name="joint_u" actuator_name="motor_u" -->
+  <!-- 							reduction="1"/> -->
+  <!-- <xacro:simple_jp_trans_v0 name="transmission_r" -->
+  <!-- 							joint_name="joint_r" actuator_name="motor_r" -->
+  <!-- 							reduction="1"/> -->
+  <!-- <xacro:simple_jp_trans_v0 name="transmission_b" -->
+  <!-- 							joint_name="joint_b" actuator_name="motor_b" -->
+  <!-- 							reduction="1"/> -->
+  <!-- <xacro:simple_jp_trans_v0 name="transmission_t" -->
+  <!-- 							joint_name="joint_t" actuator_name="motor_t" -->
+  <!-- 							reduction="1"/> -->
 </robot>

File: urdf/sia5/body.gazebo.xacro (robot description, xacro)
@@ -7,7 +7,8 @@
     </plugin>
   </gazebo>
-  <xacro:macro name="gazebo_link_color_v0" params="name color">
+  <xacro:macro name="gazebo_link_v1" params="name">
 	<gazebo reference="${name}">
-		<material>Gazebo/${color}</material>
+	  <mu1>0.2</mu1>
+	  <mu2>0.2</mu2>
 	  </gazebo>
   </xacro:macro>

Commit message: [modify] 簡略化のため、base_linkとlink_sだけにした
これで動かせるcontrollerを設計しなければならない。

File: gazebo/sia5/sia5.gazebo.xacro (robot description, xacro)
@@ -5,10 +5,10 @@
   <xacro:gazebo_link_v1 name="base_link"/>
   <xacro:gazebo_link_v1 name="link_s"/>
-  <xacro:gazebo_link_v1 name="link_l"/>
-  <xacro:gazebo_link_v1 name="link_e"/>
-  <xacro:gazebo_link_v1 name="link_u"/>
-  <xacro:gazebo_link_v1 name="link_r"/>
-  <xacro:gazebo_link_v1 name="link_b"/>
-  <xacro:gazebo_link_v1 name="link_t"/>
+  <!-- <xacro:gazebo_link_v1 name="link_l"/> -->
+  <!-- <xacro:gazebo_link_v1 name="link_e"/> -->
+  <!-- <xacro:gazebo_link_v1 name="link_u"/> -->
+  <!-- <xacro:gazebo_link_v1 name="link_r"/> -->
+  <!-- <xacro:gazebo_link_v1 name="link_b"/> -->
+  <!-- <xacro:gazebo_link_v1 name="link_t"/> -->
   <xacro:include filename="$(find motoman_description)/urdf/sia5/body.transmission.xacro"/>
   <xacro:include filename="$(find motoman_description)/robots/sia5/sia5.urdf.xacro"/>
@@ -17,21 +17,21 @@
   							joint_name="joint_s" actuator_name="motor_s"
   							reduction="1"/>
-  <xacro:simple_jp_trans_v0 name="transmission_l"
-  							joint_name="joint_l" actuator_name="motor_l"
-  							reduction="1"/>
-  <xacro:simple_jp_trans_v0 name="transmission_e"
-  							joint_name="joint_e" actuator_name="motor_e"
-  							reduction="1"/>
-  <xacro:simple_jp_trans_v0 name="transmission_u"
-  							joint_name="joint_u" actuator_name="motor_u"
-  							reduction="1"/>
-  <xacro:simple_jp_trans_v0 name="transmission_r"
-  							joint_name="joint_r" actuator_name="motor_r"
-  							reduction="1"/>
-  <xacro:simple_jp_trans_v0 name="transmission_b"
-  							joint_name="joint_b" actuator_name="motor_b"
-  							reduction="1"/>
-  <xacro:simple_jp_trans_v0 name="transmission_t"
-  							joint_name="joint_t" actuator_name="motor_t"
-  							reduction="1"/>
+  <!-- <xacro:simple_jp_trans_v0 name="transmission_l" -->
+  <!-- 							joint_name="joint_l" actuator_name="motor_l" -->
+  <!-- 							reduction="1"/> -->
+  <!-- <xacro:simple_jp_trans_v0 name="transmission_e" -->
+  <!-- 							joint_name="joint_e" actuator_name="motor_e" -->
+  <!-- 							reduction="1"/> -->
+  <!-- <xacro:simple_jp_trans_v0 name="transmission_u" -->
+  <!-- 							joint_name="joint_u" actuator_name="motor_u" -->
+  <!-- 							reduction="1"/> -->
+  <!-- <xacro:simple_jp_trans_v0 name="transmission_r" -->
+  <!-- 							joint_name="joint_r" actuator_name="motor_r" -->
+  <!-- 							reduction="1"/> -->
+  <!-- <xacro:simple_jp_trans_v0 name="transmission_b" -->
+  <!-- 							joint_name="joint_b" actuator_name="motor_b" -->
+  <!-- 							reduction="1"/> -->
+  <!-- <xacro:simple_jp_trans_v0 name="transmission_t" -->
+  <!-- 							joint_name="joint_t" actuator_name="motor_t" -->
+  <!-- 							reduction="1"/> -->
 </robot>

File: robots/sia5/sia5.urdf.xacro (robot description, xacro)
@@ -33,23 +33,23 @@
   				 ixx="1.0" ixy="0.0" ixz="0.0"
 				 iyy="1.0" iyz="0.0" izz="1.0"/>
-  <xacro:link_v1 name="link_l" mass="${l_rate/sum_rate*sum_mass}"
-  				 ixx="1.0" ixy="0.0" ixz="0.0"
-  				 iyy="1.0" iyz="0.0" izz="1.0"/>
-  <xacro:link_v1 name="link_e"  mass="${e_rate/sum_rate*sum_mass}"
-  				 ixx="1.0" ixy="0.0" ixz="0.0"
-  				 iyy="1.0" iyz="0.0" izz="1.0"/>
-  <xacro:link_v1 name="link_u" mass="${u_rate/sum_rate*sum_mass}"
-  				 ixx="1.0" ixy="0.0" ixz="0.0"
-  				 iyy="1.0" iyz="0.0" izz="1.0"/>
-  <xacro:link_v1 name="link_r" mass="${r_rate/sum_rate*sum_mass}"
-  				 ixx="1.0" ixy="0.0" ixz="0.0"
-  				 iyy="1.0" iyz="0.0" izz="1.0"/>
-  <xacro:link_v1 name="link_b" mass="${b_rate/sum_rate*sum_mass}"
-  				 ixx="1.0" ixy="0.0" ixz="0.0"
-  				 iyy="1.0" iyz="0.0" izz="1.0"/>
-  <xacro:link_v1 name="link_t" mass="${t_rate/sum_rate*sum_mass}"
-  				 ixx="1.0" ixy="0.0" ixz="0.0"
-  				 iyy="1.0" iyz="0.0" izz="1.0"/>
-  <link name="tool0"/>
+  <!-- <xacro:link_v1 name="link_l" mass="${l_rate/sum_rate*sum_mass}" -->
+  <!-- 				 ixx="1.0" ixy="0.0" ixz="0.0" -->
+  <!-- 				 iyy="1.0" iyz="0.0" izz="1.0"/> -->
+  <!-- <xacro:link_v1 name="link_e"  mass="${e_rate/sum_rate*sum_mass}" -->
+  <!-- 				 ixx="1.0" ixy="0.0" ixz="0.0" -->
+  <!-- 				 iyy="1.0" iyz="0.0" izz="1.0"/> -->
+  <!-- <xacro:link_v1 name="link_u" mass="${u_rate/sum_rate*sum_mass}" -->
+  <!-- 				 ixx="1.0" ixy="0.0" ixz="0.0" -->
+  <!-- 				 iyy="1.0" iyz="0.0" izz="1.0"/> -->
+  <!-- <xacro:link_v1 name="link_r" mass="${r_rate/sum_rate*sum_mass}" -->
+  <!-- 				 ixx="1.0" ixy="0.0" ixz="0.0" -->
+  <!-- 				 iyy="1.0" iyz="0.0" izz="1.0"/> -->
+  <!-- <xacro:link_v1 name="link_b" mass="${b_rate/sum_rate*sum_mass}" -->
+  <!-- 				 ixx="1.0" ixy="0.0" ixz="0.0" -->
+  <!-- 				 iyy="1.0" iyz="0.0" izz="1.0"/> -->
+  <!-- <xacro:link_v1 name="link_t" mass="${t_rate/sum_rate*sum_mass}" -->
+  <!-- 				 ixx="1.0" ixy="0.0" ixz="0.0" -->
+  <!-- 				 iyy="1.0" iyz="0.0" izz="1.0"/> -->
+  <!-- <link name="tool0"/> -->
   <!-- joint -->
   <joint name="world" type="fixed">
@@ -67,68 +67,68 @@
   				  skp="1" skv="1"
   				  sll="${s_axis_lower_limit}" sul="${s_axis_upper_limit}"/>
-  <xacro:joint_v1 joint_name="joint_l"
-  				  parent_name="link_s" child_name="link_l"
-  				  ox="0" oy="0.006" oz="0.136"
-  				  roll="0" pitch="0" yaw="0"
-  				  ax="0" ay="1" az="0"
-  				  el="30.0"
-  				  ll="${l_axis_lower_limit}" ul="${l_axis_upper_limit}"
-  				  vl="${l_axis_velocity_limit}"
-  				  skp="1" skv="1"
-  				  sll="${l_axis_lower_limit}" sul="${l_axis_upper_limit}"/>
-  <xacro:joint_v1 joint_name="joint_e"
-  				  parent_name="link_l" child_name="link_e"
-  				  ox="0" oy="-0.006" oz="0.15"
-  				  roll="0" pitch="0" yaw="0"
-  				  ax="0" ay="0" az="1"
-  				  el="30.0"
-  				  ll="${e_axis_lower_limit}" ul="${e_axis_upper_limit}"
-  				  vl="${e_axis_velocity_limit}"
-  				  skp="1" skv="1"
-  				  sll="${e_axis_lower_limit}" sul="${e_axis_upper_limit}"/>
-  <xacro:joint_v1 joint_name="joint_u"
-  				  parent_name="link_e" child_name="link_u"
-  				  ox="0.085" oy="-0.00826931" oz="0.12275299"
-				  roll="${M_PI/2.0}" pitch="0" yaw="0"
-  				  ax="0" ay="0" az="1"
-  				  el="30.0"
-  				  ll="${u_axis_lower_limit}" ul="${u_axis_upper_limit}"
-  				  vl="${u_axis_velocity_limit}"
-  				  skp="1" skv="1"
-  				  sll="${u_axis_lower_limit}" sul="${u_axis_upper_limit}"/>
-  <xacro:joint_v1 joint_name="joint_r"
-  				  parent_name="link_u" child_name="link_r"
-  				  ox="0.131" oy="0.06" oz="-0.008"
-				  roll="0" pitch="${M_PI/2}" yaw="0"
-  				  ax="0" ay="0" az="-1"
-  				  el="14.7"
-  				  ll="${r_axis_lower_limit}" ul="${r_axis_upper_limit}"
-  				  vl="${r_axis_velocity_limit}"
-  				  skp="1" skv="1"
-  				  sll="${r_axis_lower_limit}" sul="${r_axis_upper_limit}"/>
-  <xacro:joint_v1 joint_name="joint_b"
-  				  parent_name="link_r" child_name="link_b"
-  				  ox="-0.0045" oy="0" oz="0.139"
-				  roll="0" pitch="${-M_PI/2}" yaw="0"
-  				  ax="0" ay="0" az="1"
-  				  el="14.7"
-  				  ll="${b_axis_lower_limit}" ul="${b_axis_upper_limit}"
-  				  vl="${b_axis_velocity_limit}"
-  				  skp="1" skv="1"
-  				  sll="${b_axis_lower_limit}" sul="${b_axis_upper_limit}"/>
-  <xacro:joint_v1 joint_name="joint_t"
-  				  parent_name="link_b" child_name="link_t"
-  				  ox="0.1365" oy="0" oz="-0.0045"
-				  roll="0" pitch="0" yaw="0"
-  				  ax="-1" ay="0" az="0"
-  				  el="7.35"
-  				  ll="${t_axis_lower_limit}" ul="${t_axis_upper_limit}"
-  				  vl="${t_axis_velocity_limit}"
-  				  skp="1" skv="1"
-  				  sll="${t_axis_lower_limit}" sul="${t_axis_upper_limit}"/>
-  <joint name="joint_tool0" type="fixed">
-    <origin rpy="0 0 0" xyz="0.0115 0 0"/>
-    <parent link="link_t"/>
-    <child link="tool0"/>
-  </joint>
+  <!-- <xacro:joint_v1 joint_name="joint_l" -->
+  <!-- 				  parent_name="link_s" child_name="link_l" -->
+  <!-- 				  ox="0" oy="0.006" oz="0.136" -->
+  <!-- 				  roll="0" pitch="0" yaw="0" -->
+  <!-- 				  ax="0" ay="1" az="0" -->
+  <!-- 				  el="30.0" -->
+  <!-- 				  ll="${l_axis_lower_limit}" ul="${l_axis_upper_limit}" -->
+  <!-- 				  vl="${l_axis_velocity_limit}" -->
+  <!-- 				  skp="1" skv="1" -->
+  <!-- 				  sll="${l_axis_lower_limit}" sul="${l_axis_upper_limit}"/> -->
+  <!-- <xacro:joint_v1 joint_name="joint_e" -->
+  <!-- 				  parent_name="link_l" child_name="link_e" -->
+  <!-- 				  ox="0" oy="-0.006" oz="0.15" -->
+  <!-- 				  roll="0" pitch="0" yaw="0" -->
+  <!-- 				  ax="0" ay="0" az="1" -->
+  <!-- 				  el="30.0" -->
+  <!-- 				  ll="${e_axis_lower_limit}" ul="${e_axis_upper_limit}" -->
+  <!-- 				  vl="${e_axis_velocity_limit}" -->
+  <!-- 				  skp="1" skv="1" -->
+  <!-- 				  sll="${e_axis_lower_limit}" sul="${e_axis_upper_limit}"/> -->
+  <!-- <xacro:joint_v1 joint_name="joint_u" -->
+  <!-- 				  parent_name="link_e" child_name="link_u" -->
+  <!-- 				  ox="0.085" oy="-0.00826931" oz="0.12275299" -->
+  <!-- 				  roll="${M_PI/2.0}" pitch="0" yaw="0" -->
+  <!-- 				  ax="0" ay="0" az="1" -->
+  <!-- 				  el="30.0" -->
+  <!-- 				  ll="${u_axis_lower_limit}" ul="${u_axis_upper_limit}" -->
+  <!-- 				  vl="${u_axis_velocity_limit}" -->
+  <!-- 				  skp="1" skv="1" -->
+  <!-- 				  sll="${u_axis_lower_limit}" sul="${u_axis_upper_limit}"/> -->
+  <!-- <xacro:joint_v1 joint_name="joint_r" -->
+  <!-- 				  parent_name="link_u" child_name="link_r" -->
+  <!-- 				  ox="0.131" oy="0.06" oz="-0.008" -->
+  <!-- 				  roll="0" pitch="${M_PI/2}" yaw="0" -->
+  <!-- 				  ax="0" ay="0" az="-1" -->
+  <!-- 				  el="14.7" -->
+  <!-- 				  ll="${r_axis_lower_limit}" ul="${r_axis_upper_limit}" -->
+  <!-- 				  vl="${r_axis_velocity_limit}" -->
+  <!-- 				  skp="1" skv="1" -->
+  <!-- 				  sll="${r_axis_lower_limit}" sul="${r_axis_upper_limit}"/> -->
+  <!-- <xacro:joint_v1 joint_name="joint_b" -->
+  <!-- 				  parent_name="link_r" child_name="link_b" -->
+  <!-- 				  ox="-0.0045" oy="0" oz="0.139" -->
+  <!-- 				  roll="0" pitch="${-M_PI/2}" yaw="0" -->
+  <!-- 				  ax="0" ay="0" az="1" -->
+  <!-- 				  el="14.7" -->
+  <!-- 				  ll="${b_axis_lower_limit}" ul="${b_axis_upper_limit}" -->
+  <!-- 				  vl="${b_axis_velocity_limit}" -->
+  <!-- 				  skp="1" skv="1" -->
+  <!-- 				  sll="${b_axis_lower_limit}" sul="${b_axis_upper_limit}"/> -->
+  <!-- <xacro:joint_v1 joint_name="joint_t" -->
+  <!-- 				  parent_name="link_b" child_name="link_t" -->
+  <!-- 				  ox="0.1365" oy="0" oz="-0.0045" -->
+  <!-- 				  roll="0" pitch="0" yaw="0" -->
+  <!-- 				  ax="-1" ay="0" az="0" -->
+  <!-- 				  el="7.35" -->
+  <!-- 				  ll="${t_axis_lower_limit}" ul="${t_axis_upper_limit}" -->
+  <!-- 				  vl="${t_axis_velocity_limit}" -->
+  <!-- 				  skp="1" skv="1" -->
+  <!-- 				  sll="${t_axis_lower_limit}" sul="${t_axis_upper_limit}"/> -->
+  <!-- <joint name="joint_tool0" type="fixed"> -->
+  <!--   <origin rpy="0 0 0" xyz="0.0115 0 0"/> -->
+  <!--   <parent link="link_t"/> -->
+  <!--   <child link="tool0"/> -->
+  <!-- </joint> -->
 </robot>

Commit message: [modify] xacroの名前空間のとり方を変更
名前空間のとり方が悪いからうまく動かないのかと思ったけど、違った

File: gazebo/sia5/sia5.gazebo.xacro (robot description, xacro)
@@ -1,6 +1,12 @@
 <?xml version="1.0"?>
-<robot name="sia5" xmlns:xacro="http://ros.org/wiki/xacro">
+<robot xmlns:xacro="http://ros.org/wiki/xacro">
   <xacro:include filename="$(find motoman_description)/urdf/sia5/body.gazebo.xacro"/>
   <!-- gazebo -->
+  <gazebo>
+    <plugin name="gazebo_ros_control" filename="libgazebo_ros_control.so">
+      <robotNamespace>/sia5</robotNamespace>
+      <!-- <robotSimType>gazebo_ros_control/DefaultRobotHWSim</robotSimType> -->
+    </plugin>
+  </gazebo>
   <xacro:gazebo_link_v1 name="base_link"/>
   <xacro:gazebo_link_v1 name="link_s"/>
@@ -11,27 +17,3 @@
   <!-- <xacro:gazebo_link_v1 name="link_b"/> -->
   <!-- <xacro:gazebo_link_v1 name="link_t"/> -->
-  <xacro:include filename="$(find motoman_description)/urdf/sia5/body.transmission.xacro"/>
-  <xacro:include filename="$(find motoman_description)/robots/sia5/sia5.urdf.xacro"/>
-  <!-- transmission -->
-  <xacro:simple_jp_trans_v0 name="transmission_s"
-  							joint_name="joint_s" actuator_name="motor_s"
-  							reduction="1"/>
-  <!-- <xacro:simple_jp_trans_v0 name="transmission_l" -->
-  <!-- 							joint_name="joint_l" actuator_name="motor_l" -->
-  <!-- 							reduction="1"/> -->
-  <!-- <xacro:simple_jp_trans_v0 name="transmission_e" -->
-  <!-- 							joint_name="joint_e" actuator_name="motor_e" -->
-  <!-- 							reduction="1"/> -->
-  <!-- <xacro:simple_jp_trans_v0 name="transmission_u" -->
-  <!-- 							joint_name="joint_u" actuator_name="motor_u" -->
-  <!-- 							reduction="1"/> -->
-  <!-- <xacro:simple_jp_trans_v0 name="transmission_r" -->
-  <!-- 							joint_name="joint_r" actuator_name="motor_r" -->
-  <!-- 							reduction="1"/> -->
-  <!-- <xacro:simple_jp_trans_v0 name="transmission_b" -->
-  <!-- 							joint_name="joint_b" actuator_name="motor_b" -->
-  <!-- 							reduction="1"/> -->
-  <!-- <xacro:simple_jp_trans_v0 name="transmission_t" -->
-  <!-- 							joint_name="joint_t" actuator_name="motor_t" -->
-  <!-- 							reduction="1"/> -->
 </robot>

File: robots/sia5/sia5.urdf.xacro (robot description, xacro)
@@ -4,4 +4,6 @@
   <xacro:include filename="$(find motoman_description)/urdf/materials.xacro"/>
   <xacro:include filename="$(find motoman_description)/urdf/sia5/body.urdf.xacro" />
+  <xacro:include filename="$(find motoman_description)/urdf/sia5/body.transmission.xacro"/>
+  <xacro:include filename="$(find motoman_description)/gazebo/sia5/sia5.gazebo.xacro"/>
   <xacro:property name="s_axis_upper_limit" value="${180.0*M_PI/180.0}"/>
   <xacro:property name="s_axis_lower_limit" value="-${s_axis_upper_limit}"/>
@@ -132,3 +134,25 @@
   <!--   <child link="tool0"/> -->
   <!-- </joint> -->
+  <!-- transmission -->
+  <xacro:simple_jp_trans_v0 name="transmission_s"
+  							joint_name="joint_s" actuator_name="motor_s"
+  							reduction="1"/>
+  <!-- <xacro:simple_jp_trans_v0 name="transmission_l" -->
+  <!-- 							joint_name="joint_l" actuator_name="motor_l" -->
+  <!-- 							reduction="1"/> -->
+  <!-- <xacro:simple_jp_trans_v0 name="transmission_e" -->
+  <!-- 							joint_name="joint_e" actuator_name="motor_e" -->
+  <!-- 							reduction="1"/> -->
+  <!-- <xacro:simple_jp_trans_v0 name="transmission_u" -->
+  <!-- 							joint_name="joint_u" actuator_name="motor_u" -->
+  <!-- 							reduction="1"/> -->
+  <!-- <xacro:simple_jp_trans_v0 name="transmission_r" -->
+  <!-- 							joint_name="joint_r" actuator_name="motor_r" -->
+  <!-- 							reduction="1"/> -->
+  <!-- <xacro:simple_jp_trans_v0 name="transmission_b" -->
+  <!-- 							joint_name="joint_b" actuator_name="motor_b" -->
+  <!-- 							reduction="1"/> -->
+  <!-- <xacro:simple_jp_trans_v0 name="transmission_t" -->
+  <!-- 							joint_name="joint_t" actuator_name="motor_t" -->
+  <!-- 							reduction="1"/> -->
 </robot>

File: urdf/sia5/body.gazebo.xacro (robot description, xacro)
@@ -1,10 +1,4 @@
 <?xml version="1.0"?>
-<robot name="sia5" xmlns:xacro="http://ros.org/wiki/xacro">
-  <gazebo>
-    <plugin name="gazebo_ros_control" filename="libgazebo_ros_control.so">
-      <robotNamespace>/sia5</robotNamespace>
-      <robotSimType>gazebo_ros_control/DefaultRobotHWSim</robotSimType>
-    </plugin>
-  </gazebo>
+<robot xmlns:xacro="http://ros.org/wiki/xacro">
   <xacro:macro name="gazebo_link_v1" params="name">
 	<gazebo reference="${name}">

File: urdf/sia5/body.transmission.xacro (robot description, xacro)
@@ -1,16 +1,16 @@
 <?xml version="1.0"?>
-<robot name="sia5" xmlns:xacro="http://ros.org/wiki/xacro">
+<robot xmlns:xacro="http://ros.org/wiki/xacro">
   <xacro:macro name="simple_jp_trans_v0" params="name
-															 joint_name actuator_name
-															 reduction">
+												 joint_name actuator_name
+												 reduction">
 	<transmission name="${name}">
-	  <type>transmission_interface/SimpleTransmission</type>
-	  <joint name="${joint_name}">
+      <type>transmission_interface/SimpleTransmission</type>
+      <joint name="${joint_name}">
 		<hardwareInterface>EffortJointInterface</hardwareInterface>
-	  </joint>
-	  <actuator name="${actuator_name}">
+      </joint>
+      <actuator name="${actuator_name}">
 		<hardwareInterface>EffortJointInterface</hardwareInterface>
-		<mechanicalReduction>${reduction}</mechanicalReduction>
-	  </actuator>
+		<mechanicalReduction>1</mechanicalReduction>
+      </actuator>
 	</transmission>
   </xacro:macro>

File: urdf/sia5/body.urdf.xacro (robot description, xacro)
@@ -1,4 +1,4 @@
 <?xml version="1.0"?>
-<robot name="sia5" xmlns:xacro="http://ros.org/wiki/xacro">
+<robot xmlns:xacro="http://ros.org/wiki/xacro">
   <!-- about mass rate -->
   <property name="base_rate" value="1.2" />
@@ -45,4 +45,5 @@
       <child link="${child_name}"/>
       <axis xyz="${ax} ${ay} ${az}"/>
+	  <dynamics damping="0.7" friction="0.7"/>
       <limit effort="${el}" lower="${ll}" upper="${ul}" velocity="${vl}"/>
       <safety_controller k_position="${skp}" k_velocity="${skv}" soft_lower_limit="${sll}" soft_upper_limit="${sul}"/>
