Commit message: [modify] とりあえずGazeboで動くようにした
jointをcontiniousにした。本当はrevoluteにしたい。
各ジョイントがふわふわしているが、今度調整します。

File: gazebo/sia5/sia5.gazebo.xacro (robot description, xacro)
@@ -11,9 +11,9 @@
   <xacro:gazebo_link_v1 name="base_link"/>
   <xacro:gazebo_link_v1 name="link_s"/>
-  <!-- <xacro:gazebo_link_v1 name="link_l"/> -->
-  <!-- <xacro:gazebo_link_v1 name="link_e"/> -->
-  <!-- <xacro:gazebo_link_v1 name="link_u"/> -->
-  <!-- <xacro:gazebo_link_v1 name="link_r"/> -->
-  <!-- <xacro:gazebo_link_v1 name="link_b"/> -->
-  <!-- <xacro:gazebo_link_v1 name="link_t"/> -->
+  <xacro:gazebo_link_v1 name="link_l"/>
+  <xacro:gazebo_link_v1 name="link_e"/>
+  <xacro:gazebo_link_v1 name="link_u"/>
+  <xacro:gazebo_link_v1 name="link_r"/>
+  <xacro:gazebo_link_v1 name="link_b"/>
+  <xacro:gazebo_link_v1 name="link_t"/>
 </robot>

File: robots/sia5/sia5.urdf.xacro (robot description, xacro)
@@ -6,4 +6,5 @@
   <xacro:include filename="$(find motoman_description)/urdf/sia5/body.transmission.xacro"/>
   <xacro:include filename="$(find motoman_description)/gazebo/sia5/sia5.gazebo.xacro"/>
+  <property name="sum_mass" value="30.0" />
   <xacro:property name="s_axis_upper_limit" value="${180.0*M_PI/180.0}"/>
   <xacro:property name="s_axis_lower_limit" value="-${s_axis_upper_limit}"/>
@@ -35,23 +36,23 @@
   				 ixx="1.0" ixy="0.0" ixz="0.0"
 				 iyy="1.0" iyz="0.0" izz="1.0"/>
-  <!-- <xacro:link_v1 name="link_l" mass="${l_rate/sum_rate*sum_mass}" -->
-  <!-- 				 ixx="1.0" ixy="0.0" ixz="0.0" -->
-  <!-- 				 iyy="1.0" iyz="0.0" izz="1.0"/> -->
-  <!-- <xacro:link_v1 name="link_e"  mass="${e_rate/sum_rate*sum_mass}" -->
-  <!-- 				 ixx="1.0" ixy="0.0" ixz="0.0" -->
-  <!-- 				 iyy="1.0" iyz="0.0" izz="1.0"/> -->
-  <!-- <xacro:link_v1 name="link_u" mass="${u_rate/sum_rate*sum_mass}" -->
-  <!-- 				 ixx="1.0" ixy="0.0" ixz="0.0" -->
-  <!-- 				 iyy="1.0" iyz="0.0" izz="1.0"/> -->
-  <!-- <xacro:link_v1 name="link_r" mass="${r_rate/sum_rate*sum_mass}" -->
-  <!-- 				 ixx="1.0" ixy="0.0" ixz="0.0" -->
-  <!-- 				 iyy="1.0" iyz="0.0" izz="1.0"/> -->
-  <!-- <xacro:link_v1 name="link_b" mass="${b_rate/sum_rate*sum_mass}" -->
-  <!-- 				 ixx="1.0" ixy="0.0" ixz="0.0" -->
-  <!-- 				 iyy="1.0" iyz="0.0" izz="1.0"/> -->
-  <!-- <xacro:link_v1 name="link_t" mass="${t_rate/sum_rate*sum_mass}" -->
-  <!-- 				 ixx="1.0" ixy="0.0" ixz="0.0" -->
-  <!-- 				 iyy="1.0" iyz="0.0" izz="1.0"/> -->
-  <!-- <link name="tool0"/> -->
+  <xacro:link_v1 name="link_l" mass="${l_rate/sum_rate*sum_mass}"
+  				 ixx="1.0" ixy="0.0" ixz="0.0"
+  				 iyy="1.0" iyz="0.0" izz="1.0"/>
+  <xacro:link_v1 name="link_e"  mass="${e_rate/sum_rate*sum_mass}"
+  				 ixx="1.0" ixy="0.0" ixz="0.0"
+  				 iyy="1.0" iyz="0.0" izz="1.0"/>
+  <xacro:link_v1 name="link_u" mass="${u_rate/sum_rate*sum_mass}"
+  				 ixx="1.0" ixy="0.0" ixz="0.0"
+  				 iyy="1.0" iyz="0.0" izz="1.0"/>
+  <xacro:link_v1 name="link_r" mass="${r_rate/sum_rate*sum_mass}"
+  				 ixx="1.0" ixy="0.0" ixz="0.0"
+  				 iyy="1.0" iyz="0.0" izz="1.0"/>
+  <xacro:link_v1 name="link_b" mass="${b_rate/sum_rate*sum_mass}"
+  				 ixx="1.0" ixy="0.0" ixz="0.0"
+  				 iyy="1.0" iyz="0.0" izz="1.0"/>
+  <xacro:link_v1 name="link_t" mass="${t_rate/sum_rate*sum_mass}"
+  				 ixx="1.0" ixy="0.0" ixz="0.0"
+  				 iyy="1.0" iyz="0.0" izz="1.0"/>
+  <link name="tool0"/>
   <!-- joint -->
   <joint name="world" type="fixed">
@@ -69,90 +70,90 @@
   				  skp="1" skv="1"
   				  sll="${s_axis_lower_limit}" sul="${s_axis_upper_limit}"/>
-  <!-- <xacro:joint_v1 joint_name="joint_l" -->
-  <!-- 				  parent_name="link_s" child_name="link_l" -->
-  <!-- 				  ox="0" oy="0.006" oz="0.136" -->
-  <!-- 				  roll="0" pitch="0" yaw="0" -->
-  <!-- 				  ax="0" ay="1" az="0" -->
-  <!-- 				  el="30.0" -->
-  <!-- 				  ll="${l_axis_lower_limit}" ul="${l_axis_upper_limit}" -->
-  <!-- 				  vl="${l_axis_velocity_limit}" -->
-  <!-- 				  skp="1" skv="1" -->
-  <!-- 				  sll="${l_axis_lower_limit}" sul="${l_axis_upper_limit}"/> -->
-  <!-- <xacro:joint_v1 joint_name="joint_e" -->
-  <!-- 				  parent_name="link_l" child_name="link_e" -->
-  <!-- 				  ox="0" oy="-0.006" oz="0.15" -->
-  <!-- 				  roll="0" pitch="0" yaw="0" -->
-  <!-- 				  ax="0" ay="0" az="1" -->
-  <!-- 				  el="30.0" -->
-  <!-- 				  ll="${e_axis_lower_limit}" ul="${e_axis_upper_limit}" -->
-  <!-- 				  vl="${e_axis_velocity_limit}" -->
-  <!-- 				  skp="1" skv="1" -->
-  <!-- 				  sll="${e_axis_lower_limit}" sul="${e_axis_upper_limit}"/> -->
-  <!-- <xacro:joint_v1 joint_name="joint_u" -->
-  <!-- 				  parent_name="link_e" child_name="link_u" -->
-  <!-- 				  ox="0.085" oy="-0.00826931" oz="0.12275299" -->
-  <!-- 				  roll="${M_PI/2.0}" pitch="0" yaw="0" -->
-  <!-- 				  ax="0" ay="0" az="1" -->
-  <!-- 				  el="30.0" -->
-  <!-- 				  ll="${u_axis_lower_limit}" ul="${u_axis_upper_limit}" -->
-  <!-- 				  vl="${u_axis_velocity_limit}" -->
-  <!-- 				  skp="1" skv="1" -->
-  <!-- 				  sll="${u_axis_lower_limit}" sul="${u_axis_upper_limit}"/> -->
-  <!-- <xacro:joint_v1 joint_name="joint_r" -->
-  <!-- 				  parent_name="link_u" child_name="link_r" -->
-  <!-- 				  ox="0.131" oy="0.06" oz="-0.008" -->
-  <!-- 				  roll="0" pitch="${M_PI/2}" yaw="0" -->
-  <!-- 				  ax="0" ay="0" az="-1" -->
-  <!-- 				  el="14.7" -->
-  <!-- 				  ll="${r_axis_lower_limit}" ul="${r_axis_upper_limit}" -->
-  <!-- 				  vl="${r_axis_velocity_limit}" -->
-  <!-- 				  skp="1" skv="1" -->
-  <!-- 				  sll="${r_axis_lower_limit}" sul="${r_axis_upper_limit}"/> -->
-  <!-- <xacro:joint_v1 joint_name="joint_b" -->
-  <!-- 				  parent_name="link_r" child_name="link_b" -->
-  <!-- 				  ox="-0.0045" oy="0" oz="0.139" -->
-  <!-- 				  roll="0" pitch="${-M_PI/2}" yaw="0" -->
-  <!-- 				  ax="0" ay="0" az="1" -->
-  <!-- 				  el="14.7" -->
-  <!-- 				  ll="${b_axis_lower_limit}" ul="${b_axis_upper_limit}" -->
-  <!-- 				  vl="${b_axis_velocity_limit}" -->
-  <!-- 				  skp="1" skv="1" -->
-  <!-- 				  sll="${b_axis_lower_limit}" sul="${b_axis_upper_limit}"/> -->
-  <!-- <xacro:joint_v1 joint_name="joint_t" -->
-  <!-- 				  parent_name="link_b" child_name="link_t" -->
-  <!-- 				  ox="0.1365" oy="0" oz="-0.0045" -->
-  <!-- 				  roll="0" pitch="0" yaw="0" -->
-  <!-- 				  ax="-1" ay="0" az="0" -->
-  <!-- 				  el="7.35" -->
-  <!-- 				  ll="${t_axis_lower_limit}" ul="${t_axis_upper_limit}" -->
-  <!-- 				  vl="${t_axis_velocity_limit}" -->
-  <!-- 				  skp="1" skv="1" -->
-  <!-- 				  sll="${t_axis_lower_limit}" sul="${t_axis_upper_limit}"/> -->
-  <!-- <joint name="joint_tool0" type="fixed"> -->
-  <!--   <origin rpy="0 0 0" xyz="0.0115 0 0"/> -->
-  <!--   <parent link="link_t"/> -->
-  <!--   <child link="tool0"/> -->
-  <!-- </joint> -->
+  <xacro:joint_v1 joint_name="joint_l"
+  				  parent_name="link_s" child_name="link_l"
+  				  ox="0" oy="0.006" oz="0.136"
+  				  roll="0" pitch="0" yaw="0"
+  				  ax="0" ay="1" az="0"
+  				  el="30.0"
+  				  ll="${l_axis_lower_limit}" ul="${l_axis_upper_limit}"
+  				  vl="${l_axis_velocity_limit}"
+  				  skp="1" skv="1"
+  				  sll="${l_axis_lower_limit}" sul="${l_axis_upper_limit}"/>
+  <xacro:joint_v1 joint_name="joint_e"
+  				  parent_name="link_l" child_name="link_e"
+  				  ox="0" oy="-0.006" oz="0.15"
+  				  roll="0" pitch="0" yaw="0"
+  				  ax="0" ay="0" az="1"
+  				  el="30.0"
+  				  ll="${e_axis_lower_limit}" ul="${e_axis_upper_limit}"
+  				  vl="${e_axis_velocity_limit}"
+  				  skp="1" skv="1"
+  				  sll="${e_axis_lower_limit}" sul="${e_axis_upper_limit}"/>
+  <xacro:joint_v1 joint_name="joint_u"
+  				  parent_name="link_e" child_name="link_u"
+  				  ox="0.085" oy="-0.00826931" oz="0.12275299"
+  				  roll="${M_PI/2.0}" pitch="0" yaw="0"
+  				  ax="0" ay="0" az="1"
+  				  el="30.0"
+  				  ll="${u_axis_lower_limit}" ul="${u_axis_upper_limit}"
+  				  vl="${u_axis_velocity_limit}"
+  				  skp="1" skv="1"
+  				  sll="${u_axis_lower_limit}" sul="${u_axis_upper_limit}"/>
+  <xacro:joint_v1 joint_name="joint_r"
+  				  parent_name="link_u" child_name="link_r"
+  				  ox="0.131" oy="0.06" oz="-0.008"
+  				  roll="0" pitch="${M_PI/2}" yaw="0"
+  				  ax="0" ay="0" az="-1"
+  				  el="14.7"
+  				  ll="${r_axis_lower_limit}" ul="${r_axis_upper_limit}"
+  				  vl="${r_axis_velocity_limit}"
+  				  skp="1" skv="1"
+  				  sll="${r_axis_lower_limit}" sul="${r_axis_upper_limit}"/>
+  <xacro:joint_v1 joint_name="joint_b"
+  				  parent_name="link_r" child_name="link_b"
+  				  ox="-0.0045" oy="0" oz="0.139"
+  				  roll="0" pitch="${-M_PI/2}" yaw="0"
+  				  ax="0" ay="0" az="1"
+  				  el="14.7"
+  				  ll="${b_axis_lower_limit}" ul="${b_axis_upper_limit}"
+  				  vl="${b_axis_velocity_limit}"
+  				  skp="1" skv="1"
+  				  sll="${b_axis_lower_limit}" sul="${b_axis_upper_limit}"/>
+  <xacro:joint_v1 joint_name="joint_t"
+  				  parent_name="link_b" child_name="link_t"
+  				  ox="0.1365" oy="0" oz="-0.0045"
+  				  roll="0" pitch="0" yaw="0"
+  				  ax="-1" ay="0" az="0"
+  				  el="7.35"
+  				  ll="${t_axis_lower_limit}" ul="${t_axis_upper_limit}"
+  				  vl="${t_axis_velocity_limit}"
+  				  skp="1" skv="1"
+  				  sll="${t_axis_lower_limit}" sul="${t_axis_upper_limit}"/>
+  <joint name="joint_tool0" type="fixed">
+    <origin rpy="0 0 0" xyz="0.0115 0 0"/>
+    <parent link="link_t"/>
+    <child link="tool0"/>
+  </joint>
   <!-- transmission -->
   <xacro:simple_jp_trans_v0 name="transmission_s"
   							joint_name="joint_s" actuator_name="motor_s"
   							reduction="1"/>
-  <!-- <xacro:simple_jp_trans_v0 name="transmission_l" -->
-  <!-- 							joint_name="joint_l" actuator_name="motor_l" -->
-  <!-- 							reduction="1"/> -->
-  <!-- <xacro:simple_jp_trans_v0 name="transmission_e" -->
-  <!-- 							joint_name="joint_e" actuator_name="motor_e" -->
-  <!-- 							reduction="1"/> -->
-  <!-- <xacro:simple_jp_trans_v0 name="transmission_u" -->
-  <!-- 							joint_name="joint_u" actuator_name="motor_u" -->
-  <!-- 							reduction="1"/> -->
-  <!-- <xacro:simple_jp_trans_v0 name="transmission_r" -->
-  <!-- 							joint_name="joint_r" actuator_name="motor_r" -->
-  <!-- 							reduction="1"/> -->
-  <!-- <xacro:simple_jp_trans_v0 name="transmission_b" -->
-  <!-- 							joint_name="joint_b" actuator_name="motor_b" -->
-  <!-- 							reduction="1"/> -->
-  <!-- <xacro:simple_jp_trans_v0 name="transmission_t" -->
-  <!-- 							joint_name="joint_t" actuator_name="motor_t" -->
-  <!-- 							reduction="1"/> -->
+  <xacro:simple_jp_trans_v0 name="transmission_l"
+  							joint_name="joint_l" actuator_name="motor_l"
+  							reduction="1"/>
+  <xacro:simple_jp_trans_v0 name="transmission_e"
+  							joint_name="joint_e" actuator_name="motor_e"
+  							reduction="1"/>
+  <xacro:simple_jp_trans_v0 name="transmission_u"
+  							joint_name="joint_u" actuator_name="motor_u"
+  							reduction="1"/>
+  <xacro:simple_jp_trans_v0 name="transmission_r"
+  							joint_name="joint_r" actuator_name="motor_r"
+  							reduction="1"/>
+  <xacro:simple_jp_trans_v0 name="transmission_b"
+  							joint_name="joint_b" actuator_name="motor_b"
+  							reduction="1"/>
+  <xacro:simple_jp_trans_v0 name="transmission_t"
+  							joint_name="joint_t" actuator_name="motor_t"
+  							reduction="1"/>
 </robot>

File: urdf/sia5/body.transmission.xacro (robot description, xacro)
@@ -11,5 +11,5 @@
       <actuator name="${actuator_name}">
 		<hardwareInterface>EffortJointInterface</hardwareInterface>
-		<mechanicalReduction>1</mechanicalReduction>
+		<mechanicalReduction>${reduction}</mechanicalReduction>
       </actuator>
 	</transmission>

File: urdf/sia5/body.urdf.xacro (robot description, xacro)
@@ -2,17 +2,16 @@
 <robot xmlns:xacro="http://ros.org/wiki/xacro">
   <!-- about mass rate -->
-  <property name="base_rate" value="1.2" />
-  <property name="s_rate" value="1.0" />
+  <property name="base_rate" value="5.0" />
+  <property name="s_rate" value="1.2" />
   <property name="l_rate" value="1.0" />
-  <property name="e_rate" value="1.0" />
-  <property name="u_rate" value="0.7" />
-  <property name="r_rate" value="0.7" />
-  <property name="b_rate" value="0.6" />
-  <property name="t_rate" value="0.2" />
+  <property name="e_rate" value="0.15" />
+  <property name="u_rate" value="0.05" />
+  <property name="r_rate" value="0.02" />
+  <property name="b_rate" value="0.02" />
+  <property name="t_rate" value="0.005" />
   <property name="sum_rate" value="${base_rate + s_rate
 								   + l_rate + e_rate
 								   + u_rate + r_rate
 								   + b_rate + t_rate}" />
-  <property name="sum_mass" value="30.0" />
   <xacro:macro name="link_v1" params="name mass
                                       ixx ixy ixz
@@ -40,5 +39,5 @@
 									   el ll ul vl
 									   skp skv sll sul">
-    <joint name="${joint_name}" type="revolute">
+    <joint name="${joint_name}" type="continuous">
       <origin xyz="${ox} ${oy} ${oz}" rpy="${roll} ${pitch} ${yaw}"/>
       <parent link="${parent_name}"/>
