Commit message: [modify] safety_controlをコメントアウト
joint_s joint_r joint_t だけがおかしくなってしまった。。。
これから修正します。

File: urdf/sia5/body.urdf.xacro (robot description, xacro)
@@ -39,5 +39,5 @@
 									   el ll ul vl
 									   skp skv sll sul">
-    <joint name="${joint_name}" type="continuous">
+    <joint name="${joint_name}" type="revolute">
       <origin xyz="${ox} ${oy} ${oz}" rpy="${roll} ${pitch} ${yaw}"/>
       <parent link="${parent_name}"/>
@@ -46,5 +46,5 @@
 	  <dynamics damping="0.7" friction="0.7"/>
       <limit effort="${el}" lower="${ll}" upper="${ul}" velocity="${vl}"/>
-      <safety_controller k_position="${skp}" k_velocity="${skv}" soft_lower_limit="${sll}" soft_upper_limit="${sul}"/>
+      <!-- <safety_controller k_position="0" k_velocity="0" soft_lower_limit="0" soft_upper_limit="0"/> -->
     </joint>
   </xacro:macro>

Commit message: [modify] collision判定を簡易化するマクロを新たに定義

File: urdf/sia5/body.urdf.xacro (robot description, xacro)
@@ -69,4 +69,27 @@
     </link>
   </xacro:macro>
+  <xacro:macro name="link_box_v1" params="name mass width depth height
+										  ox oy oz oroll opitch oyaw">
+    <link name="${name}">
+      <visual>
+        <geometry>
+          <mesh filename="package://motoman_description/meshes/sia5/visual/COLLADA/${name}.dae"/>
+        </geometry>
+      </visual>
+      <collision>
+		<origin xyz="0 ${oy} -${oz}" rpy="${oroll} ${opitch} ${oyaw}"/>
+        <geometry>
+		  <box size="${depth} ${width} ${height}"/>
+        </geometry>
+      </collision>
+      <inertial>
+		<origin xyz="${ox} ${oy} ${oz}" rpy="${oroll} ${opitch} ${oyaw}"/>
+        <mass value="${mass}"/>
+        <inertia ixx="${(mass*((width/2)*(width/2)+(height/2)*(height/2)))/3}" ixy="0" ixz="0"
+				 iyy="${(mass*((depth/2)*(depth/2)+(height/2)*(height/2)))/3}" iyz="0"
+				 izz="${(mass*((depth/2)*(depth/2)+(width/2)*(width/2)))/3}" />
+      </inertial>
+    </link>
+  </xacro:macro>
   <xacro:macro name="link_cylinder_plus_box_v0" params="name
 														ox oy oz oroll opitch oyaw
