Commit message: [modify] tool0のlinkの位置を変更

File: robots/sia5/sia5_no_tool.urdf.xacro (robot description, xacro)
@@ -173,5 +173,5 @@
 				  sll="${t_axis_lower_limit}" sul="${t_axis_upper_limit}"/>
   <joint name="joint_tool0" type="fixed">
-    <origin rpy="0 0 0" xyz="0.0115 0 -0.040"/>
+    <origin rpy="0 0 0" xyz="0.0115 0 0"/>
     <parent link="link_t"/>
     <child link="tool0"/>
