Commit message: [fix] テーブルの大きさ等を変更
変更前は高さが0.53[m]であったが、これが間違いだった
0.51[m]に変更し、collisionの高さは0.50に変更した
それに伴い、他のurdfファイルも変更になった

File: robots/sia5/sia5_with_table.urdf.xacro (robot description, xacro)
@@ -46,6 +46,6 @@
   <link name="world"/>
   <xacro:link_box_v1 name="table_link" mass="${table_mass}"
-					 width="0.676" depth="1.116" height="0.53"
-					 ox="0.20" oy="0" oz="0.265" oroll="0" opitch="0" oyaw="0"/>
+					 width="0.676" depth="1.116" height="0.50"
+					 ox="0.20" oy="0" oz="0.245" oroll="0" opitch="0" oyaw="0"/>
   <xacro:link_box_v0 name="base_link" mass="${base_rate/sum_rate*sum_mass}"
 					 width="0.1665" depth="0.1976" height="0.1465"
@@ -96,5 +96,5 @@
     <parent link="world"/>
     <child link="table_link"/>
-	<origin xyz="0 0 0.53"/>
+	<origin xyz="0 0 0.51"/>
   </joint>
   <joint name="joint_base" type="fixed">

File: robots/sia5/urdf/sia5_nishida_lab.urdf (robot description, URDF)
Before this commit: robot sia5, 15 links, 14 joints
Links:
- link kinect2_link: mass 0.5 -> 0.935; geometry collision box size=0.065 0.25 0.082; visual mesh filename=package://motoman_description/meshes/sensor/visual/COLLADA/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
- link table_link: geometry collision box size=1.116 0.676 0.5; visual mesh filename=package://motoman_description/meshes/sia5/visual/COLLADA/ta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
Joints:
- joint world: origin xyz=0 0 0.53 -> xyz=0 0 0.51

File: robots/sia5/urdf/sia5_with_jamming.urdf (robot description, URDF)
Before this commit: robot sia5, 13 links, 12 joints
Links:
- link table_link: geometry collision box size=1.116 0.676 0.5; visual mesh filename=package://motoman_description/meshes/sia5/visual/COLLADA/ta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
Joints:
- joint world: origin xyz=0 0 0.53 -> xyz=0 0 0.51

File: robots/sia5/urdf/sia5_with_table.urdf (robot description, URDF)
Before this commit: robot sia5, 11 links, 10 joints
Links:
- link table_link: geometry collision box size=1.116 0.676 0.5; visual mesh filename=package://motoman_description/meshes/sia5/visual/COLLADA/ta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
Joints:
- joint world: origin xyz=0 0 0.53 -> xyz=0 0 0.51
