Commit message: [modify] 風船部分の衝突判定をなくした

File: robots/sia5/sia5_with_jamming.urdf.xacro (robot description, xacro)
@@ -10,5 +10,5 @@
   							   ox="0" oy="0" oz="0"
   							   oroll="0" opitch="0" oyaw="0"/>
-  <xacro:tool_link_v1 name="balloon" mass="0.3"
+  <xacro:tool_link_no_collision_v0 name="balloon" mass="0.3"
   					  ixx="0.001" ixy="0" ixz="0"
   					  iyy="0.001" iyz="0" izz="0.001"/>

File: robots/sia5/urdf/sia5_with_jamming.urdf (robot description, URDF)
Before this commit: robot sia5, 13 links, 12 joints
Links:
- link balloon: geometry visual mesh filename=package://motoman_description/meshes/tool/visual/COLLADA/ba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

File: urdf/tool/jamming.urdf.xacro (robot description, xacro)
@@ -22,5 +22,5 @@
     </link>
   </xacro:macro>
-  <xacro:macro name="tool_link_v1" params="name mass
+  <xacro:macro name="tool_link_no_collision_v0" params="name mass
 										   ixx ixy ixz
 										   iyy iyz izz">
@@ -32,9 +32,4 @@
         </geometry>
       </visual>
-      <collision>
-        <geometry>
-          <mesh filename="package://motoman_description/meshes/tool/collision/STL/${name}.stl"/>
-        </geometry>
-      </collision>
       <inertial>
         <mass value="${mass}"/>
@@ -44,5 +39,5 @@
   </xacro:macro>
   <xacro:macro name="tool_link_cylinder_v0" params="name mass radius height
-											   ox oy oz oroll opitch oyaw">
+													ox oy oz oroll opitch oyaw">
     <link name="${name}">
       <visual>

Commit message: [fix] グリッパをlink_tから少しだけ離した
プランニング刷るときに、collision判定が出て動かなくなるので修正

File: robots/sia5/sia5_with_jamming.urdf.xacro (robot description, xacro)
@@ -15,5 +15,5 @@
   <!-- Joint -->
   <joint name="joint_gripper" type="fixed">
-    <origin rpy="-0.1745 0 0" xyz="0 0 0"/>
+    <origin rpy="-0.1745 0 0" xyz="0.0001 0 0"/>
     <parent link="tool0"/>
     <child link="gripper_link"/>

File: robots/sia5/urdf/sia5_nishida_lab.urdf (robot description, URDF)
Before this commit: robot sia5, 15 links, 14 joints
Joints:
- joint joint_gripper: origin xyz=0 0 0 rpy=-0.1745 0 0 -> xyz=0.0001 0 0 rpy=-0.1745 0 0

File: robots/sia5/urdf/sia5_with_jamming.urdf (robot description, URDF)
Before this commit: robot sia5, 13 links, 12 joints
Joints:
- joint joint_gripper: origin xyz=0 0 0 rpy=-0.1745 0 0 -> xyz=0.0001 0 0 rpy=-0.1745 0 0
