Commit message: [modfy] kinectの親フレームをbase_linkに変更
元はworldがおやでした。

File: robots/sia5/sia5_with_kinectv2.urdf.xacro (robot description, xacro)
@@ -12,5 +12,5 @@
   <joint name="joint_kinect2" type="fixed">
     <origin rpy="0 ${10*M_PI/180} ${M_PI}" xyz="1.05024 0 0.3195"/>
-    <parent link="world"/>
+    <parent link="base_link"/>
     <child link="kinect2_link"/>
   </joint>

File: robots/sia5/urdf/sia5_with_kinectv2.urdf (robot description, URDF)
Before this commit: robot sia5, 12 links, 11 joints
Joints:
- joint joint_kinect2: parent world -> base_link
