Commit message: [add] sia5_nishida_labのurdfとxacroを追加
sia5 + テーブル + ジャミンググリッパ + kinect2

File: robots/sia5/sia5_nishida_lab.urdf.xacro (robot description, xacro)
@@ -10,5 +10,5 @@
   <!-- Joint -->
   <joint name="joint_kinect2" type="fixed">
-    <origin rpy="0 -0.1745 0" xyz="0.50024 0 0.8195"/>
+    <origin rpy="0 ${10*M_PI/180} ${M_PI}" xyz="1.05024 0 0.8195"/>
     <parent link="world"/>
     <child link="kinect2_link"/>

Commit message: [modify] 前回と同じ

File: robots/sia5/sia5_nishida_lab.urdf.xacro (robot description, xacro)
@@ -8,4 +8,5 @@
   <!-- Link -->
   <xacro:kinect2_link_box_v0 name="kinect2_link"/>
+  <link name="kinect2_rgb_optical_frame"/>
   <!-- Joint -->
   <joint name="joint_kinect2" type="fixed">
@@ -14,4 +15,9 @@
     <child link="kinect2_link"/>
   </joint>
+  <joint name="joint_rgb_kinect2" type="fixed">
+	<origin rpy="${M_PI/2} ${M_PI} ${M_PI/2}"/>
+	<parent link="kinect2_link"/>
+	<child link="kinect2_rgb_optical_frame"/>
+  </joint>
   <!-- Gazebo -->
   <xacro:kinect_gazebo name="kinect2"/>

File: robots/sia5/urdf/sia5_nishida_lab.urdf (robot description, URDF)
Before this commit: robot sia5, 14 links, 13 joints
Links:
- added link kinect2_rgb_optical_frame
Joints:
- added joint joint_rgb_kinect2: type fixed, parent kinect2_link, child kinect2_rgb_optical_frame, origin rpy=1.57079637 3.14159274 1.57079637
- joint joint_kinect2: origin xyz=0.50024 0 0.8195 rpy=0 -0.1745 0 -> xyz=1.05024 0 0.8195 rpy=0 0.17453293 3.14159274

Commit message: [modify] ロボットモデルからテーブルを削除

File: robots/sia5/sia5_nishida_lab.urdf.xacro (robot description, xacro)
@@ -11,6 +11,6 @@
   <!-- Joint -->
   <joint name="joint_kinect2" type="fixed">
-    <origin rpy="0 ${10*M_PI/180} ${M_PI}" xyz="1.05024 0 0.8195"/>
-    <parent link="world"/>
+    <origin rpy="0 ${10*M_PI/180} ${M_PI}" xyz="1.02024 0.30 0.3595"/>
+    <parent link="base_link"/>
     <child link="kinect2_link"/>
   </joint>

File: robots/sia5/sia5_with_jamming.urdf.xacro (robot description, xacro)
@@ -4,5 +4,5 @@
   <xacro:include filename="$(find motoman_description)/urdf/tool/jamming.urdf.xacro"/>
   <xacro:include filename="$(find motoman_description)/urdf/tool/jamming.gazebo.xacro"/>
-  <xacro:include filename="$(find motoman_description)/robots/sia5/sia5_with_table.urdf.xacro"/>
+  <xacro:include filename="$(find motoman_description)/robots/sia5/sia5.urdf.xacro"/>
   <!-- Link -->
   <xacro:tool_link_cylinder_v0 name="gripper_link" mass="1.0"

File: robots/sia5/urdf/sia5_nishida_lab.urdf (robot description, URDF)
Before this commit: robot sia5, 15 links, 14 joints
Links:
- removed link table_link
Joints:
- removed joint joint_base
- joint joint_kinect2: origin xyz=1.05024 0 0.8195 rpy=0 0.17453293 3.14159274 -> xyz=1.02024 0.30 0.3595 rpy=0 0.17453293 3.14159274; parent world -> base_link
- joint world: child table_link -> base_link; origin xyz=0 0 0.51 -> (none)

File: robots/sia5/urdf/sia5_with_jamming.urdf (robot description, URDF)
Before this commit: robot sia5, 13 links, 12 joints
Links:
- removed link table_link
Joints:
- removed joint joint_base
- joint world: child table_link -> base_link; origin xyz=0 0 0.51 -> (none)
