Commit message: [modify] tableをなくしたことによるxacro等の変更

File: robots/sia5/sia5_table_gazebo.urdf.xacro (robot description, xacro)
@@ -4,5 +4,5 @@
   <xacro:include filename="$(find motoman_description)/robots/sia5/sia5_basic.urdf.xacro" />
   <xacro:add_world>
-	<origin xyz="0 0 0" rpy="0 0 0"/>
+	<origin xyz="0 0 0.511" rpy="0 0 0"/>
   </xacro:add_world>
 </robot>

File: robots/sia5/sia5_with_jamming.urdf.xacro (robot description, xacro)
@@ -11,7 +11,7 @@
   							   oroll="0" opitch="0" oyaw="0"/>
   <xacro:tool_link_no_collision_v0 name="balloon" mass="0.3"
-  					  ixx="0.001" ixy="0" ixz="0"
-  					  iyy="0.001" iyz="0" izz="0.001"/>
-  <!-- Joint -->
+  								   ixx="0.001" ixy="0" ixz="0"
+  								   iyy="0.001" iyz="0" izz="0.001"/>
+  <!-- Joint  -->
   <joint name="joint_gripper" type="fixed">
     <origin rpy="-0.1745 0 0" xyz="0.0001 0 0"/>

File: robots/sia5/sia5_with_jamming_and_kinectv2.urdf.xacro (robot description, xacro)
@@ -4,5 +4,5 @@
   <xacro:include filename="$(find motoman_description)/urdf/sensor/kinect.urdf.xacro"/>
   <xacro:include filename="$(find motoman_description)/urdf/sensor/kinect.gazebo.xacro"/>
-  <xacro:include filename="$(find motoman_description)/robots/sia5/sia5_table_gazebo.urdf.xacro"/>
+  <xacro:include filename="$(find motoman_description)/robots/sia5/sia5_with_jamming.urdf.xacro"/>
   <!-- add Kinect V2 -->
   <!-- Link -->
