Commit message: [modify] tableモデルをGazeboの時だけ追加

File: robots/sia5/sia5_gazebo_nishida_lab.urdf.xacro (robot description, xacro)
@@ -6,5 +6,8 @@
   <xacro:include filename="$(find motoman_description)/urdf/tool/jamming.urdf.xacro"/>
   <xacro:include filename="$(find motoman_description)/urdf/tool/jamming.gazebo.xacro"/>
-  <xacro:include filename="$(find motoman_description)/robots/sia5/sia5_table_gazebo.urdf.xacro"/>
+  <xacro:include filename="$(find motoman_description)/robots/sia5/sia5_basic.urdf.xacro"/>
+  <xacro:add_world>
+	<origin xyz="0 0 0.511" rpy="0 0 0"/>
+  </xacro:add_world>
   <!-- add Kinect V2 -->
   <!-- Link -->

Commit message: [modify] 風船のモデルをなくしました
もともとcollision判定はなしにしていたのですが、把持計画の際に、visual要
素も加味されるようなので、なくしました。

File: robots/sia5/sia5_gazebo_nishida_lab.urdf.xacro (robot description, xacro)
@@ -33,7 +33,8 @@
   							   ox="0" oy="0" oz="0"
   							   oroll="0" opitch="0" oyaw="0"/>
-  <xacro:tool_link_no_collision_v0 name="balloon" mass="0.3"
-  								   ixx="0.001" ixy="0" ixz="0"
-  								   iyy="0.001" iyz="0" izz="0.001"/>
+  <link name="balloon"/>
+  <!-- <xacro:tool_link_no_collision_v0 name="balloon" mass="0.3" -->
+  <!-- 								   ixx="0.001" ixy="0" ixz="0" -->
+  <!-- 								   iyy="0.001" iyz="0" izz="0.001"/> -->
   <!-- Joint  -->
   <joint name="joint_gripper" type="fixed">
@@ -49,4 +50,4 @@
   <!-- Gazebo -->
   <xacro:gazebo_tool_link_v0 name="gripper_link" color="Blue"/>
-  <xacro:gazebo_tool_link_v0 name="balloon" color="Red"/>
+  <!-- <xacro:gazebo_tool_link_v0 name="balloon" color="Red"/> -->
 </robot>

File: robots/sia5/sia5_with_jamming.urdf.xacro (robot description, xacro)
@@ -10,7 +10,8 @@
   							   ox="0" oy="0" oz="0"
   							   oroll="0" opitch="0" oyaw="0"/>
-  <xacro:tool_link_no_collision_v0 name="balloon" mass="0.3"
-  								   ixx="0.001" ixy="0" ixz="0"
-  								   iyy="0.001" iyz="0" izz="0.001"/>
+  <link name="balloon"/>
+  <!-- <xacro:tool_link_no_collision_v0 name="balloon" mass="0.3" -->
+  <!-- 								   ixx="0.001" ixy="0" ixz="0" -->
+  <!-- 								   iyy="0.001" iyz="0" izz="0.001"/> -->
   <!-- Joint  -->
   <joint name="joint_gripper" type="fixed">

Commit message: [Add] ２台のkinectを設置してインテリジェント空間を作っています

File: robots/sia5/sia5_gazebo_nishida_lab.urdf.xacro (robot description, xacro)
@@ -26,5 +26,5 @@
   </joint>
   <!-- Gazebo -->
-  <xacro:kinect_gazebo name="kinect2"/>
+  <xacro:kinect_gazebo suffix=""  name="kinect2"/>
   <!-- add Jamming Gripper -->
    <!-- Link -->

File: robots/sia5/sia5_with_jamming_and_kinectv2.urdf.xacro (robot description, xacro)
@@ -21,4 +21,4 @@
   </joint>
   <!-- Gazebo -->
-  <xacro:kinect_gazebo name="kinect2"/>
+  <xacro:kinect_gazebo suffix="" name="kinect2"/>
 </robot>

File: robots/sia5/sia5_with_kinectv2.urdf.xacro (robot description, xacro)
@@ -21,4 +21,4 @@
   </joint>
   <!-- Gazebo -->
-  <xacro:kinect_gazebo name="kinect2"/>
+  <xacro:kinect_gazebo suffix="" name="kinect2"/>
 </robot>

File: urdf/sensor/kinect.gazebo.xacro (robot description, xacro)
@@ -2,32 +2,32 @@
 <robot xmlns:xacro="http://ros.org/wiki/xacro">
   <xacro:include filename="$(find motoman_description)/urdf/common.xacro" />
-  <xacro:macro name="kinect_gazebo" params="name">
-	<gazebo reference="${name}_link">
-	  <mu1>0.2</mu1>
-	  <mu2>0.2</mu2>
-	  <material>Gazebo/Black</material>
-	  <!-- hd -->
+  <xacro:macro name="kinect_gazebo" params="name suffix">
+    <gazebo reference="${name}_link">
+      <mu1>0.2</mu1>
+      <mu2>0.2</mu2>
+      <material>Gazebo/Black</material>
+      <!-- hd -->
       <sensor type="depth" name="${name}">
-		<always_on>true</always_on>
-		<update_rate>30.0</update_rate>
-		<camera>
+        <always_on>true</always_on>
+        <update_rate>30.0</update_rate>
+        <camera>
           <horizontal_fov>${84.1*M_PI/180.0}</horizontal_fov>
           <image>
-			<format>R8G8B8</format>
-			<width>512</width>
-			<height>424</height>
+        <format>R8G8B8</format>
+        <width>512</width>
+        <height>424</height>
           </image>
           <clip>
-			<near>0.05</near>
-			<far>4.5</far>
+        <near>0.05</near>
+        <far>4.5</far>
           </clip>
-		  <noise>
-			<type>gaussian</type>
-			<mean>0.0</mean>
-			<stddev>0.005</stddev>
-		  </noise>
-		</camera>
-		<plugin name="${name}_camera_controller" filename="libgazebo_ros_openni_kinect.so">
-          <cameraName>kinect2/hd</cameraName>
+          <noise>
+            <type>gaussian</type>
+            <mean>0.0</mean>
+            <stddev>0.005</stddev>
+          </noise>
+        </camera>
+        <plugin name="${name}_camera_controller" filename="libgazebo_ros_openni_kinect.so">
+          <cameraName>${suffix}/kinect2/hd</cameraName>
           <alwaysOn>true</alwaysOn>
           <updateRate>30</updateRate>
@@ -45,30 +45,30 @@
           <distortion_t2>0.0</distortion_t2>
           <pointCloudCutoff>0.05</pointCloudCutoff>
-		  <pointCloudCutoffMax>4.5</pointCloudCutoffMax>
-		</plugin>
+          <pointCloudCutoffMax>4.5</pointCloudCutoffMax>
+        </plugin>
       </sensor>
-	  <!-- qhd -->
+      <!-- qhd -->
       <sensor type="depth" name="${name}">
-		<always_on>true</always_on>
-		<update_rate>30.0</update_rate>
-		<camera>
+        <always_on>true</always_on>
+        <update_rate>30.0</update_rate>
+        <camera>
           <horizontal_fov>${84.1*M_PI/180.0}</horizontal_fov>
           <image>
-			<format>R8G8B8</format>
-			<width>512</width>
-			<height>424</height>
+            <format>R8G8B8</format>
+            <width>512</width>
+            <height>424</height>
           </image>
           <clip>
-			<near>0.05</near>
-			<far>4.5</far>
+            <near>0.05</near>
+            <far>4.5</far>
           </clip>
-		  <noise>
-			<type>gaussian</type>
-			<mean>0.0</mean>
-			<stddev>0.005</stddev>
-		  </noise>
-		</camera>
-		<plugin name="${name}_camera_controller" filename="libgazebo_ros_openni_kinect.so">
-          <cameraName>kinect2/qhd</cameraName>
+          <noise>
+            <type>gaussian</type>
+            <mean>0.0</mean>
+            <stddev>0.005</stddev>
+          </noise>
+        </camera>
+        <plugin name="${name}_camera_controller" filename="libgazebo_ros_openni_kinect.so">
+          <cameraName>${suffix}/kinect2/qhd</cameraName>
           <alwaysOn>true</alwaysOn>
           <updateRate>30</updateRate>
@@ -86,30 +86,30 @@
           <distortion_t2>0.0</distortion_t2>
           <pointCloudCutoff>0.05</pointCloudCutoff>
-		  <pointCloudCutoffMax>4.5</pointCloudCutoffMax>
-		</plugin>
+          <pointCloudCutoffMax>4.5</pointCloudCutoffMax>
+        </plugin>
       </sensor>
 	  <!-- sd -->
       <sensor type="depth" name="${name}">
-		<always_on>true</always_on>
-		<update_rate>30.0</update_rate>
-		<camera>
+        <always_on>true</always_on>
+        <update_rate>30.0</update_rate>
+        <camera>
           <horizontal_fov>${84.1*M_PI/180.0}</horizontal_fov>
           <image>
-			<format>R8G8B8</format>
-			<width>512</width>
-			<height>424</height>
+            <format>R8G8B8</format>
+            <width>512</width>
+            <height>424</height>
           </image>
           <clip>
-			<near>0.05</near>
-			<far>4.5</far>
+          <near>0.05</near>
+          <far>4.5</far>
           </clip>
-		  <noise>
-			<type>gaussian</type>
-			<mean>0.0</mean>
-			<stddev>0.005</stddev>
-		  </noise>
-		</camera>
-		<plugin name="${name}_camera_controller" filename="libgazebo_ros_openni_kinect.so">
-          <cameraName>kinect2/sd</cameraName>
+          <noise>
+            <type>gaussian</type>
+            <mean>0.0</mean>
+            <stddev>0.005</stddev>
+          </noise>
+        </camera>
+        <plugin name="${name}_camera_controller" filename="libgazebo_ros_openni_kinect.so">
+          <cameraName>${suffix}/kinect2/sd</cameraName>
           <alwaysOn>true</alwaysOn>
           <updateRate>30</updateRate>
@@ -127,8 +127,8 @@
           <distortion_t2>0.0</distortion_t2>
           <pointCloudCutoff>0.05</pointCloudCutoff>
-		  <pointCloudCutoffMax>4.5</pointCloudCutoffMax>
-		</plugin>
+          <pointCloudCutoffMax>4.5</pointCloudCutoffMax>
+        </plugin>
       </sensor>
-	</gazebo>
+    </gazebo>
   </xacro:macro>
 </robot>

File: urdf/sensor/kinect.urdf.xacro (robot description, xacro)
@@ -1,8 +1,8 @@
 <?xml version="1.0"?>
 <robot xmlns:xacro="http://ros.org/wiki/xacro">
-<xacro:macro name="kinect2_link_box_v0" params="name">
+  <xacro:macro name="kinect2_link_box_v0" params="name">
     <link name="${name}">
       <visual>
-		<material name="black"/>
+        <material name="black"/>
         <geometry>
           <mesh filename="package://motoman_description/meshes/sensor/visual/COLLADA/kinectv2.stl"/>
@@ -10,7 +10,7 @@
       </visual>
       <collision>
-		<origin xyz="0 0 0.041"/>
+        <origin xyz="0 0 0.041"/>
         <geometry>
-		  <box size="0.065 0.25 0.082"/>
+          <box size="0.065 0.25 0.082"/>
         </geometry>
       </collision>
@@ -18,8 +18,25 @@
         <mass value="0.935"/>
         <inertia ixx="0.0053937" ixy="0" ixz="0"
-				 iyy="0.00085311" iyz="0"
-				 izz="0.00519899" />
+                 iyy="0.00085311" iyz="0"
+                 izz="0.00519899" />
       </inertial>
     </link>
-</xacro:macro>
+  </xacro:macro>
+  <xacro:macro name="kinect_joints" params="suffix rpy xyz">
+    <xacro:kinect2_link_box_v0 name="${suffix}/kinect2_link"/>
+    <link name="${suffix}/kinect2_rgb_optical_frame"/>
+    <!-- Joint -->
+    <joint name="${suffix}/joint_kinect2" type="fixed">
+      <origin rpy="${rpy}" xyz="${xyz}"/>
+      <parent link="base_link"/>
+      <child link="${suffix}/kinect2_link"/>
+    </joint>
+    <joint name="${suffix}/joint_rgb_kinect2" type="fixed">
+      <origin rpy="${M_PI/2} ${M_PI} ${M_PI/2}"/>
+      <parent link="${suffix}/kinect2_link"/>
+      <child link="${suffix}/kinect2_rgb_optical_frame"/>
+    </joint>
+    <!-- Gazebo -->
+    <xacro:kinect_gazebo name="${suffix}/kinect2" suffix="${suffix}"/>
+  </xacro:macro>
 </robot>

Commit message: [modify] gazeboモデルには風船をつけておくことにします。
モデル上ではうまく行っているので、そのように判断しました。

File: robots/sia5/sia5_gazebo_nishida_lab.urdf.xacro (robot description, xacro)
@@ -28,13 +28,12 @@
   <xacro:kinect_gazebo suffix=""  name="kinect2"/>
   <!-- add Jamming Gripper -->
-   <!-- Link -->
+  <!-- Link -->
   <xacro:tool_link_cylinder_v0 name="gripper_link" mass="1.0"
   							   radius="0.0965" height="0.61445"
   							   ox="0" oy="0" oz="0"
   							   oroll="0" opitch="0" oyaw="0"/>
-  <link name="balloon"/>
-  <!-- <xacro:tool_link_no_collision_v0 name="balloon" mass="0.3" -->
-  <!-- 								   ixx="0.001" ixy="0" ixz="0" -->
-  <!-- 								   iyy="0.001" iyz="0" izz="0.001"/> -->
+  <xacro:tool_link_no_collision_v0 name="balloon" mass="0.3"
+  								   ixx="0.001" ixy="0" ixz="0"
+  								   iyy="0.001" iyz="0" izz="0.001"/>
   <!-- Joint  -->
   <joint name="joint_gripper" type="fixed">
