Commit message: [modify] 前回と一緒

File: robots/sia5/sia5.urdf.xacro (robot description, xacro)
@@ -25,39 +25,40 @@
   <xacro:property name="b_axis_velocity_limit" value="${230.0*M_PI/180.0}"/>
   <xacro:property name="t_axis_velocity_limit" value="${350.0*M_PI/180.0}"/>
-  <!-- link -->
-  <xacro:base_link_v0 color="blue" mass="${30.0/sum*base}"
-					  ixx="0.006046" ixy="0.000006" ixz="-0.000237"
-					  iyy="0.006272" iyz="0.000011" izz="0.006950"/>
-  <xacro:link_v0 name="s" color="white" mass="${30.0/sum*s}"
+  <xacro:link_v1 name="base_link" color="blue" mass="${30.0/sum*base}"
+				 ixx="0.006046" ixy="0.000006" ixz="-0.000237"
+				 iyy="0.006272" iyz="0.000011" izz="0.006950"/>
+  <xacro:link_v1 name="link_s" color="white" mass="${30.0/sum*s}"
 				 ixx="0.005277" ixy="-0.000002" ixz="-0.000002"
 				 iyy="0.005321" iyz="-0.000384" izz="0.003218"/>
-  <xacro:link_v0 name="l" color="blue" mass="${30.0/sum*l}"
+  <xacro:link_v1 name="link_l" color="blue" mass="${30.0/sum*l}"
 				 ixx="0.004612" ixy="0.000001" ixz="-0.000003"
 				 iyy="0.004681" iyz="-0.000652" izz="0.001990"/>
-  <xacro:link_v0 name="e" color="white" mass="${30.0/sum*e}"
+  <xacro:link_v1 name="link_e" color="white" mass="${30.0/sum*e}"
 				 ixx="0.002892" ixy="-0.000172" ixz="-0.001110"
 				 iyy="0.004050" iyz="-0.000261" izz="0.003426"/>
-  <xacro:link_v0 name="u" color="blue" mass="${30.0/sum*u}"
+  <xacro:link_v1 name="link_u" color="blue" mass="${30.0/sum*u}"
 				 ixx="0.002100" ixy="-0.000490" ixz="-0.000856"
 				 iyy="0.003544" iyz="-0.000268" izz="0.002971" />
-  <xacro:link_v0 name="r" color="white" mass="${30.0/sum*r}"
+  <xacro:link_v1 name="link_r" color="white" mass="${30.0/sum*r}"
 				 ixx="0.002848" ixy="0.000271" ixz="0.000000"
 				 iyy="0.005945" iyz="0.000000" izz="0.006357"/>
-  <xacro:link_v0 name="b" color="blue" mass="${30.0/sum*b}"
+  <xacro:link_v1 name="link_b" color="blue" mass="${30.0/sum*b}"
 				 ixx="0.001710" ixy="0.000714" ixz="-0.000007"
 				 iyy="0.004150" iyz="0.000002" izz="0.004303"/>
-  <xacro:link_v0 name="t" color="white" mass="${30.0/sum*t}"
+  <xacro:link_v1 name="link_t" color="white" mass="${30.0/sum*t}"
 				 ixx="0.002411" ixy="-0.000001" ixz="0.000002"
 				 iyy="0.001266" iyz="0.000035" izz="0.001206"/>
   <link name="tool0"/>
-  <!-- joint -->
-  <xacro:base_joint_v0 ox="0" oy="0" oz="0.31"
-  					   ax="0" ay="0" az="1"
-  					   el="30.0"
-  					   ll="${s_axis_lower_limit}" ul="${s_axis_upper_limit}"
-  					   vl="${s_axis_velocity_limit}"
-  					   skp="0" skv="0"
-  					   sll="${s_axis_lower_limit}" sul="${s_axis_upper_limit}"/>
-  <xacro:joint_v0 parent_name="s" child_name="l"
+  <xacro:joint_v1 joint_name="joint_s"
+				  parent_name="base_link" child_name="link_s"
+				  ox="0" oy="0" oz="0.31"
+  				  ax="0" ay="0" az="1"
+  				  el="30.0"
+  				  ll="${s_axis_lower_limit}" ul="${s_axis_upper_limit}"
+  				  vl="${s_axis_velocity_limit}"
+  				  skp="0" skv="0"
+  				  sll="${s_axis_lower_limit}" sul="${s_axis_upper_limit}"/>
+  <xacro:joint_v1 joint_name="joint_l"
+				  parent_name="link_s" child_name="link_l"
   				  ox="0" oy="0" oz="0"
   				  ax="0" ay="1" az="0"
@@ -67,5 +68,6 @@
   				  skp="0" skv="0"
   				  sll="${l_axis_lower_limit}" sul="${l_axis_upper_limit}"/>
-  <xacro:joint_v0 parent_name="l" child_name="e"
+  <xacro:joint_v1 joint_name="joint_e"
+				  parent_name="link_l" child_name="link_e"
   				  ox="0" oy="0" oz="0.27"
   				  ax="0" ay="0" az="1"
@@ -75,5 +77,6 @@
   				  skp="0" skv="0"
   				  sll="${e_axis_lower_limit}" sul="${e_axis_upper_limit}"/>
-  <xacro:joint_v0 parent_name="e" child_name="u"
+  <xacro:joint_v1 joint_name="joint_u"
+				  parent_name="link_e" child_name="link_u"
   				  ox="0.085" oy="0" oz="0"
   				  ax="0" ay="1" az="0"
@@ -83,5 +86,6 @@
   				  skp="0" skv="0"
   				  sll="${u_axis_lower_limit}" sul="${u_axis_upper_limit}"/>
-  <xacro:joint_v0 parent_name="u" child_name="r"
+  <xacro:joint_v1 joint_name="joint_r"
+				  parent_name="link_u" child_name="link_r"
   				  ox="0.27" oy="0" oz="0.06"
   				  ax="-1" ay="0" az="0"
@@ -91,5 +95,6 @@
   				  skp="0" skv="0"
   				  sll="${r_axis_lower_limit}" sul="${r_axis_upper_limit}"/>
-  <xacro:joint_v0 parent_name="r" child_name="b"
+  <xacro:joint_v1 joint_name="joint_b"
+				  parent_name="link_r" child_name="link_b"
   				  ox="0" oy="0" oz="0"
   				  ax="0" ay="1" az="0"
@@ -99,5 +104,6 @@
   				  skp="0" skv="0"
 				  sll="${b_axis_lower_limit}" sul="${b_axis_upper_limit}"/>
-  <xacro:joint_v0 parent_name="b" child_name="t"
+  <xacro:joint_v1 joint_name="joint_t"
+				  parent_name="link_b" child_name="link_t"
   				  ox="0.134" oy="0" oz="0"
   				  ax="-1" ay="0" az="0"
@@ -107,5 +113,5 @@
   				  skp="0" skv="0"
   				  sll="${t_axis_lower_limit}" sul="${t_axis_upper_limit}"/>
-  <joint name="link_t-tool0" type="fixed">
+  <joint name="joint_tool0" type="fixed">
     <origin rpy="0 0 0" xyz="0.011 0 0"/>
     <parent link="link_t"/>

Commit message: [modify] モデルを新しくするついでに、ソースのディレクトリ階層も変更

File: robots/sia5/sia5.urdf.xacro (robot description, xacro)
@@ -1,7 +1,7 @@
 <?xml version="1.0"?>
 <robot name="sia5" xmlns:xacro="http://ros.org/wiki/xacro">
-  <xacro:include filename="$(find motoman_description)/urdf/sia5/common.xacro" />
-  <xacro:include filename="$(find motoman_description)/urdf/sia5/materials.xacro"/>
-  <xacro:include filename="$(find motoman_description)/urdf/sia5/body/body.urdf.xacro" />
+  <xacro:include filename="$(find motoman_description)/urdf/common.xacro" />
+  <xacro:include filename="$(find motoman_description)/urdf/materials.xacro"/>
+  <xacro:include filename="$(find motoman_description)/urdf/sia5/body.urdf.xacro" />
   <xacro:property name="s_axis_upper_limit" value="${180.0*M_PI/180.0}"/>
   <xacro:property name="s_axis_lower_limit" value="-${s_axis_upper_limit}"/>
@@ -25,32 +25,32 @@
   <xacro:property name="b_axis_velocity_limit" value="${230.0*M_PI/180.0}"/>
   <xacro:property name="t_axis_velocity_limit" value="${350.0*M_PI/180.0}"/>
-  <xacro:link_v1 name="base_link" color="blue" mass="${30.0/sum*base}"
-				 ixx="0.006046" ixy="0.000006" ixz="-0.000237"
-				 iyy="0.006272" iyz="0.000011" izz="0.006950"/>
-  <xacro:link_v1 name="link_s" color="white" mass="${30.0/sum*s}"
-				 ixx="0.005277" ixy="-0.000002" ixz="-0.000002"
-				 iyy="0.005321" iyz="-0.000384" izz="0.003218"/>
-  <xacro:link_v1 name="link_l" color="blue" mass="${30.0/sum*l}"
-				 ixx="0.004612" ixy="0.000001" ixz="-0.000003"
-				 iyy="0.004681" iyz="-0.000652" izz="0.001990"/>
-  <xacro:link_v1 name="link_e" color="white" mass="${30.0/sum*e}"
-				 ixx="0.002892" ixy="-0.000172" ixz="-0.001110"
-				 iyy="0.004050" iyz="-0.000261" izz="0.003426"/>
-  <xacro:link_v1 name="link_u" color="blue" mass="${30.0/sum*u}"
-				 ixx="0.002100" ixy="-0.000490" ixz="-0.000856"
-				 iyy="0.003544" iyz="-0.000268" izz="0.002971" />
-  <xacro:link_v1 name="link_r" color="white" mass="${30.0/sum*r}"
-				 ixx="0.002848" ixy="0.000271" ixz="0.000000"
-				 iyy="0.005945" iyz="0.000000" izz="0.006357"/>
-  <xacro:link_v1 name="link_b" color="blue" mass="${30.0/sum*b}"
-				 ixx="0.001710" ixy="0.000714" ixz="-0.000007"
-				 iyy="0.004150" iyz="0.000002" izz="0.004303"/>
-  <xacro:link_v1 name="link_t" color="white" mass="${30.0/sum*t}"
-				 ixx="0.002411" ixy="-0.000001" ixz="0.000002"
-				 iyy="0.001266" iyz="0.000035" izz="0.001206"/>
-  <link name="tool0"/>
+  <xacro:link_v1 name="base_link" mass="${base_rate/sum_rate*sum_mass}"
+				 ixx="0.000023" ixy="0.000000" ixz="-0.000001"
+				 iyy="0.000027" iyz="-0.000000" izz="0.000028"/>
+  <xacro:link_v1 name="link_s" mass="${s_rate/sum_rate*sum_mass}"
+  				 ixx="0.000008" ixy="0.000000" ixz="-0.000000"
+  				 iyy="0.000008" iyz="0.000001" izz="0.000004"/>
+  <!-- <xacro:link_v1 name="link_l" color="blue" mass="${30.0/sum*l}" -->
+  <!-- 				 ixx="0.004612" ixy="0.000001" ixz="-0.000003" -->
+  <!-- 				 iyy="0.004681" iyz="-0.000652" izz="0.001990"/> -->
+  <!-- <xacro:link_v1 name="link_e" color="white" mass="${30.0/sum*e}" -->
+  <!-- 				 ixx="0.002892" ixy="-0.000172" ixz="-0.001110" -->
+  <!-- 				 iyy="0.004050" iyz="-0.000261" izz="0.003426"/> -->
+  <!-- <xacro:link_v1 name="link_u" color="blue" mass="${30.0/sum*u}" -->
+  <!-- 				 ixx="0.002100" ixy="-0.000490" ixz="-0.000856" -->
+  <!-- 				 iyy="0.003544" iyz="-0.000268" izz="0.002971" /> -->
+  <!-- <xacro:link_v1 name="link_r" color="white" mass="${30.0/sum*r}" -->
+  <!-- 				 ixx="0.002848" ixy="0.000271" ixz="0.000000" -->
+  <!-- 				 iyy="0.005945" iyz="0.000000" izz="0.006357"/> -->
+  <!-- <xacro:link_v1 name="link_b" color="blue" mass="${30.0/sum*b}" -->
+  <!-- 				 ixx="0.001710" ixy="0.000714" ixz="-0.000007" -->
+  <!-- 				 iyy="0.004150" iyz="0.000002" izz="0.004303"/> -->
+  <!-- <xacro:link_v1 name="link_t" color="white" mass="${30.0/sum*t}" -->
+  <!-- 				 ixx="0.002411" ixy="-0.000001" ixz="0.000002" -->
+  <!-- 				 iyy="0.001266" iyz="0.000035" izz="0.001206"/> -->
+  <!-- <link name="tool0"/> -->
   <xacro:joint_v1 joint_name="joint_s"
-				  parent_name="base_link" child_name="link_s"
-				  ox="0" oy="0" oz="0.31"
+  				  parent_name="base_link" child_name="link_s"
+  				  ox="0" oy="0" oz="0.1765"
   				  ax="0" ay="0" az="1"
   				  el="30.0"
@@ -59,62 +59,62 @@
   				  skp="1" skv="1"
   				  sll="${s_axis_lower_limit}" sul="${s_axis_upper_limit}"/>
-  <xacro:joint_v1 joint_name="joint_l"
-				  parent_name="link_s" child_name="link_l"
-  				  ox="0" oy="0" oz="0"
-  				  ax="0" ay="1" az="0"
-  				  el="30.0"
-  				  ll="${l_axis_lower_limit}" ul="${l_axis_upper_limit}"
-  				  vl="${l_axis_velocity_limit}"
-  				  skp="1" skv="1"
-  				  sll="${l_axis_lower_limit}" sul="${l_axis_upper_limit}"/>
-  <xacro:joint_v1 joint_name="joint_e"
-				  parent_name="link_l" child_name="link_e"
-  				  ox="0" oy="0" oz="0.27"
-  				  ax="0" ay="0" az="1"
-  				  el="30.0"
-  				  ll="${e_axis_lower_limit}" ul="${e_axis_upper_limit}"
-  				  vl="${e_axis_velocity_limit}"
-  				  skp="1" skv="1"
-  				  sll="${e_axis_lower_limit}" sul="${e_axis_upper_limit}"/>
-  <xacro:joint_v1 joint_name="joint_u"
-				  parent_name="link_e" child_name="link_u"
-  				  ox="0.085" oy="0" oz="0"
-  				  ax="0" ay="1" az="0"
-  				  el="30.0"
-  				  ll="${u_axis_lower_limit}" ul="${u_axis_upper_limit}"
-  				  vl="${u_axis_velocity_limit}"
-  				  skp="1" skv="1"
-  				  sll="${u_axis_lower_limit}" sul="${u_axis_upper_limit}"/>
-  <xacro:joint_v1 joint_name="joint_r"
-				  parent_name="link_u" child_name="link_r"
-  				  ox="0.27" oy="0" oz="0.06"
-  				  ax="-1" ay="0" az="0"
-  				  el="14.7"
-  				  ll="${r_axis_lower_limit}" ul="${r_axis_upper_limit}"
-				  vl="${r_axis_velocity_limit}"
-  				  skp="1" skv="1"
-  				  sll="${r_axis_lower_limit}" sul="${r_axis_upper_limit}"/>
-  <xacro:joint_v1 joint_name="joint_b"
-				  parent_name="link_r" child_name="link_b"
-  				  ox="0" oy="0" oz="0"
-  				  ax="0" ay="1" az="0"
-  				  el="14.7"
-				  ll="${b_axis_lower_limit}" ul="${b_axis_upper_limit}"
-				  vl="${b_axis_velocity_limit}"
-  				  skp="1" skv="1"
-				  sll="${b_axis_lower_limit}" sul="${b_axis_upper_limit}"/>
-  <xacro:joint_v1 joint_name="joint_t"
-				  parent_name="link_b" child_name="link_t"
-  				  ox="0.134" oy="0" oz="0"
-  				  ax="-1" ay="0" az="0"
-  				  el="7.35"
-  				  ll="${t_axis_lower_limit}" ul="${t_axis_upper_limit}"
-  				  vl="${t_axis_velocity_limit}"
-  				  skp="1" skv="1"
-  				  sll="${t_axis_lower_limit}" sul="${t_axis_upper_limit}"/>
-  <joint name="joint_tool0" type="fixed">
-    <origin rpy="0 0 0" xyz="0.011 0 0"/>
-    <parent link="link_t"/>
-    <child link="tool0"/>
-  </joint>
+  <!-- <xacro:joint_v1 joint_name="joint_l" -->
+  <!-- 				  parent_name="link_s" child_name="link_l" -->
+  <!-- 				  ox="0" oy="0" oz="0" -->
+  <!-- 				  ax="0" ay="1" az="0" -->
+  <!-- 				  el="30.0" -->
+  <!-- 				  ll="${l_axis_lower_limit}" ul="${l_axis_upper_limit}" -->
+  <!-- 				  vl="${l_axis_velocity_limit}" -->
+  <!-- 				  skp="1" skv="1" -->
+  <!-- 				  sll="${l_axis_lower_limit}" sul="${l_axis_upper_limit}"/> -->
+  <!-- <xacro:joint_v1 joint_name="joint_e" -->
+  <!-- 				  parent_name="link_l" child_name="link_e" -->
+  <!-- 				  ox="0" oy="0" oz="0.27" -->
+  <!-- 				  ax="0" ay="0" az="1" -->
+  <!-- 				  el="30.0" -->
+  <!-- 				  ll="${e_axis_lower_limit}" ul="${e_axis_upper_limit}" -->
+  <!-- 				  vl="${e_axis_velocity_limit}" -->
+  <!-- 				  skp="1" skv="1" -->
+  <!-- 				  sll="${e_axis_lower_limit}" sul="${e_axis_upper_limit}"/> -->
+  <!-- <xacro:joint_v1 joint_name="joint_u" -->
+  <!-- 				  parent_name="link_e" child_name="link_u" -->
+  <!-- 				  ox="0.085" oy="0" oz="0" -->
+  <!-- 				  ax="0" ay="1" az="0" -->
+  <!-- 				  el="30.0" -->
+  <!-- 				  ll="${u_axis_lower_limit}" ul="${u_axis_upper_limit}" -->
+  <!-- 				  vl="${u_axis_velocity_limit}" -->
+  <!-- 				  skp="1" skv="1" -->
+  <!-- 				  sll="${u_axis_lower_limit}" sul="${u_axis_upper_limit}"/> -->
+  <!-- <xacro:joint_v1 joint_name="joint_r" -->
+  <!-- 				  parent_name="link_u" child_name="link_r" -->
+  <!-- 				  ox="0.27" oy="0" oz="0.06" -->
+  <!-- 				  ax="-1" ay="0" az="0" -->
+  <!-- 				  el="14.7" -->
+  <!-- 				  ll="${r_axis_lower_limit}" ul="${r_axis_upper_limit}" -->
+  <!-- 				  vl="${r_axis_velocity_limit}" -->
+  <!-- 				  skp="1" skv="1" -->
+  <!-- 				  sll="${r_axis_lower_limit}" sul="${r_axis_upper_limit}"/> -->
+  <!-- <xacro:joint_v1 joint_name="joint_b" -->
+  <!-- 				  parent_name="link_r" child_name="link_b" -->
+  <!-- 				  ox="0" oy="0" oz="0" -->
+  <!-- 				  ax="0" ay="1" az="0" -->
+  <!-- 				  el="14.7" -->
+  <!-- 				  ll="${b_axis_lower_limit}" ul="${b_axis_upper_limit}" -->
+  <!-- 				  vl="${b_axis_velocity_limit}"				   -->
+  <!-- 				  skp="1" skv="1" -->
+  <!-- 				  sll="${b_axis_lower_limit}" sul="${b_axis_upper_limit}"/> -->
+  <!-- <xacro:joint_v1 joint_name="joint_t" -->
+  <!-- 				  parent_name="link_b" child_name="link_t" -->
+  <!-- 				  ox="0.134" oy="0" oz="0" -->
+  <!-- 				  ax="-1" ay="0" az="0" -->
+  <!-- 				  el="7.35" -->
+  <!-- 				  ll="${t_axis_lower_limit}" ul="${t_axis_upper_limit}" -->
+  <!-- 				  vl="${t_axis_velocity_limit}" -->
+  <!-- 				  skp="1" skv="1" -->
+  <!-- 				  sll="${t_axis_lower_limit}" sul="${t_axis_upper_limit}"/> -->
+  <!-- <joint name="joint_tool0" type="fixed"> -->
+  <!--   <origin rpy="0 0 0" xyz="0.011 0 0"/> -->
+  <!--   <parent link="link_t"/> -->
+  <!--   <child link="tool0"/> -->
+  <!-- </joint> -->
 </robot>

File: urdf/sia5/body.gazebo.xacro (robot description, xacro)
@@ -7,8 +7,8 @@
     </plugin>
   </gazebo>
-  <xacro:macro name="gazebo_link_v0" params="name color">
+  <xacro:macro name="gazebo_link_color_v0" params="name color">
 	<gazebo reference="${name}">
-      <material>Gazebo/${color}</material>
-	</gazebo>
+		<material>Gazebo/${color}</material>
+	  </gazebo>
   </xacro:macro>
 </robot>

File: urdf/sia5/body.urdf.xacro (robot description, xacro)
@@ -1,5 +1,19 @@
 <?xml version="1.0"?>
 <robot name="sia5" xmlns:xacro="http://ros.org/wiki/xacro">
-  <xacro:macro name="link_v1" params="name color mass
+  <!-- about mass rate -->
+  <property name="base_rate" value="1.2" />
+  <property name="s_rate" value="1.0" />
+  <property name="l_rate" value="1.0" />
+  <property name="e_rate" value="1.0" />
+  <property name="u_rate" value="0.7" />
+  <property name="r_rate" value="0.7" />
+  <property name="b_rate" value="0.6" />
+  <property name="t_rate" value="0.2" />
+  <property name="sum_rate" value="${base_rate + s_rate
+								   + l_rate + e_rate
+								   + u_rate + r_rate
+								   + b_rate + t_rate}" />
+  <property name="sum_mass" value="30.0" />
+  <xacro:macro name="link_v1" params="name mass
                                       ixx ixy ixz
                                       iyy iyz izz">
@@ -8,12 +22,11 @@
         <origin rpy="0 0 0" xyz="0 0 0"/>
         <geometry>
-          <mesh filename="package://motoman_description/meshes/sia5/visual/stl/${name}.stl"/>
+          <mesh filename="package://motoman_description/meshes/sia5/visual/COLLADA/${name}.dae"/>
         </geometry>
-        <material name="${color}"/>
       </visual>
       <collision>
         <origin rpy="0 0 0" xyz="0 0 0"/>
         <geometry>
-          <mesh filename="package://motoman_description/meshes/sia5/collision/stl/${name}.stl"/>
+          <mesh filename="package://motoman_description/meshes/sia5/collision/STL/${name}.stl"/>
         </geometry>
       </collision>
@@ -30,5 +43,5 @@
 									   el ll ul vl
 									   skp skv sll sul">
-    <joint name="${joint_name}" type="continuous"><!-- revolute"> -->
+    <joint name="${joint_name}" type="revolute">
       <origin rpy="0 0 0" xyz="${ox} ${oy} ${oz}"/>
       <parent link="${parent_name}"/>

Commit message: [add] link_lを追加

File: robots/sia5/sia5.urdf.xacro (robot description, xacro)
@@ -26,12 +26,15 @@
   <xacro:property name="t_axis_velocity_limit" value="${350.0*M_PI/180.0}"/>
   <xacro:link_v1 name="base_link" mass="${base_rate/sum_rate*sum_mass}"
+				 x="0" y="0" z="0" roll="0" pitch="0" yaw="0"
 				 ixx="0.000023" ixy="0.000000" ixz="-0.000001"
 				 iyy="0.000027" iyz="-0.000000" izz="0.000028"/>
   <xacro:link_v1 name="link_s" mass="${s_rate/sum_rate*sum_mass}"
+				 x="0" y="0" z="0" roll="0" pitch="0" yaw="0"
   				 ixx="0.000008" ixy="0.000000" ixz="-0.000000"
   				 iyy="0.000008" iyz="0.000001" izz="0.000004"/>
-  <!-- <xacro:link_v1 name="link_l" color="blue" mass="${30.0/sum*l}" -->
-  <!-- 				 ixx="0.004612" ixy="0.000001" ixz="-0.000003" -->
-  <!-- 				 iyy="0.004681" iyz="-0.000652" izz="0.001990"/> -->
+  <xacro:link_v1 name="link_l" mass="${l_rate/sum_rate*sum_mass}"
+				 x="0" y="0" z="0" roll="${-M_PI/2.0}" pitch="0" yaw="0"
+  				 ixx="0.000011" ixy="0.000000" ixz="0.000000"
+  				 iyy="0.000005" iyz="-0.000002" izz="0.000012"/>
   <!-- <xacro:link_v1 name="link_e" color="white" mass="${30.0/sum*e}" -->
   <!-- 				 ixx="0.002892" ixy="-0.000172" ixz="-0.001110" -->
@@ -59,13 +62,13 @@
   				  skp="1" skv="1"
   				  sll="${s_axis_lower_limit}" sul="${s_axis_upper_limit}"/>
-  <!-- <xacro:joint_v1 joint_name="joint_l" -->
-  <!-- 				  parent_name="link_s" child_name="link_l" -->
-  <!-- 				  ox="0" oy="0" oz="0" -->
-  <!-- 				  ax="0" ay="1" az="0" -->
-  <!-- 				  el="30.0" -->
-  <!-- 				  ll="${l_axis_lower_limit}" ul="${l_axis_upper_limit}" -->
-  <!-- 				  vl="${l_axis_velocity_limit}" -->
-  <!-- 				  skp="1" skv="1" -->
-  <!-- 				  sll="${l_axis_lower_limit}" sul="${l_axis_upper_limit}"/> -->
+  <xacro:joint_v1 joint_name="joint_l"
+  				  parent_name="link_s" child_name="link_l"
+  				  ox="0" oy=" 0.006" oz="0.136"
+  				  ax="0" ay="1" az="0"
+  				  el="30.0"
+  				  ll="${l_axis_lower_limit}" ul="${l_axis_upper_limit}"
+  				  vl="${l_axis_velocity_limit}"
+  				  skp="1" skv="1"
+  				  sll="${l_axis_lower_limit}" sul="${l_axis_upper_limit}"/>
   <!-- <xacro:joint_v1 joint_name="joint_e" -->
   <!-- 				  parent_name="link_l" child_name="link_e" -->

File: urdf/sia5/body.urdf.xacro (robot description, xacro)
@@ -16,9 +16,10 @@
   <property name="sum_mass" value="30.0" />
   <xacro:macro name="link_v1" params="name mass
+									  x y z roll pitch yaw
                                       ixx ixy ixz
                                       iyy iyz izz">
     <link name="${name}">
       <visual>
-        <origin rpy="0 0 0" xyz="0 0 0"/>
+        <origin rpy="${roll} ${pitch} ${yaw}" xyz="${x} ${y} ${z}"/>
         <geometry>
           <mesh filename="package://motoman_description/meshes/sia5/visual/COLLADA/${name}.dae"/>
@@ -26,5 +27,5 @@
       </visual>
       <collision>
-        <origin rpy="0 0 0" xyz="0 0 0"/>
+		<origin rpy="${roll} ${pitch} ${yaw}" xyz="${x} ${y} ${z}"/>
         <geometry>
           <mesh filename="package://motoman_description/meshes/sia5/collision/STL/${name}.stl"/>
