Commit message: [fix] izzが0なのが原因でした。。。マジかよ。。。
やはり、徹底的に自分を疑え。

File: robots/sia5/sia5.urdf.xacro (robot description, xacro)
@@ -29,31 +29,27 @@
   <xacro:link_v1 name="base_link" mass="${base_rate/sum_rate*sum_mass}"
 				 ixx="1.0" ixy="0.0" ixz="0.0"
-				 iyy="1.0" iyz="0.0" izz="0.0"/>
+				 iyy="1.0" iyz="0.0" izz="1.0"/>
   <xacro:link_v1 name="link_s" mass="${s_rate/sum_rate*sum_mass}"
   				 ixx="1.0" ixy="0.0" ixz="0.0"
-				 iyy="1.0" iyz="0.0" izz="0.0"/>
+				 iyy="1.0" iyz="0.0" izz="1.0"/>
   <xacro:link_v1 name="link_l" mass="${l_rate/sum_rate*sum_mass}"
   				 ixx="1.0" ixy="0.0" ixz="0.0"
-  				 iyy="1.0" iyz="0.0" izz="0.0"/>
-  <!-- <xacro:link_v1 name="link_e"  mass="${e_rate/sum_rate*sum_mass}" -->
-  <!-- 				 ixx="1.0" ixy="0.0" ixz="0.0" -->
-  <!-- 				 iyy="1.0" iyz="0.0" izz="0.0"/> -->
-  <!-- <xacro:link_v1 name="link_u" mass="${u_rate/sum_rate*sum_mass}" -->
-  <!-- 				 x="0" y="0" z="0" roll="${M_PI/2.0}" pitch="0" yaw="0" -->
-  <!-- 				 ixx="1.0" ixy="0.0" ixz="0.0" -->
-  <!-- 				 iyy="1.0" iyz="0.0" izz="0.0"/> -->
-  <!-- <xacro:link_v1 name="link_r" mass="${r_rate/sum_rate*sum_mass}" -->
-  <!-- 				 x="0" y="0" z="0" roll="${M_PI/2.0}" pitch="0" yaw="${M_PI/2.0}" -->
-  <!-- 				 ixx="1.0" ixy="0.0" ixz="0.0" -->
-  <!-- 				 iyy="1.0" iyz="0.0" izz="0.0"/> -->
-  <!-- <xacro:link_v1 name="link_b" mass="${b_rate/sum_rate*sum_mass}" -->
-  <!-- 				 x="0" y="0" z="0" roll="${M_PI/2.0}" pitch="0" yaw="0" -->
-  <!-- 				 ixx="1.0" ixy="0.0" ixz="0.0" -->
-  <!-- 				 iyy="1.0" iyz="0.0" izz="0.0"/> -->
-  <!-- <xacro:link_v1 name="link_t" mass="${t_rate/sum_rate*sum_mass}" -->
-  <!-- 				 x="0" y="0" z="0" roll="0" pitch="0" yaw="0" -->
-  <!-- 				 ixx="1.0" ixy="0.0" ixz="0.0" -->
-  <!-- 				 iyy="1.0" iyz="0.0" izz="0.0"/> -->
-  <!-- <link name="tool0"/> -->
+  				 iyy="1.0" iyz="0.0" izz="1.0"/>
+  <xacro:link_v1 name="link_e"  mass="${e_rate/sum_rate*sum_mass}"
+  				 ixx="1.0" ixy="0.0" ixz="0.0"
+  				 iyy="1.0" iyz="0.0" izz="1.0"/>
+  <xacro:link_v1 name="link_u" mass="${u_rate/sum_rate*sum_mass}"
+  				 ixx="1.0" ixy="0.0" ixz="0.0"
+  				 iyy="1.0" iyz="0.0" izz="1.0"/>
+  <xacro:link_v1 name="link_r" mass="${r_rate/sum_rate*sum_mass}"
+  				 ixx="1.0" ixy="0.0" ixz="0.0"
+  				 iyy="1.0" iyz="0.0" izz="1.0"/>
+  <xacro:link_v1 name="link_b" mass="${b_rate/sum_rate*sum_mass}"
+  				 ixx="1.0" ixy="0.0" ixz="0.0"
+  				 iyy="1.0" iyz="0.0" izz="1.0"/>
+  <xacro:link_v1 name="link_t" mass="${t_rate/sum_rate*sum_mass}"
+  				 ixx="1.0" ixy="0.0" ixz="0.0"
+  				 iyy="1.0" iyz="0.0" izz="1.0"/>
+  <link name="tool0"/>
   <!-- joint -->
   <joint name="world" type="fixed">
@@ -81,55 +77,58 @@
   				  skp="1" skv="1"
   				  sll="${l_axis_lower_limit}" sul="${l_axis_upper_limit}"/>
-  <!-- <xacro:joint_v1 joint_name="joint_e" -->
-  <!-- 				  parent_name="link_l" child_name="link_e" -->
-  <!-- 				  ox="0" oy="-0.006" oz="0.15" -->
-  <!-- 				  roll="0" pitch="0" yaw="0" -->
-  <!-- 				  ax="0" ay="0" az="1" -->
-  <!-- 				  el="30.0" -->
-  <!-- 				  ll="${e_axis_lower_limit}" ul="${e_axis_upper_limit}" -->
-  <!-- 				  vl="${e_axis_velocity_limit}" -->
-  <!-- 				  skp="1" skv="1" -->
-  <!-- 				  sll="${e_axis_lower_limit}" sul="${e_axis_upper_limit}"/> -->
-  <!-- <xacro:joint_v1 joint_name="joint_u" -->
-  <!-- 				  parent_name="link_e" child_name="link_u" -->
-  <!-- 				  ox="0.085" oy="-0.00826931" oz="0.12275299" -->
-  <!-- 				  ax="0" ay="-1" az="0" -->
-  <!-- 				  el="30.0" -->
-  <!-- 				  ll="${u_axis_lower_limit}" ul="${u_axis_upper_limit}" -->
-  <!-- 				  vl="${u_axis_velocity_limit}" -->
-  <!-- 				  skp="1" skv="1" -->
-  <!-- 				  sll="${u_axis_lower_limit}" sul="${u_axis_upper_limit}"/> -->
-  <!-- <xacro:joint_v1 joint_name="joint_r" -->
-  <!-- 				  parent_name="link_u" child_name="link_r" -->
-  <!-- 				  ox="0.131" oy="0.008" oz="0.06" -->
-  <!-- 				  ax="-1" ay="0" az="0" -->
-  <!-- 				  el="14.7" -->
-  <!-- 				  ll="${r_axis_lower_limit}" ul="${r_axis_upper_limit}" -->
-  <!-- 				  vl="${r_axis_velocity_limit}" -->
-  <!-- 				  skp="1" skv="1" -->
-  <!-- 				  sll="${r_axis_lower_limit}" sul="${r_axis_upper_limit}"/> -->
-  <!-- <xacro:joint_v1 joint_name="joint_b" -->
-  <!-- 				  parent_name="link_r" child_name="link_b" -->
-  <!-- 				  ox="0.139" oy="-0.0045" oz="0" -->
-  <!-- 				  ax="0" ay="-1" az="0" -->
-  <!-- 				  el="14.7" -->
-  <!-- 				  ll="${b_axis_lower_limit}" ul="${b_axis_upper_limit}" -->
-  <!-- 				  vl="${b_axis_velocity_limit}" -->
-  <!-- 				  skp="1" skv="1" -->
-  <!-- 				  sll="${b_axis_lower_limit}" sul="${b_axis_upper_limit}"/> -->
-  <!-- <xacro:joint_v1 joint_name="joint_t" -->
-  <!-- 				  parent_name="link_b" child_name="link_t" -->
-  <!-- 				  ox="0.1365" oy="0.0045" oz="0" -->
-  <!-- 				  ax="-1" ay="0" az="0" -->
-  <!-- 				  el="7.35" -->
-  <!-- 				  ll="${t_axis_lower_limit}" ul="${t_axis_upper_limit}" -->
-  <!-- 				  vl="${t_axis_velocity_limit}" -->
-  <!-- 				  skp="1" skv="1" -->
-  <!-- 				  sll="${t_axis_lower_limit}" sul="${t_axis_upper_limit}"/> -->
-  <!-- <joint name="joint_tool0" type="fixed"> -->
-  <!--   <origin rpy="0 0 0" xyz="0.0115 0 0"/> -->
-  <!--   <parent link="link_t"/> -->
-  <!--   <child link="tool0"/> -->
-  <!-- </joint> -->
-  <!-- transmission -->
+  <xacro:joint_v1 joint_name="joint_e"
+  				  parent_name="link_l" child_name="link_e"
+  				  ox="0" oy="-0.006" oz="0.15"
+  				  roll="0" pitch="0" yaw="0"
+  				  ax="0" ay="0" az="1"
+  				  el="30.0"
+  				  ll="${e_axis_lower_limit}" ul="${e_axis_upper_limit}"
+  				  vl="${e_axis_velocity_limit}"
+  				  skp="1" skv="1"
+  				  sll="${e_axis_lower_limit}" sul="${e_axis_upper_limit}"/>
+  <xacro:joint_v1 joint_name="joint_u"
+  				  parent_name="link_e" child_name="link_u"
+  				  ox="0.085" oy="-0.00826931" oz="0.12275299"
+				  roll="${M_PI/2.0}" pitch="0" yaw="0"
+  				  ax="0" ay="0" az="1"
+  				  el="30.0"
+  				  ll="${u_axis_lower_limit}" ul="${u_axis_upper_limit}"
+  				  vl="${u_axis_velocity_limit}"
+  				  skp="1" skv="1"
+  				  sll="${u_axis_lower_limit}" sul="${u_axis_upper_limit}"/>
+  <xacro:joint_v1 joint_name="joint_r"
+  				  parent_name="link_u" child_name="link_r"
+  				  ox="0.131" oy="0.06" oz="-0.008"
+				  roll="0" pitch="${M_PI/2}" yaw="0"
+  				  ax="0" ay="0" az="-1"
+  				  el="14.7"
+  				  ll="${r_axis_lower_limit}" ul="${r_axis_upper_limit}"
+  				  vl="${r_axis_velocity_limit}"
+  				  skp="1" skv="1"
+  				  sll="${r_axis_lower_limit}" sul="${r_axis_upper_limit}"/>
+  <xacro:joint_v1 joint_name="joint_b"
+  				  parent_name="link_r" child_name="link_b"
+  				  ox="-0.0045" oy="0" oz="0.139"
+				  roll="0" pitch="${-M_PI/2}" yaw="0"
+  				  ax="0" ay="0" az="1"
+  				  el="14.7"
+  				  ll="${b_axis_lower_limit}" ul="${b_axis_upper_limit}"
+  				  vl="${b_axis_velocity_limit}"
+  				  skp="1" skv="1"
+  				  sll="${b_axis_lower_limit}" sul="${b_axis_upper_limit}"/>
+  <xacro:joint_v1 joint_name="joint_t"
+  				  parent_name="link_b" child_name="link_t"
+  				  ox="0.1365" oy="0.0045" oz="0"
+				  roll="0" pitch="0" yaw="0"
+  				  ax="-1" ay="0" az="0"
+  				  el="7.35"
+  				  ll="${t_axis_lower_limit}" ul="${t_axis_upper_limit}"
+  				  vl="${t_axis_velocity_limit}"
+  				  skp="1" skv="1"
+  				  sll="${t_axis_lower_limit}" sul="${t_axis_upper_limit}"/>
+  <joint name="joint_tool0" type="fixed">
+    <origin rpy="0 0 0" xyz="0.0115 0 0"/>
+    <parent link="link_t"/>
+    <child link="tool0"/>
+  </joint>
 </robot>

File: urdf/sia5/body.urdf.xacro (robot description, xacro)
@@ -20,5 +20,4 @@
     <link name="${name}">
       <visual>
-        <origin rpy="0 0 0" xyz="0 0 0"/>
         <geometry>
           <mesh filename="package://motoman_description/meshes/sia5/visual/COLLADA/${name}.dae"/>
@@ -26,5 +25,4 @@
       </visual>
       <collision>
-		<origin rpy="0 0 0" xyz="0 0 0"/>
         <geometry>
           <mesh filename="package://motoman_description/meshes/sia5/collision/STL/${name}.stl"/>
@@ -33,5 +31,4 @@
       <inertial>
         <mass value="${mass}"/>
-        <origin rpy="0 0 0" xyz="0 0 0"/>
         <inertia ixx="${ixx}" ixy="${ixy}" ixz="${ixz}" iyy="${iyy}" iyz="${iyz}" izz="${izz}" />
       </inertial>

Commit message: [fix] joint_s joint_r joint_t の limit値を変更
それぞれのlimit値が、-180[deg]〜180[deg] であったので、
うまくいかなかったと考えられる。
今回は、 -179.9999[deg]〜179.9999[deg] に設定することで回避。

File: robots/sia5/sia5.urdf.xacro (robot description, xacro)
@@ -7,5 +7,5 @@
   <xacro:include filename="$(find motoman_description)/gazebo/sia5/sia5.gazebo.xacro"/>
   <property name="sum_mass" value="30.0" />
-  <xacro:property name="s_axis_upper_limit" value="${180.0*M_PI/180.0}"/>
+  <xacro:property name="s_axis_upper_limit" value="${179.99999*M_PI/180.0}"/>
   <xacro:property name="s_axis_lower_limit" value="-${s_axis_upper_limit}"/>
   <xacro:property name="l_axis_upper_limit" value="${110.0*M_PI/180.0}"/>
@@ -15,9 +15,9 @@
   <xacro:property name="u_axis_upper_limit" value="${115.0*M_PI/180.0}"/>
   <xacro:property name="u_axis_lower_limit" value="${-90.0*M_PI/180.0}"/>
-  <xacro:property name="r_axis_upper_limit" value="${180.0*M_PI/180.0}"/>
+  <xacro:property name="r_axis_upper_limit" value="${179.99999*M_PI/180.0}"/>
   <xacro:property name="r_axis_lower_limit" value="-${r_axis_upper_limit}"/>
   <xacro:property name="b_axis_upper_limit" value="${110.0*M_PI/180.0}"/>
   <xacro:property name="b_axis_lower_limit" value="-${b_axis_upper_limit}"/>
-  <xacro:property name="t_axis_upper_limit" value="${180.0*M_PI/180.0}"/>
+  <xacro:property name="t_axis_upper_limit" value="${179.99999*M_PI/180.0}"/>
   <xacro:property name="t_axis_lower_limit" value="-${t_axis_upper_limit}"/>
   <xacro:property name="s_axis_velocity_limit" value="${200.0*M_PI/180.0}"/>

Commit message: [modify] tool_0の位置を変更

File: robots/sia5/sia5.urdf.xacro (robot description, xacro)
@@ -131,5 +131,5 @@
   				  sll="${t_axis_lower_limit}" sul="${t_axis_upper_limit}"/>
   <joint name="joint_tool0" type="fixed">
-    <origin rpy="0 0 0" xyz="0.0115 0 0"/>
+    <origin rpy="0 0 0" xyz="0.0115 0 -0.040"/>
     <parent link="link_t"/>
     <child link="tool0"/>

Commit message: [modify] massの記述位置を変更

File: robots/sia5/sia5.urdf.xacro (robot description, xacro)
@@ -1,4 +1,5 @@
 <?xml version="1.0"?>
 <robot name="sia5" xmlns:xacro="http://ros.org/wiki/xacro">
+  <!-- File Include -->
   <xacro:include filename="$(find motoman_description)/urdf/common.xacro" />
   <xacro:include filename="$(find motoman_description)/urdf/materials.xacro"/>
@@ -6,5 +7,17 @@
   <xacro:include filename="$(find motoman_description)/urdf/sia5/body.transmission.xacro"/>
   <xacro:include filename="$(find motoman_description)/gazebo/sia5/sia5.gazebo.xacro"/>
+  <!-- Mass -->
   <property name="sum_mass" value="30.0" />
+  <!-- about mass rate -->
+  <property name="base_rate" value="6.9" />
+  <property name="s_rate" value="6.6" />
+  <property name="l_rate" value="6.0" />
+  <property name="e_rate" value="4.3" />
+  <property name="u_rate" value="3.7"/>
+  <property name="r_rate" value="1.5" />
+  <property name="b_rate" value="1.0" />
+  <property name="t_rate" value="0.3" />
+  <!-- Hard ware limits -->
+  <!-- Range limits -->
   <xacro:property name="s_axis_upper_limit" value="${179.99999*M_PI/180.0}"/>
   <xacro:property name="s_axis_lower_limit" value="-${s_axis_upper_limit}"/>
@@ -21,4 +34,5 @@
   <xacro:property name="t_axis_upper_limit" value="${179.99999*M_PI/180.0}"/>
   <xacro:property name="t_axis_lower_limit" value="-${t_axis_upper_limit}"/>
+  <!-- Velocity limits -->
   <xacro:property name="s_axis_velocity_limit" value="${200.0*M_PI/180.0}"/>
   <xacro:property name="l_axis_velocity_limit" value="${200.0*M_PI/180.0}"/>
@@ -139,5 +153,5 @@
   				  sll="${t_axis_lower_limit}" sul="${t_axis_upper_limit}"/>
   <joint name="joint_tool0" type="fixed">
-    <origin rpy="0 0 0" xyz="0.0115 0 0"/>
+    <origin rpy="0 0 0" xyz="0.0115 0 -0.040"/>
     <parent link="link_t"/>
     <child link="tool0"/>

File: urdf/sia5/body.urdf.xacro (robot description, xacro)
@@ -1,13 +1,4 @@
 <?xml version="1.0"?>
 <robot xmlns:xacro="http://ros.org/wiki/xacro">
-  <!-- about mass rate -->
-  <property name="base_rate" value="6.9" />
-  <property name="s_rate" value="6.6" />
-  <property name="l_rate" value="6.0" />
-  <property name="e_rate" value="4.3" />
-  <property name="u_rate" value="3.7"/>
-  <property name="r_rate" value="1.5" />
-  <property name="b_rate" value="1.0" />
-  <property name="t_rate" value="0.3" />
   <property name="sum_rate" value="${base_rate + s_rate
 								   + l_rate + e_rate

Commit message: [add] 円柱と箱の近似イナーシャ等を追加
link_cylinder_v0 と link_box_v0 で追加

File: robots/sia5/sia5.urdf.xacro (robot description, xacro)
@@ -10,12 +10,12 @@
   <property name="sum_mass" value="30.0" />
   <!-- about mass rate -->
-  <property name="base_rate" value="6.9" />
-  <property name="s_rate" value="6.6" />
-  <property name="l_rate" value="6.0" />
-  <property name="e_rate" value="4.3" />
-  <property name="u_rate" value="3.7"/>
-  <property name="r_rate" value="1.5" />
-  <property name="b_rate" value="1.0" />
-  <property name="t_rate" value="0.3" />
+  <property name="base_rate" value="6.4" />
+  <property name="s_rate" value="6.1" />
+  <property name="l_rate" value="5.5" />
+  <property name="e_rate" value="4.0" />
+  <property name="u_rate" value="3.5"/>
+  <property name="r_rate" value="2.0" />
+  <property name="b_rate" value="1.5" />
+  <property name="t_rate" value="1.0" />
   <!-- Hard ware limits -->
   <!-- Range limits -->
@@ -44,8 +44,7 @@
   <!-- link -->
   <link name="world"/>
-  <xacro:link_v1 name="base_link" mass="${base_rate/sum_rate*sum_mass}"
-				 ixx="0.001322" ixy="0.0" ixz="0.0"
-				 iyy="0.001281" iyz="0.0"
-				 izz="0.001341"/>
+  <xacro:link_box_v0 name="base_link" mass="${base_rate/sum_rate*sum_mass}"
+					 width="0.08325" depth="0.0988" height="0.07325"
+					 ox="-0.025918" oy="-0.000376" oz="0.076105" oroll="0" opitch="0" oyaw="0"/>
   <xacro:link_v1 name="link_s" mass="${s_rate/sum_rate*sum_mass}"
   				 ixx="0.0012143" ixy="0.0" ixz="0.0"
@@ -72,9 +71,8 @@
   				 iyy="0.0004653" iyz="0.0"
 				 izz="0.0004592"/>
-  <xacro:link_v1 name="link_t" mass="${t_rate/sum_rate*sum_mass}"
-  				 ixx="0.0004568" ixy="0.0" ixz="0.0"
-  				 iyy="0.0006562" iyz="0.0"
-				 izz="0.0005343"/>
-  <link name="tool0"/>
+  <xacro:link_cylinder_v0 name="link_t" mass="${t_rate/sum_rate*sum_mass}"
+					   radius="0.045" height="0.0115"
+					   ox="0.005406" oy="0.0" oz="-0.000191" oroll="0" opitch="0" oyaw="0"/>
+ <link name="tool0"/>
   <!-- joint -->
   <joint name="world" type="fixed">

File: urdf/sia5/body.urdf.xacro (robot description, xacro)
@@ -25,4 +25,48 @@
     </link>
   </xacro:macro>
+  <xacro:macro name="link_cylinder_v0" params="name mass radius height
+											ox oy oz oroll opitch oyaw">
+    <link name="${name}">
+      <visual>
+        <geometry>
+          <mesh filename="package://motoman_description/meshes/sia5/visual/COLLADA/${name}.dae"/>
+        </geometry>
+      </visual>
+      <collision>
+        <geometry>
+          <mesh filename="package://motoman_description/meshes/sia5/collision/STL/${name}.stl"/>
+        </geometry>
+      </collision>
+      <inertial>
+		<origin xyz="${ox} ${oy} ${oz}" rpy="${oroll} ${opitch} ${oyaw}"/>
+        <mass value="${mass}"/>
+        <inertia ixx="${mass*((radius*radius)/4+(height*height)/12)}" ixy="0" ixz="0"
+				 iyy="${mass*((radius*radius)/4+(height*height)/12)}" iyz="0"
+				 izz="${(mass*radius*radius)/2}" />
+      </inertial>
+    </link>
+  </xacro:macro>
+  <xacro:macro name="link_box_v0" params="name mass width depth  height
+											ox oy oz oroll opitch oyaw">
+    <link name="${name}">
+      <visual>
+        <geometry>
+          <mesh filename="package://motoman_description/meshes/sia5/visual/COLLADA/${name}.dae"/>
+        </geometry>
+      </visual>
+      <collision>
+        <geometry>
+          <mesh filename="package://motoman_description/meshes/sia5/collision/STL/${name}.stl"/>
+        </geometry>
+      </collision>
+      <inertial>
+		<origin xyz="${ox} ${oy} ${oz}" rpy="${oroll} ${opitch} ${oyaw}"/>
+        <mass value="${mass}"/>
+        <inertia ixx="${(mass*(width*width+height*height))/3}" ixy="0" ixz="0"
+				 iyy="${(mass*(depth*depth+height*height))/3}" iyz="0"
+				 izz="${(mass*(depth*depth+width*width))/3}" />
+      </inertial>
+    </link>
+  </xacro:macro>
   <xacro:macro name="joint_v1" params="joint_name
 									   parent_name child_name

Commit message: [modify] link_box_v0の引数を変更
今まではwidth，depth，heightに，実際の大きさの半分の値を入れる必要があっ
たが、わかりづらいので，そのままの値を入れるように変更

File: robots/sia5/sia5.urdf.xacro (robot description, xacro)
@@ -45,5 +45,5 @@
   <link name="world"/>
   <xacro:link_box_v0 name="base_link" mass="${base_rate/sum_rate*sum_mass}"
-					 width="0.08325" depth="0.0988" height="0.07325"
+					 width="0.1665" depth="0.1976" height="0.1465"
 					 ox="-0.025918" oy="-0.000376" oz="0.076105" oroll="0" opitch="0" oyaw="0"/>
   <xacro:link_v1 name="link_s" mass="${s_rate/sum_rate*sum_mass}"

File: urdf/sia5/body.urdf.xacro (robot description, xacro)
@@ -63,7 +63,7 @@
 		<origin xyz="${ox} ${oy} ${oz}" rpy="${oroll} ${opitch} ${oyaw}"/>
         <mass value="${mass}"/>
-        <inertia ixx="${(mass*(width*width+height*height))/3}" ixy="0" ixz="0"
-				 iyy="${(mass*(depth*depth+height*height))/3}" iyz="0"
-				 izz="${(mass*(depth*depth+width*width))/3}" />
+        <inertia ixx="${(mass*((width/2)*(width/2)+(height/2)*(height/2)))/3}" ixy="0" ixz="0"
+				 iyy="${(mass*((depth/2)*(depth/2)+(height/2)*(height/2)))/3}" iyz="0"
+				 izz="${(mass*((depth/2)*(depth/2)+(width/2)*(width/2)))/3}" />
       </inertial>
     </link>
