Commit message: [modify] 全てに概形のイナーシャを適用した
適用したけど、まだあまりうまく行かない。
- 質量で調整する
- joint_lのコントローラゲインを調整する

というので対処すべきなのでは。。。？

File: robots/sia5/sia5.urdf.xacro (robot description, xacro)
@@ -10,12 +10,12 @@
   <property name="sum_mass" value="30.0" />
   <!-- about mass rate -->
-  <property name="base_rate" value="6.4" />
-  <property name="s_rate" value="6.1" />
-  <property name="l_rate" value="5.5" />
-  <property name="e_rate" value="4.0" />
-  <property name="u_rate" value="3.5"/>
-  <property name="r_rate" value="2.0" />
-  <property name="b_rate" value="1.5" />
-  <property name="t_rate" value="1.0" />
+  <property name="base_rate" value="8.5" />
+  <property name="s_rate" value="7.7" />
+  <property name="l_rate" value="7.0" />
+  <property name="e_rate" value="1.8" />
+  <property name="u_rate" value="1.7" />
+  <property name="r_rate" value="1.3" />
+  <property name="b_rate" value="1.2" />
+  <property name="t_rate" value="0.8" />
   <!-- Hard ware limits -->
   <!-- Range limits -->
@@ -47,32 +47,44 @@
 					 width="0.1665" depth="0.1976" height="0.1465"
 					 ox="-0.025918" oy="-0.000376" oz="0.076105" oroll="0" opitch="0" oyaw="0"/>
-  <xacro:link_v1 name="link_s" mass="${s_rate/sum_rate*sum_mass}"
-  				 ixx="0.0012143" ixy="0.0" ixz="0.0"
-				 iyy="0.0009784" iyz="0.0"
-				 izz="0.0010342"/>
-  <xacro:link_v1 name="link_l" mass="${l_rate/sum_rate*sum_mass}"
-  				 ixx="0.0008890" ixy="0.0" ixz="0.0"
-  				 iyy="0.0009864" iyz="0.0"
-				 izz="0.0008971"/>
-  <xacro:link_v1 name="link_e"  mass="${e_rate/sum_rate*sum_mass}"
-  				 ixx="0.0007581" ixy="0.0" ixz="0.0"
-  				 iyy="0.0007672" iyz="0.0"
-				 izz="0.0008762"/>
-  <xacro:link_v1 name="link_u" mass="${u_rate/sum_rate*sum_mass}"
-  				 ixx="0.0007594" ixy="0.0" ixz="0.0"
-  				 iyy="0.0007247" iyz="0.0"
-				 izz="0.0005782"/>
-  <xacro:link_v1 name="link_r" mass="${r_rate/sum_rate*sum_mass}"
-  				 ixx="0.0005783" ixy="0.0" ixz="0.0"
-  				 iyy="0.0005986" iyz="0.0"
-				 izz="0.0006781"/>
-  <xacro:link_v1 name="link_b" mass="${b_rate/sum_rate*sum_mass}"
-  				 ixx="0.0005374" ixy="0.0" ixz="0.0"
-  				 iyy="0.0004653" iyz="0.0"
-				 izz="0.0004592"/>
+  <xacro:link_cylinder_plus_box_v0 name="link_s"
+								   ox="0" oy="0" oz="0" oroll="0" opitch="0" oyaw="0"
+								   mass_cyl="${s_rate/sum_rate*sum_mass*0.2}"
+								   radius_cyl="0.066" height_cyl="0.031"
+								   mass_box="${s_rate/sum_rate*sum_mass*0.8}"
+								   width_box="0.0851" depth_box="0.1" height_box="0.1823"/>
+  <xacro:link_cylinder_plus_box_v0 name="link_l"
+								   ox="0" oy="-0.006" oz="0.15" oroll="${M_PI}" opitch="0" oyaw="0"
+								   mass_cyl="${l_rate/sum_rate*sum_mass*0.4}"
+								   radius_cyl="0.066" height_cyl="0.073"
+								   mass_box="${l_rate/sum_rate*sum_mass*0.6}"
+								   width_box="0.073" depth_box="0.1089" height_box="0.149"/>
+  <xacro:link_cylinder_plus_box_v0 name="link_e"
+								   ox="0" oy="0" oz="0" oroll="0" opitch="0" oyaw="${-M_PI/2}"
+								   mass_cyl="${e_rate/sum_rate*sum_mass*0.56}"
+								   radius_cyl="0.0685" height_cyl="0.0661"
+								   mass_box="${e_rate/sum_rate*sum_mass*0.44}"
+								   width_box="0.1234" depth_box="0.063" height_box="0.1176"/>
+  <xacro:link_cylinder_plus_box_v0 name="link_u"
+								   ox="0.008" oy="-0.06" oz="-0.131" oroll="${-M_PI}" opitch="${M_PI/2}" oyaw="0"
+								   mass_cyl="${u_rate/sum_rate*sum_mass*0.48}"
+								   radius_cyl="0.055" height_cyl="0.0698"
+								   mass_box="${u_rate/sum_rate*sum_mass*0.52}"
+								   width_box="0.13174" depth_box="0.068" height_box="0.104"/>
+  <xacro:link_cylinder_plus_box_v0 name="link_r"
+  								   ox="0" oy="0" oz="0" oroll="0" opitch="0" oyaw="${-M_PI/2}"
+  								   mass_cyl="${r_rate/sum_rate*sum_mass*0.25}"
+  								   radius_cyl="0.0525" height_cyl="0.038"
+  								   mass_box="${r_rate/sum_rate*sum_mass*0.75}"
+  								   width_box="0.0645" depth_box="0.084" height_box="0.1425"/>
+  <xacro:link_cylinder_plus_box_v0 name="link_b"
+  								   ox="0" oy="0.0045" oz="0.1365" oroll="${M_PI/2}" opitch="${-M_PI/2}" oyaw="0"
+  								   mass_cyl="${b_rate/sum_rate*sum_mass*0.55}"
+  								   radius_cyl="0.04" height_cyl="0.0948"
+  								   mass_box="${b_rate/sum_rate*sum_mass*0.45}"
+  								   width_box="0.0676" depth_box="0.076" height_box="0.0627"/>
   <xacro:link_cylinder_v0 name="link_t" mass="${t_rate/sum_rate*sum_mass}"
-					   radius="0.045" height="0.0115"
-					   ox="0.005406" oy="0.0" oz="-0.000191" oroll="0" opitch="0" oyaw="0"/>
- <link name="tool0"/>
+						  radius="0.045" height="0.0115"
+						  ox="0.005406" oy="0.0" oz="-0.000191" oroll="0" opitch="0" oyaw="0"/>
+  <link name="tool0"/>
   <!-- joint -->
   <joint name="world" type="fixed">
@@ -144,10 +156,10 @@
   				  ox="0.1365" oy="0" oz="-0.0045"
   				  roll="${-M_PI/2}" pitch="0" yaw="0"
-  				  ax="-1" ay="0" az="0"
-  				  el="7.35"
-  				  ll="${t_axis_lower_limit}" ul="${t_axis_upper_limit}"
-  				  vl="${t_axis_velocity_limit}"
-  				  skp="1" skv="1"
-  				  sll="${t_axis_lower_limit}" sul="${t_axis_upper_limit}"/>
+ax="-1" ay="0" az="0"
+el="7.35"
+ll="${t_axis_lower_limit}" ul="${t_axis_upper_limit}"
+vl="${t_axis_velocity_limit}"
+skp="1" skv="1"
+sll="${t_axis_lower_limit}" sul="${t_axis_upper_limit}"/>
   <joint name="joint_tool0" type="fixed">
     <origin rpy="0 0 0" xyz="0.0115 0 -0.040"/>

File: urdf/sia5/body.urdf.xacro (robot description, xacro)
@@ -26,5 +26,5 @@
   </xacro:macro>
   <xacro:macro name="link_cylinder_v0" params="name mass radius height
-											ox oy oz oroll opitch oyaw">
+											   ox oy oz oroll opitch oyaw">
     <link name="${name}">
       <visual>
@@ -48,5 +48,5 @@
   </xacro:macro>
   <xacro:macro name="link_box_v0" params="name mass width depth  height
-											ox oy oz oroll opitch oyaw">
+										  ox oy oz oroll opitch oyaw">
     <link name="${name}">
       <visual>
@@ -69,4 +69,28 @@
     </link>
   </xacro:macro>
+  <xacro:macro name="link_cylinder_plus_box_v0" params="name
+														ox oy oz oroll opitch oyaw
+														mass_cyl radius_cyl height_cyl
+														mass_box width_box depth_box height_box">
+    <link name="${name}">
+      <visual>
+        <geometry>
+          <mesh filename="package://motoman_description/meshes/sia5/visual/COLLADA/${name}.dae"/>
+        </geometry>
+      </visual>
+      <collision>
+        <geometry>
+          <mesh filename="package://motoman_description/meshes/sia5/collision/STL/${name}.stl"/>
+        </geometry>
+      </collision>
+      <inertial>
+		<origin xyz="${ox} ${oy} ${oz}" rpy="${oroll} ${opitch} ${oyaw}"/>
+        <mass value="${mass_cyl+mass_box}"/>
+        <inertia ixx="${mass_cyl*((radius_cyl*radius_cyl)/4+(height_cyl*height_cyl)/3)+mass_box/3*(width_box*width_box+height_box*height_box)+mass_box*(radius_cyl*radius_cyl-radius_cyl*width_box+height_cyl*height_cyl+height_cyl*height_box)}" ixy="0" ixz="0"
+				 iyy="${mass_cyl*((radius_cyl*radius_cyl)/4+(height_cyl*height_cyl)/12)+mass_box/3*(depth_box*depth_box+height_box*height_box)+mass_box*(radius_cyl*radius_cyl-radius_cyl*depth_box+height_cyl*height_cyl+height_cyl*height_box)}" iyz="0"
+				 izz="${(mass_cyl*radius_cyl*radius_cyl)/2+mass_box/3*(depth_box*depth_box+width_box*width_box)+mass_box*(2*radius_cyl*radius_cyl-radius_cyl*depth_box-radius_cyl*width_box)}" />
+      </inertial>
+    </link>
+  </xacro:macro>
   <xacro:macro name="joint_v1" params="joint_name
 									   parent_name child_name

Commit message: [add] テーブルを追加したxacroに変更
STLファイルをblenderで[cm]->[m]単位系にしたが、
出力フォーマットがよろしく無いらしい（ROSで読めない）ので、
今後STLファイルの変更が必要。
尚、STLファイルはcollisiont判定に使用している。

File: robots/sia5/sia5.urdf.xacro (robot description, xacro)
@@ -10,4 +10,5 @@
   <property name="sum_mass" value="30.0" />
   <!-- about mass rate -->
+  <property name="table_mass" value="40.0" />
   <property name="base_rate" value="8.5" />
   <property name="s_rate" value="7.7" />
@@ -44,4 +45,7 @@
   <!-- link -->
   <link name="world"/>
+  <xacro:link_box_v0 name="table_link" mass="${table_mass}"
+					 width="0.676" depth="1.116" height="0.53"
+					 ox="0.20" oy="0" oz="0.265" oroll="0" opitch="0" oyaw="0"/>
   <xacro:link_box_v0 name="base_link" mass="${base_rate/sum_rate*sum_mass}"
 					 width="0.1665" depth="0.1976" height="0.1465"
@@ -91,5 +95,10 @@
   <joint name="world" type="fixed">
     <parent link="world"/>
-    <child link="base_link"/>
+    <child link="table_link"/>
+	<origin xyz="0 0 0.53"/>
+  </joint>
+  <joint name="joint_base" type="fixed">
+	<parent link="table_link"/>
+	<child link="base_link"/>
   </joint>
   <xacro:joint_v1 joint_name="joint_s"
