Commit message: [Fix] 小さな変更．xacroやlaunchのインデント変更，余計な文字を取り除いたりしました．

File: robots/sia5/sia5.urdf.xacro (robot description, xacro)
@@ -4,5 +4,5 @@
   <xacro:include filename="$(find motoman_description)/robots/sia5/sia5_basic.urdf.xacro" />
   <xacro:add_world>
-	<origin xyz="0 0 0" rpy="0 0 0"/>
+    <origin xyz="0 0 0" rpy="0 0 0"/>
   </xacro:add_world>
 </robot>

File: robots/sia5/sia5_basic.urdf.xacro (robot description, xacro)
@@ -26,5 +26,5 @@
   <xacro:property name="l_axis_lower_limit" value="-${l_axis_upper_limit}"/>
   <xacro:property name="e_axis_upper_limit" value="${170.0*M_PI/180.0}"/>
-  pp  <xacro:property name="e_axis_lower_limit" value="-${e_axis_upper_limit}"/>
+  <xacro:property name="e_axis_lower_limit" value="-${e_axis_upper_limit}"/>
   <xacro:property name="u_axis_upper_limit" value="${115.0*M_PI/180.0}"/>
   <xacro:property name="u_axis_lower_limit" value="${-90.0*M_PI/180.0}"/>
@@ -45,127 +45,127 @@
   <!-- Add macro -->
   <xacro:macro name="add_world" params="*origin">
-	<link name="world"/>
-	<joint name="world" type="fixed">
-	  <insert_block name="origin"/>
-	  <parent link="world"/>
-	  <child link="base_link"/>
-	</joint>
+    <link name="world"/>
+    <joint name="world" type="fixed">
+      <insert_block name="origin"/>
+      <parent link="world"/>
+      <child link="base_link"/>
+    </joint>
   </xacro:macro>
   <!-- link -->
   <xacro:link_box_v0 name="base_link" mass="${base_rate/sum_rate*sum_mass}"
-					 width="0.1665" depth="0.1976" height="0.1465"
-					 ox="-0.025918" oy="-0.000376" oz="0.076105" oroll="0" opitch="0" oyaw="0"/>
+                     width="0.1665" depth="0.1976" height="0.1465"
+                     ox="-0.025918" oy="-0.000376" oz="0.076105" oroll="0" opitch="0" oyaw="0"/>
   <xacro:link_cylinder_plus_box_v0 name="link_s"
-								   ox="0" oy="0" oz="0" oroll="0" opitch="0" oyaw="0"
-								   mass_cyl="${s_rate/sum_rate*sum_mass*0.2}"
-								   radius_cyl="0.066" height_cyl="0.031"
-								   mass_box="${s_rate/sum_rate*sum_mass*0.8}"
-								   width_box="0.0851" depth_box="0.1" height_box="0.1823"/>
+                                   ox="0" oy="0" oz="0" oroll="0" opitch="0" oyaw="0"
+                                   mass_cyl="${s_rate/sum_rate*sum_mass*0.2}"
+                                   radius_cyl="0.066" height_cyl="0.031"
+                                   mass_box="${s_rate/sum_rate*sum_mass*0.8}"
+                                   width_box="0.0851" depth_box="0.1" height_box="0.1823"/>
   <xacro:link_cylinder_plus_box_v0 name="link_l"
-								   ox="0" oy="-0.006" oz="0.15" oroll="${M_PI}" opitch="0" oyaw="0"
-								   mass_cyl="${l_rate/sum_rate*sum_mass*0.4}"
-								   radius_cyl="0.066" height_cyl="0.073"
-								   mass_box="${l_rate/sum_rate*sum_mass*0.6}"
-								   width_box="0.073" depth_box="0.1089" height_box="0.149"/>
+                                   ox="0" oy="-0.006" oz="0.15" oroll="${M_PI}" opitch="0" oyaw="0"
+                                   mass_cyl="${l_rate/sum_rate*sum_mass*0.4}"
+                                   radius_cyl="0.066" height_cyl="0.073"
+                                   mass_box="${l_rate/sum_rate*sum_mass*0.6}"
+                                   width_box="0.073" depth_box="0.1089" height_box="0.149"/>
   <xacro:link_cylinder_plus_box_v0 name="link_e"
-								   ox="0" oy="0" oz="0" oroll="0" opitch="0" oyaw="${-M_PI/2}"
-								   mass_cyl="${e_rate/sum_rate*sum_mass*0.56}"
-								   radius_cyl="0.0685" height_cyl="0.0661"
-								   mass_box="${e_rate/sum_rate*sum_mass*0.44}"
-								   width_box="0.1234" depth_box="0.063" height_box="0.1176"/>
+                                   ox="0" oy="0" oz="0" oroll="0" opitch="0" oyaw="${-M_PI/2}"
+                                   mass_cyl="${e_rate/sum_rate*sum_mass*0.56}"
+                                   radius_cyl="0.0685" height_cyl="0.0661"
+                                   mass_box="${e_rate/sum_rate*sum_mass*0.44}"
+                                   width_box="0.1234" depth_box="0.063" height_box="0.1176"/>
   <xacro:link_cylinder_plus_box_v0 name="link_u"
-								   ox="0.008" oy="-0.06" oz="-0.131" oroll="${-M_PI}" opitch="${M_PI/2}" oyaw="0"
-								   mass_cyl="${u_rate/sum_rate*sum_mass*0.48}"
-								   radius_cyl="0.055" height_cyl="0.0698"
-								   mass_box="${u_rate/sum_rate*sum_mass*0.52}"
-								   width_box="0.13174" depth_box="0.068" height_box="0.104"/>
+                                   ox="0.008" oy="-0.06" oz="-0.131" oroll="${-M_PI}" opitch="${M_PI/2}" oyaw="0"
+                                   mass_cyl="${u_rate/sum_rate*sum_mass*0.48}"
+                                   radius_cyl="0.055" height_cyl="0.0698"
+                                   mass_box="${u_rate/sum_rate*sum_mass*0.52}"
+                                   width_box="0.13174" depth_box="0.068" height_box="0.104"/>
   <xacro:link_cylinder_plus_box_v0 name="link_r"
-  								   ox="0" oy="0" oz="0" oroll="0" opitch="0" oyaw="${-M_PI/2}"
-  								   mass_cyl="${r_rate/sum_rate*sum_mass*0.25}"
-  								   radius_cyl="0.0525" height_cyl="0.038"
-  								   mass_box="${r_rate/sum_rate*sum_mass*0.75}"
-  								   width_box="0.0645" depth_box="0.084" height_box="0.1425"/>
+                                     ox="0" oy="0" oz="0" oroll="0" opitch="0" oyaw="${-M_PI/2}"
+                                     mass_cyl="${r_rate/sum_rate*sum_mass*0.25}"
+                                     radius_cyl="0.0525" height_cyl="0.038"
+                                     mass_box="${r_rate/sum_rate*sum_mass*0.75}"
+                                     width_box="0.0645" depth_box="0.084" height_box="0.1425"/>
   <xacro:link_cylinder_plus_box_v0 name="link_b"
-  								   ox="0" oy="0.0045" oz="0.1365" oroll="${M_PI/2}" opitch="${-M_PI/2}" oyaw="0"
-  								   mass_cyl="${b_rate/sum_rate*sum_mass*0.55}"
-  								   radius_cyl="0.04" height_cyl="0.0948"
-  								   mass_box="${b_rate/sum_rate*sum_mass*0.45}"
-  								   width_box="0.0676" depth_box="0.076" height_box="0.0627"/>
+                                     ox="0" oy="0.0045" oz="0.1365" oroll="${M_PI/2}" opitch="${-M_PI/2}" oyaw="0"
+                                     mass_cyl="${b_rate/sum_rate*sum_mass*0.55}"
+                                     radius_cyl="0.04" height_cyl="0.0948"
+                                     mass_box="${b_rate/sum_rate*sum_mass*0.45}"
+                                     width_box="0.0676" depth_box="0.076" height_box="0.0627"/>
   <xacro:link_v1 name="link_t" mass="${t_rate/sum_rate*sum_mass}"
-  				 ixx="0.003" ixy="0" ixz="0"
-  				 iyy="0.003" iyz="0"
-  				 izz="0.001"/>
+                   ixx="0.003" ixy="0" ixz="0"
+                   iyy="0.003" iyz="0"
+                   izz="0.001"/>
   <link name="tool0"/>
   <!-- joint -->
   <xacro:joint_v1 joint_name="joint_s"
-  				  parent_name="base_link" child_name="link_s"
-				  ox="0" oy="0" oz="0.1765"
-				  roll="0" pitch="0" yaw="0"
-  				  ax="0" ay="0" az="1"
-  				  el="30.0"
-  				  ll="${s_axis_lower_limit}" ul="${s_axis_upper_limit}"
-  				  vl="${s_axis_velocity_limit}"
-  				  skp="1" skv="1"
-  				  sll="${s_axis_lower_limit}" sul="${s_axis_upper_limit}"/>
+                  parent_name="base_link" child_name="link_s"
+                  ox="0" oy="0" oz="0.1765"
+                  roll="0" pitch="0" yaw="0"
+                  ax="0" ay="0" az="1"
+                  el="30.0"
+                  ll="${s_axis_lower_limit}" ul="${s_axis_upper_limit}"
+                  vl="${s_axis_velocity_limit}"
+                  skp="1" skv="1"
+                  sll="${s_axis_lower_limit}" sul="${s_axis_upper_limit}"/>
   <xacro:joint_v1 joint_name="joint_l"
-  				  parent_name="link_s" child_name="link_l"
-  				  ox="0" oy="0.006" oz="0.136"
-  				  roll="0" pitch="0" yaw="0"
-  				  ax="0" ay="1" az="0"
-  				  el="30.0"
-  				  ll="${l_axis_lower_limit}" ul="${l_axis_upper_limit}"
-  				  vl="${l_axis_velocity_limit}"
-  				  skp="1" skv="1"
-  				  sll="${l_axis_lower_limit}" sul="${l_axis_upper_limit}"/>
+                  parent_name="link_s" child_name="link_l"
+                  ox="0" oy="0.006" oz="0.136"
+                  roll="0" pitch="0" yaw="0"
+                  ax="0" ay="1" az="0"
+                  el="30.0"
+                  ll="${l_axis_lower_limit}" ul="${l_axis_upper_limit}"
+                  vl="${l_axis_velocity_limit}"
+                  skp="1" skv="1"
+                  sll="${l_axis_lower_limit}" sul="${l_axis_upper_limit}"/>
   <xacro:joint_v1 joint_name="joint_e"
-  				  parent_name="link_l" child_name="link_e"
-  				  ox="0" oy="-0.006" oz="0.15"
-  				  roll="0" pitch="0" yaw="0"
-  				  ax="0" ay="0" az="1"
-  				  el="30.0"
-  				  ll="${e_axis_lower_limit}" ul="${e_axis_upper_limit}"
-  				  vl="${e_axis_velocity_limit}"
-  				  skp="1" skv="1"
-  				  sll="${e_axis_lower_limit}" sul="${e_axis_upper_limit}"/>
+                  parent_name="link_l" child_name="link_e"
+                  ox="0" oy="-0.006" oz="0.15"
+                  roll="0" pitch="0" yaw="0"
+                  ax="0" ay="0" az="1"
+                  el="30.0"
+                  ll="${e_axis_lower_limit}" ul="${e_axis_upper_limit}"
+                  vl="${e_axis_velocity_limit}"
+                  skp="1" skv="1"
+                  sll="${e_axis_lower_limit}" sul="${e_axis_upper_limit}"/>
   <xacro:joint_v1 joint_name="joint_u"
-  				  parent_name="link_e" child_name="link_u"
-  				  ox="0.085" oy="-0.00826931" oz="0.12275299"
-  				  roll="${M_PI/2.0}" pitch="0" yaw="0"
-  				  ax="0" ay="0" az="1"
-  				  el="30.0"
-  				  ll="${u_axis_lower_limit}" ul="${u_axis_upper_limit}"
-  				  vl="${u_axis_velocity_limit}"
-  				  skp="1" skv="1"
-  				  sll="${u_axis_lower_limit}" sul="${u_axis_upper_limit}"/>
+                  parent_name="link_e" child_name="link_u"
+                  ox="0.085" oy="-0.00826931" oz="0.12275299"
+                  roll="${M_PI/2.0}" pitch="0" yaw="0"
+                  ax="0" ay="0" az="1"
+                  el="30.0"
+                  ll="${u_axis_lower_limit}" ul="${u_axis_upper_limit}"
+                  vl="${u_axis_velocity_limit}"
+                  skp="1" skv="1"
+                  sll="${u_axis_lower_limit}" sul="${u_axis_upper_limit}"/>
   <xacro:joint_v1 joint_name="joint_r"
-  				  parent_name="link_u" child_name="link_r"
-  				  ox="0.131" oy="0.06" oz="-0.008"
-  				  roll="0" pitch="${M_PI/2}" yaw="0"
-  				  ax="0" ay="0" az="-1"
-  				  el="14.7"
-  				  ll="${r_axis_lower_limit}" ul="${r_axis_upper_limit}"
-  				  vl="${r_axis_velocity_limit}"
-  				  skp="1" skv="1"
-  				  sll="${r_axis_lower_limit}" sul="${r_axis_upper_limit}"/>
+                  parent_name="link_u" child_name="link_r"
+                  ox="0.131" oy="0.06" oz="-0.008"
+                  roll="0" pitch="${M_PI/2}" yaw="0"
+                  ax="0" ay="0" az="-1"
+                  el="14.7"
+                  ll="${r_axis_lower_limit}" ul="${r_axis_upper_limit}"
+                  vl="${r_axis_velocity_limit}"
+                  skp="1" skv="1"
+                  sll="${r_axis_lower_limit}" sul="${r_axis_upper_limit}"/>
   <xacro:joint_v1 joint_name="joint_b"
-  				  parent_name="link_r" child_name="link_b"
-  				  ox="-0.0045" oy="0" oz="0.139"
-  				  roll="0" pitch="${-M_PI/2}" yaw="0"
-  				  ax="0" ay="0" az="1"
-  				  el="14.7"
-  				  ll="${b_axis_lower_limit}" ul="${b_axis_upper_limit}"
-  				  vl="${b_axis_velocity_limit}"
-  				  skp="1" skv="1"
-  				  sll="${b_axis_lower_limit}" sul="${b_axis_upper_limit}"/>
+                  parent_name="link_r" child_name="link_b"
+                  ox="-0.0045" oy="0" oz="0.139"
+                  roll="0" pitch="${-M_PI/2}" yaw="0"
+                  ax="0" ay="0" az="1"
+                  el="14.7"
+                  ll="${b_axis_lower_limit}" ul="${b_axis_upper_limit}"
+                  vl="${b_axis_velocity_limit}"
+                  skp="1" skv="1"
+                  sll="${b_axis_lower_limit}" sul="${b_axis_upper_limit}"/>
   <xacro:joint_v1 joint_name="joint_t"
-  				  parent_name="link_b" child_name="link_t"
-  				  ox="0.1365" oy="0" oz="-0.0045"
-  				  roll="${-M_PI/2}" pitch="0" yaw="0"
-				  ax="-1" ay="0" az="0"
-				  el="7.35"
-				  ll="${t_axis_lower_limit}" ul="${t_axis_upper_limit}"
-				  vl="${t_axis_velocity_limit}"
-				  skp="1" skv="1"
-				  sll="${t_axis_lower_limit}" sul="${t_axis_upper_limit}"/>
+                  parent_name="link_b" child_name="link_t"
+                  ox="0.1365" oy="0" oz="-0.0045"
+                  roll="${-M_PI/2}" pitch="0" yaw="0"
+                  ax="-1" ay="0" az="0"
+                  el="7.35"
+                  ll="${t_axis_lower_limit}" ul="${t_axis_upper_limit}"
+                  vl="${t_axis_velocity_limit}"
+                  skp="1" skv="1"
+                  sll="${t_axis_lower_limit}" sul="${t_axis_upper_limit}"/>
   <joint name="joint_tool0" type="fixed">
     <origin rpy="0 0 0" xyz="0.0115 0 0"/>
@@ -175,24 +175,24 @@
   <!-- transmission -->
   <xacro:simple_jp_trans_v0 name="transmission_s"
-  							joint_name="joint_s" actuator_name="motor_s"
-  							reduction="300"/>
+                            joint_name="joint_s" actuator_name="motor_s"
+                            reduction="300"/>
   <xacro:simple_jp_trans_v0 name="transmission_l"
-  							joint_name="joint_l" actuator_name="motor_l"
-  							reduction="300"/>
+                            joint_name="joint_l" actuator_name="motor_l"
+                            reduction="300"/>
   <xacro:simple_jp_trans_v0 name="transmission_e"
-  							joint_name="joint_e" actuator_name="motor_e"
-  							reduction="100"/>
+                            joint_name="joint_e" actuator_name="motor_e"
+                            reduction="100"/>
   <xacro:simple_jp_trans_v0 name="transmission_u"
-  							joint_name="joint_u" actuator_name="motor_u"
-  							reduction="50"/>
+                            joint_name="joint_u" actuator_name="motor_u"
+                            reduction="50"/>
   <xacro:simple_jp_trans_v0 name="transmission_r"
-  							joint_name="joint_r" actuator_name="motor_r"
-  							reduction="30"/>
+                            joint_name="joint_r" actuator_name="motor_r"
+                            reduction="30"/>
   <xacro:simple_jp_trans_v0 name="transmission_b"
-  							joint_name="joint_b" actuator_name="motor_b"
-  							reduction="30"/>
+                            joint_name="joint_b" actuator_name="motor_b"
+                            reduction="30"/>
   <xacro:simple_jp_trans_v0 name="transmission_t"
-  							joint_name="joint_t" actuator_name="motor_t"
-  							reduction="10"/>
+                            joint_name="joint_t" actuator_name="motor_t"
+                            reduction="10"/>
   <!-- gazebo -->
   <gazebo>

File: robots/sia5/sia5_gazebo_nishida_lab.urdf.xacro (robot description, xacro)
@@ -21,7 +21,7 @@
   </joint>
   <joint name="joint_rgb_kinect2" type="fixed">
-	<origin rpy="${M_PI/2} ${M_PI} ${M_PI/2}"/>
-	<parent link="kinect2_link"/>
-	<child link="kinect2_rgb_optical_frame"/>
+    <origin rpy="${M_PI/2} ${M_PI} ${M_PI/2}"/>
+    <parent link="kinect2_link"/>
+    <child link="kinect2_rgb_optical_frame"/>
   </joint>
   <!-- Gazebo -->
@@ -30,7 +30,7 @@
    <!-- Link -->
   <xacro:tool_link_cylinder_v0 name="gripper_link" mass="1.0"
-  							   radius="0.0965" height="0.61445"
-  							   ox="0" oy="0" oz="0"
-  							   oroll="0" opitch="0" oyaw="0"/>
+                               radius="0.0965" height="0.61445"
+                               ox="0" oy="0" oz="0"
+                               oroll="0" opitch="0" oyaw="0"/>
   <link name="balloon"/>
   <!-- <xacro:tool_link_no_collision_v0 name="balloon" mass="0.3" -->

File: robots/sia5/sia5_with_jamming.urdf.xacro (robot description, xacro)
@@ -7,7 +7,7 @@
   <!-- Link -->
   <xacro:tool_link_cylinder_v0 name="gripper_link" mass="1.0"
-  							   radius="0.0965" height="0.61445"
-  							   ox="0" oy="0" oz="0"
-  							   oroll="0" opitch="0" oyaw="0"/>
+                               radius="0.0965" height="0.61445"
+                               ox="0" oy="0" oz="0"
+                               oroll="0" opitch="0" oyaw="0"/>
   <link name="balloon"/>
   <!-- <xacro:tool_link_no_collision_v0 name="balloon" mass="0.3" -->

File: robots/sia5/sia5_with_jamming_and_kinectv2.urdf.xacro (robot description, xacro)
@@ -16,7 +16,7 @@
   </joint>
   <joint name="joint_rgb_kinect2" type="fixed">
-	<origin rpy="${M_PI/2} ${M_PI} ${M_PI/2}"/>
-	<parent link="kinect2_link"/>
-	<child link="kinect2_rgb_optical_frame"/>
+    <origin rpy="${M_PI/2} ${M_PI} ${M_PI/2}"/>
+    <parent link="kinect2_link"/>
+    <child link="kinect2_rgb_optical_frame"/>
   </joint>
   <!-- Gazebo -->

File: robots/sia5/sia5_with_kinectv2.urdf.xacro (robot description, xacro)
@@ -16,7 +16,7 @@
   </joint>
   <joint name="joint_rgb_kinect2" type="fixed">
-	<origin rpy="${M_PI/2} ${M_PI} ${M_PI/2}"/>
-	<parent link="kinect2_link"/>
-	<child link="kinect2_rgb_optical_frame"/>
+    <origin rpy="${M_PI/2} ${M_PI} ${M_PI/2}"/>
+    <parent link="kinect2_link"/>
+    <child link="kinect2_rgb_optical_frame"/>
   </joint>
   <!-- Gazebo -->

File: urdf/sia5/body.gazebo.xacro (robot description, xacro)
@@ -2,9 +2,9 @@
 <robot xmlns:xacro="http://ros.org/wiki/xacro">
   <xacro:macro name="gazebo_link_v1" params="name">
-	<gazebo reference="${name}">
-	  <mu1>0.2</mu1>
-	  <mu2>0.2</mu2>
-	  <selfCollide>true</selfCollide>
-	</gazebo>
+    <gazebo reference="${name}">
+      <mu1>0.2</mu1>
+      <mu2>0.2</mu2>
+      <selfCollide>true</selfCollide>
+    </gazebo>
   </xacro:macro>
 </robot>

File: urdf/sia5/body.transmission.xacro (robot description, xacro)
@@ -2,16 +2,16 @@
 <robot xmlns:xacro="http://ros.org/wiki/xacro">
   <xacro:macro name="simple_jp_trans_v0" params="name
-												 joint_name actuator_name
-												 reduction">
-	<transmission name="${name}">
+                                                 joint_name actuator_name
+                                                 reduction">
+    <transmission name="${name}">
       <type>transmission_interface/SimpleTransmission</type>
       <joint name="${joint_name}">
-		<hardwareInterface>PositionJointInterface</hardwareInterface>
+      <hardwareInterface>PositionJointInterface</hardwareInterface>
       </joint>
       <actuator name="${actuator_name}">
-		<hardwareInterface>PositionJointInterface</hardwareInterface>
-		<mechanicalReduction>${reduction}</mechanicalReduction>
+      <hardwareInterface>PositionJointInterface</hardwareInterface>
+      <mechanicalReduction>${reduction}</mechanicalReduction>
       </actuator>
-	</transmission>
+    </transmission>
   </xacro:macro>
 </robot>

File: urdf/sia5/body.urdf.xacro (robot description, xacro)
@@ -1,8 +1,8 @@
-<?xml version="1.0"?>
+ <?xml version="1.0"?>
 <robot xmlns:xacro="http://ros.org/wiki/xacro">
   <property name="sum_rate" value="${base_rate + s_rate
-								   + l_rate + e_rate
-								   + u_rate + r_rate
-								   + b_rate + t_rate}" />
+                                      + l_rate + e_rate
+                                      + u_rate + r_rate
+                                      + b_rate + t_rate}" />
   <xacro:macro name="link_v1" params="name mass
                                       ixx ixy ixz
@@ -26,5 +26,5 @@
   </xacro:macro>
   <xacro:macro name="link_cylinder_v0" params="name mass radius height
-											   ox oy oz oroll opitch oyaw">
+                                               ox oy oz oroll opitch oyaw">
     <link name="${name}">
       <visual>
@@ -48,5 +48,5 @@
   </xacro:macro>
   <xacro:macro name="link_box_v0" params="name mass width depth  height
-										  ox oy oz oroll opitch oyaw">
+                                          ox oy oz oroll opitch oyaw">
     <link name="${name}">
       <visual>
@@ -70,5 +70,5 @@
   </xacro:macro>
   <xacro:macro name="link_box_v1" params="name mass width depth height
-										  ox oy oz oroll opitch oyaw">
+                                          ox oy oz oroll opitch oyaw">
     <link name="${name}">
       <visual>
@@ -93,7 +93,7 @@
   </xacro:macro>
   <xacro:macro name="link_cylinder_plus_box_v0" params="name
-														ox oy oz oroll opitch oyaw
-														mass_cyl radius_cyl height_cyl
-														mass_box width_box depth_box height_box">
+                                                        ox oy oz oroll opitch oyaw
+                                                        mass_cyl radius_cyl height_cyl
+                                                        mass_box width_box depth_box height_box">
     <link name="${name}">
       <visual>
@@ -111,14 +111,14 @@
         <mass value="${mass_cyl+mass_box}"/>
         <inertia ixx="${mass_cyl*((radius_cyl*radius_cyl)/4+(height_cyl*height_cyl)/3)+mass_box/3*(width_box*width_box+height_box*height_box)+mass_box*(radius_cyl*radius_cyl-radius_cyl*width_box+height_cyl*height_cyl+height_cyl*height_box)}" ixy="0" ixz="0"
-				 iyy="${mass_cyl*((radius_cyl*radius_cyl)/4+(height_cyl*height_cyl)/12)+mass_box/3*(depth_box*depth_box+height_box*height_box)+mass_box*(radius_cyl*radius_cyl-radius_cyl*depth_box+height_cyl*height_cyl+height_cyl*height_box)}" iyz="0"
-				 izz="${(mass_cyl*radius_cyl*radius_cyl)/2+mass_box/3*(depth_box*depth_box+width_box*width_box)+mass_box*(2*radius_cyl*radius_cyl-radius_cyl*depth_box-radius_cyl*width_box)}" />
+                 iyy="${mass_cyl*((radius_cyl*radius_cyl)/4+(height_cyl*height_cyl)/12)+mass_box/3*(depth_box*depth_box+height_box*height_box)+mass_box*(radius_cyl*radius_cyl-radius_cyl*depth_box+height_cyl*height_cyl+height_cyl*height_box)}" iyz="0"
+                 izz="${(mass_cyl*radius_cyl*radius_cyl)/2+mass_box/3*(depth_box*depth_box+width_box*width_box)+mass_box*(2*radius_cyl*radius_cyl-radius_cyl*depth_box-radius_cyl*width_box)}" />
       </inertial>
     </link>
   </xacro:macro>
   <xacro:macro name="joint_v1" params="joint_name
-									   parent_name child_name
+                                       parent_name child_name
                                        ox oy oz roll pitch yaw ax ay az
-									   el ll ul vl
-									   skp skv sll sul">
+                                       el ll ul vl
+                                       skp skv sll sul">
     <joint name="${joint_name}" type="revolute">
       <origin xyz="${ox} ${oy} ${oz}" rpy="${roll} ${pitch} ${yaw}"/>
@@ -126,5 +126,5 @@
       <child link="${child_name}"/>
       <axis xyz="${ax} ${ay} ${az}"/>
-	  <dynamics damping="0.7" friction="0.7"/>
+      <dynamics damping="0.7" friction="0.7"/>
       <limit effort="${el}" lower="${ll}" upper="${ul}" velocity="${vl}"/>
     </joint>
