Commit message: [Fix] 小さな変更．xacroやlaunchのインデント変更，余計な文字を取り除いたりしました．

File: urdf/tool/jamming.gazebo.xacro (robot description, xacro)
@@ -2,10 +2,10 @@
 <robot xmlns:xacro="http://ros.org/wiki/xacro">
   <xacro:macro name="gazebo_tool_link_v0" params="name color">
-	<gazebo reference="${name}">
-	  <mu1>0.2</mu1>
-	  <mu2>0.2</mu2>
-	  <selfCollide>true</selfCollide>
-	  <material>Gazebo/${color}</material>
-	</gazebo>
+    <gazebo reference="${name}">
+      <mu1>0.2</mu1>
+      <mu2>0.2</mu2>
+      <selfCollide>true</selfCollide>
+      <material>Gazebo/${color}</material>
+    </gazebo>
   </xacro:macro>
 </robot>

File: urdf/tool/jamming.urdf.xacro (robot description, xacro)
@@ -2,9 +2,9 @@
 <robot xmlns:xacro="http://ros.org/wiki/xacro">
   <xacro:macro name="tool_link_v0" params="name mass
-										   ixx ixy ixz
-										   iyy iyz izz">
+                                           ixx ixy ixz
+                                           iyy iyz izz">
     <link name="${name}">
       <visual>
-		<material name="blue"/>
+        <material name="blue"/>
         <geometry>
           <mesh filename="package://motoman_description/meshes/tool/visual/COLLADA/${name}.stl"/>
@@ -23,6 +23,6 @@
   </xacro:macro>
   <xacro:macro name="tool_link_no_collision_v0" params="name mass
-										   ixx ixy ixz
-										   iyy iyz izz">
+                                                        ixx ixy ixz
+                                                        iyy iyz izz">
     <link name="${name}">
       <visual>
@@ -39,8 +39,8 @@
   </xacro:macro>
   <xacro:macro name="tool_link_cylinder_v0" params="name mass radius height
-													ox oy oz oroll opitch oyaw">
+                                                    ox oy oz oroll opitch oyaw">
     <link name="${name}">
       <visual>
-		<material name="blue"/>
+        <material name="blue"/>
         <geometry>
           <mesh filename="package://motoman_description/meshes/tool/visual/COLLADA/${name}.stl"/>
@@ -53,9 +53,9 @@
       </collision>
       <inertial>
-		<origin xyz="${ox} ${oy} ${oz}" rpy="${oroll} ${opitch} ${oyaw}"/>
+        <origin xyz="${ox} ${oy} ${oz}" rpy="${oroll} ${opitch} ${oyaw}"/>
         <mass value="${mass}"/>
         <inertia ixx="${mass*((radius*radius)/4+(height*height)/12)}" ixy="0" ixz="0"
-				 iyy="${mass*((radius*radius)/4+(height*height)/12)}" iyz="0"
-				 izz="${(mass*radius*radius)/2}" />
+                 iyy="${mass*((radius*radius)/4+(height*height)/12)}" iyz="0"
+                 izz="${(mass*radius*radius)/2}" />
       </inertial>
     </link>
