Commit message: [modify] デモ用にlimit角度を変更

File: robots/sia5/sia5_basic.urdf.xacro (robot description, xacro)
@@ -21,26 +21,26 @@
   <!-- Hard ware limits -->
   <!-- Range limits -->
-  <xacro:property name="s_axis_upper_limit" value="${179.99999*M_PI/180.0}"/>
+  <xacro:property name="s_axis_upper_limit" value="${179.99999*M_PI/180.0*0.95}"/>
   <xacro:property name="s_axis_lower_limit" value="-${s_axis_upper_limit}"/>
-  <xacro:property name="l_axis_upper_limit" value="${110.0*M_PI/180.0}"/>
+  <xacro:property name="l_axis_upper_limit" value="${110.0*M_PI/180.0*0.95}"/>
   <xacro:property name="l_axis_lower_limit" value="-${l_axis_upper_limit}"/>
-  <xacro:property name="e_axis_upper_limit" value="${170.0*M_PI/180.0}"/>
+  <xacro:property name="e_axis_upper_limit" value="${170.0*M_PI/180.0*0.95}"/>
   pp  <xacro:property name="e_axis_lower_limit" value="-${e_axis_upper_limit}"/>
-  <xacro:property name="u_axis_upper_limit" value="${115.0*M_PI/180.0}"/>
-  <xacro:property name="u_axis_lower_limit" value="${-90.0*M_PI/180.0}"/>
-  <xacro:property name="r_axis_upper_limit" value="${179.99999*M_PI/180.0}"/>
+  <xacro:property name="u_axis_upper_limit" value="${115.0*M_PI/180.0*0.95}"/>
+  <xacro:property name="u_axis_lower_limit" value="${-90.0*M_PI/180.0*0.95}"/>
+  <xacro:property name="r_axis_upper_limit" value="${179.99999*M_PI/180.0*0.95}"/>
   <xacro:property name="r_axis_lower_limit" value="-${r_axis_upper_limit}"/>
-  <xacro:property name="b_axis_upper_limit" value="${110.0*M_PI/180.0}"/>
+  <xacro:property name="b_axis_upper_limit" value="${110.0*M_PI/180.0*0.95}"/>
   <xacro:property name="b_axis_lower_limit" value="-${b_axis_upper_limit}"/>
-  <xacro:property name="t_axis_upper_limit" value="${179.99999*M_PI/180.0}"/>
+  <xacro:property name="t_axis_upper_limit" value="${179.99999*M_PI/180.0*0.95}"/>
   <xacro:property name="t_axis_lower_limit" value="-${t_axis_upper_limit}"/>
   <!-- Velocity limits -->
-  <xacro:property name="s_axis_velocity_limit" value="${200.0*M_PI/180.0}"/>
-  <xacro:property name="l_axis_velocity_limit" value="${200.0*M_PI/180.0}"/>
-  <xacro:property name="e_axis_velocity_limit" value="${200.0*M_PI/180.0}"/>
-  <xacro:property name="u_axis_velocity_limit" value="${200.0*M_PI/180.0}"/>
-  <xacro:property name="r_axis_velocity_limit" value="${200.0*M_PI/180.0}"/>
-  <xacro:property name="b_axis_velocity_limit" value="${230.0*M_PI/180.0}"/>
-  <xacro:property name="t_axis_velocity_limit" value="${350.0*M_PI/180.0}"/>
+  <xacro:property name="s_axis_velocity_limit" value="${200.0*M_PI/180.0*0.95}"/>
+  <xacro:property name="l_axis_velocity_limit" value="${200.0*M_PI/180.0*0.95}"/>
+  <xacro:property name="e_axis_velocity_limit" value="${200.0*M_PI/180.0*0.95}"/>
+  <xacro:property name="u_axis_velocity_limit" value="${200.0*M_PI/180.0*0.95}"/>
+  <xacro:property name="r_axis_velocity_limit" value="${200.0*M_PI/180.0*0.95}"/>
+  <xacro:property name="b_axis_velocity_limit" value="${230.0*M_PI/180.0*0.95}"/>
+  <xacro:property name="t_axis_velocity_limit" value="${350.0*M_PI/180.0*0.95}"/>
   <!-- Add macro -->
   <xacro:macro name="add_world" params="*origin">

File: robots/sia5/sia5_with_jamming_and_kinectv2.urdf.xacro (robot description, xacro)
@@ -11,8 +11,9 @@
   <!-- Joint -->
   <joint name="joint_kinect2" type="fixed">
-    <origin rpy="0 ${10*M_PI/180} ${M_PI}" xyz="1.02024 0.30 0.3595"/>
+	<origin rpy="0 ${29*M_PI/180} ${114/180*M_PI}" xyz="0.885 -0.78 0.75"/>
     <parent link="base_link"/>
     <child link="kinect2_link"/>
   </joint>
+  <!-- <origin rpy="0 ${10*M_PI/180} ${M_PI}" xyz="1.02024 0.30 0.3595"/> -->
   <joint name="joint_rgb_kinect2" type="fixed">
 	<origin rpy="${M_PI/2} ${M_PI} ${M_PI/2}"/>
@@ -21,4 +22,4 @@
   </joint>
   <!-- Gazebo -->
-  <xacro:kinect_gazebo suffix="" name="kinect2"/>
+  <xacro:kinect_gazebo name="kinect2"/>
 </robot>
