Commit message: [modify] kinectの位置を実機に近づけるように変更

File: robots/sia5/sia5_with_jamming_and_kinectv2.urdf.xacro (robot description, xacro)
@@ -11,5 +11,5 @@
   <!-- Joint -->
   <joint name="joint_kinect2" type="fixed">
-	<origin rpy="0 ${29*M_PI/180} ${114/180*M_PI}" xyz="0.885 -0.78 0.75"/>
+	<origin xyz="0.8863 -0.7398 0.7912" rpy="0.0 0.5061 1.9897" />
     <parent link="base_link"/>
     <child link="kinect2_link"/>

File: robots/sia5/sia5_with_kinectv2.urdf.xacro (robot description, xacro)
@@ -11,5 +11,5 @@
   <!-- Joint -->
   <joint name="joint_kinect2" type="fixed">
-    <origin rpy="0 ${10*M_PI/180} ${M_PI}" xyz="1.05024 0 0.3195"/>
+	<origin xyz="0.8863 -0.7398 0.7912" rpy="0.0 0.5061 1.9897" />
     <parent link="base_link"/>
     <child link="kinect2_link"/>

File: robots/sia5/sia5_with_multi_kinectv2.urdf.xacro (robot description, xacro)
@@ -12,5 +12,5 @@
   <!-- Joint -->
   <joint name="joint_kinect_first" type="fixed">
-    <origin rpy="0 ${29*M_PI/180} ${114/180*M_PI}" xyz="0.86 -0.78 0.75"/>
+    <origin xyz="0.8863 -0.7398 0.7912" rpy="0.0 0.5061 1.9897" />
     <parent link="base_link"/>
     <child link="kinect_first_link"/>
@@ -24,16 +24,10 @@
   <xacro:kinect_gazebo name="kinect_first"/>
   <!-- Link -->
-  <xacro:kinect2_link_box_v0 name="kinect_second_link"/>
-  <link name="kinect_second_rgb_optical_frame"/>
+  <xacro:kinect2_link_box_v0 name="camera_link"/>
   <!-- Joint -->
   <joint name="joint_kinect_second" type="fixed">
-    <origin rpy="0 ${29*M_PI/180} -${114/180*M_PI}" xyz="0.86 0.78 0.75"/>
+    <origin rpy="0 ${20*M_PI/180} -${125/180*M_PI}" xyz="0.92 1.02 0.68"/>
     <parent link="base_link"/>
-    <child link="kinect_second_link"/>
-  </joint>
-  <joint name="joint_rgb_kinect_second" type="fixed">
-    <origin rpy="${M_PI/2} ${M_PI} ${M_PI/2}"/>
-    <parent link="kinect_second_link"/>
-    <child link="kinect_second_rgb_optical_frame"/>
+    <child link="camera_link"/>
   </joint>
   <!-- Gazebo -->
