Commit message: [modify] 20 [cm]の台を想定した高さに変更

File: robots/sia5/sia5_with_dhand.urdf.xacro (robot description, xacro)
@@ -2,6 +2,9 @@
 <robot name="sia5" xmlns:xacro="http://ros.org/wiki/xacro">
   <!-- File Include -->
-  <xacro:include filename="$(find motoman_description)/robots/sia5/sia5.urdf.xacro"/>
+  <xacro:include filename="$(find motoman_description)/robots/sia5/sia5_basic.urdf.xacro"/>
   <xacro:include filename="$(find dhand_description)/robots/dhand_adapted.urdf.xacro"/>
+  <xacro:add_world>
+    <origin xyz="0 0 0.2" rpy="0 0 0"/>
+  </xacro:add_world>
   <!-- Joint -->
   <joint name="dhand_adapter_joint" type="fixed">
