Commit message: [modify] kinect multiを変更
実機と同じlink、topic名になるように変更

File: robots/sia5/sia5_with_multi_kinectv2.urdf.xacro (robot description, xacro)
@@ -4,8 +4,39 @@
   <xacro:include filename="$(find motoman_description)/urdf/sensor/kinect.urdf.xacro"/>
   <xacro:include filename="$(find motoman_description)/urdf/sensor/kinect.gazebo.xacro"/>
-  <xacro:include filename="$(find motoman_description)/robots/sia5/sia5.urdf.xacro"/>
+  <xacro:include filename="$(find motoman_description)/robots/sia5/sia5_with_jamming.urdf.xacro"/>
   <!-- add Kinect V2 -->
+  <!-- Kinect_first -->
+  <!-- Link -->
+  <xacro:kinect2_link_box_v0 name="kinect_first_link"/>
+  <link name="kinect_first_rgb_optical_frame"/>
+  <!-- Joint -->
+  <joint name="joint_kinect_first" type="fixed">
+    <origin rpy="0 ${29*M_PI/180} ${114/180*M_PI}" xyz="0.86 -0.78 0.75"/>
+    <parent link="base_link"/>
+    <child link="kinect_first_link"/>
+  </joint>
+  <joint name="joint_rgb_kinect_first" type="fixed">
+	<origin rpy="${M_PI/2} ${M_PI} ${M_PI/2}"/>
+	<parent link="kinect_first_link"/>
+	<child link="kinect_first_rgb_optical_frame"/>
+  </joint>
   <!-- Gazebo -->
-  <xacro:kinect_joints suffix="/kinect_first" rpy="0 0 -${120*M_PI/180}" xyz="1 0.8660 0.5"/>
-  <xacro:kinect_joints suffix="/kinect_second" rpy="0 0 ${120*M_PI/180}" xyz="1 -0.8660 0.5"/>
+  <xacro:kinect_gazebo name="kinect_first"/>
+  <!-- Kinect_second -->
+  <!-- Link -->
+  <xacro:kinect2_link_box_v0 name="kinect_second_link"/>
+  <link name="kinect_second_rgb_optical_frame"/>
+  <!-- Joint -->
+  <joint name="joint_kinect_second" type="fixed">
+    <origin rpy="0 ${10*M_PI/180} ${M_PI}" xyz="1.05024 -1 0.3195"/>
+    <parent link="base_link"/>
+    <child link="kinect_second_link"/>
+  </joint>
+  <joint name="joint_rgb_kinect_second" type="fixed">
+	<origin rpy="${M_PI/2} ${M_PI} ${M_PI/2}"/>
+	<parent link="kinect_second_link"/>
+	<child link="kinect_second_rgb_optical_frame"/>
+  </joint>
+  <!-- Gazebo -->
+  <xacro:kinect_gazebo name="kinect_second"/>
 </robot>

File: urdf/sensor/kinect.gazebo.xacro (robot description, xacro)
@@ -2,32 +2,32 @@
 <robot xmlns:xacro="http://ros.org/wiki/xacro">
   <xacro:include filename="$(find motoman_description)/urdf/common.xacro" />
-  <xacro:macro name="kinect_gazebo" params="name suffix">
-    <gazebo reference="${name}_link">
-      <mu1>0.2</mu1>
-      <mu2>0.2</mu2>
-      <material>Gazebo/Black</material>
-      <!-- hd -->
+  <xacro:macro name="kinect_gazebo" params="name">
+	<gazebo reference="${name}_link">
+	  <mu1>0.2</mu1>
+	  <mu2>0.2</mu2>
+	  <material>Gazebo/Black</material>
+	  <!-- hd -->
       <sensor type="depth" name="${name}">
-        <always_on>true</always_on>
-        <update_rate>30.0</update_rate>
-        <camera>
+		<always_on>true</always_on>
+		<update_rate>30.0</update_rate>
+		<camera>
           <horizontal_fov>${84.1*M_PI/180.0}</horizontal_fov>
           <image>
-        <format>R8G8B8</format>
-        <width>512</width>
-        <height>424</height>
+			<format>R8G8B8</format>
+			<width>512</width>
+			<height>424</height>
           </image>
           <clip>
-        <near>0.05</near>
-        <far>4.5</far>
+			<near>0.05</near>
+			<far>4.5</far>
           </clip>
-          <noise>
-            <type>gaussian</type>
-            <mean>0.0</mean>
-            <stddev>0.005</stddev>
-          </noise>
-        </camera>
-        <plugin name="${name}_camera_controller" filename="libgazebo_ros_openni_kinect.so">
-          <cameraName>${suffix}/kinect2/hd</cameraName>
+		  <noise>
+			<type>gaussian</type>
+			<mean>0.0</mean>
+			<stddev>0.005</stddev>
+		  </noise>
+		</camera>
+		<plugin name="${name}_camera_controller" filename="libgazebo_ros_openni_kinect.so">
+          <cameraName>${name}/hd</cameraName>
           <alwaysOn>true</alwaysOn>
           <updateRate>30</updateRate>
@@ -45,30 +45,30 @@
           <distortion_t2>0.0</distortion_t2>
           <pointCloudCutoff>0.05</pointCloudCutoff>
-          <pointCloudCutoffMax>4.5</pointCloudCutoffMax>
-        </plugin>
+		  <pointCloudCutoffMax>4.5</pointCloudCutoffMax>
+		</plugin>
       </sensor>
-      <!-- qhd -->
+	  <!-- qhd -->
       <sensor type="depth" name="${name}">
-        <always_on>true</always_on>
-        <update_rate>30.0</update_rate>
-        <camera>
+		<always_on>true</always_on>
+		<update_rate>30.0</update_rate>
+		<camera>
           <horizontal_fov>${84.1*M_PI/180.0}</horizontal_fov>
           <image>
-            <format>R8G8B8</format>
-            <width>512</width>
-            <height>424</height>
+			<format>R8G8B8</format>
+			<width>512</width>
+			<height>424</height>
           </image>
           <clip>
-            <near>0.05</near>
-            <far>4.5</far>
+			<near>0.05</near>
+			<far>4.5</far>
           </clip>
-          <noise>
-            <type>gaussian</type>
-            <mean>0.0</mean>
-            <stddev>0.005</stddev>
-          </noise>
-        </camera>
-        <plugin name="${name}_camera_controller" filename="libgazebo_ros_openni_kinect.so">
-          <cameraName>${suffix}/kinect2/qhd</cameraName>
+		  <noise>
+			<type>gaussian</type>
+			<mean>0.0</mean>
+			<stddev>0.005</stddev>
+		  </noise>
+		</camera>
+		<plugin name="${name}_camera_controller" filename="libgazebo_ros_openni_kinect.so">
+          <cameraName>${name}/qhd</cameraName>
           <alwaysOn>true</alwaysOn>
           <updateRate>30</updateRate>
@@ -86,30 +86,30 @@
           <distortion_t2>0.0</distortion_t2>
           <pointCloudCutoff>0.05</pointCloudCutoff>
-          <pointCloudCutoffMax>4.5</pointCloudCutoffMax>
-        </plugin>
+		  <pointCloudCutoffMax>4.5</pointCloudCutoffMax>
+		</plugin>
       </sensor>
 	  <!-- sd -->
       <sensor type="depth" name="${name}">
-        <always_on>true</always_on>
-        <update_rate>30.0</update_rate>
-        <camera>
+		<always_on>true</always_on>
+		<update_rate>30.0</update_rate>
+		<camera>
           <horizontal_fov>${84.1*M_PI/180.0}</horizontal_fov>
           <image>
-            <format>R8G8B8</format>
-            <width>512</width>
-            <height>424</height>
+			<format>R8G8B8</format>
+			<width>512</width>
+			<height>424</height>
           </image>
           <clip>
-          <near>0.05</near>
-          <far>4.5</far>
+			<near>0.05</near>
+			<far>4.5</far>
           </clip>
-          <noise>
-            <type>gaussian</type>
-            <mean>0.0</mean>
-            <stddev>0.005</stddev>
-          </noise>
-        </camera>
-        <plugin name="${name}_camera_controller" filename="libgazebo_ros_openni_kinect.so">
-          <cameraName>${suffix}/kinect2/sd</cameraName>
+		  <noise>
+			<type>gaussian</type>
+			<mean>0.0</mean>
+			<stddev>0.005</stddev>
+		  </noise>
+		</camera>
+		<plugin name="${name}_camera_controller" filename="libgazebo_ros_openni_kinect.so">
+          <cameraName>${name}/sd</cameraName>
           <alwaysOn>true</alwaysOn>
           <updateRate>30</updateRate>
@@ -127,8 +127,8 @@
           <distortion_t2>0.0</distortion_t2>
           <pointCloudCutoff>0.05</pointCloudCutoff>
-          <pointCloudCutoffMax>4.5</pointCloudCutoffMax>
-        </plugin>
+		  <pointCloudCutoffMax>4.5</pointCloudCutoffMax>
+		</plugin>
       </sensor>
-    </gazebo>
+	</gazebo>
   </xacro:macro>
 </robot>

File: urdf/sensor/kinect.urdf.xacro (robot description, xacro)
@@ -1,8 +1,8 @@
 <?xml version="1.0"?>
 <robot xmlns:xacro="http://ros.org/wiki/xacro">
-  <xacro:macro name="kinect2_link_box_v0" params="name">
+<xacro:macro name="kinect2_link_box_v0" params="name">
     <link name="${name}">
       <visual>
-        <material name="black"/>
+		<material name="black"/>
         <geometry>
           <mesh filename="package://motoman_description/meshes/sensor/visual/COLLADA/kinectv2.stl"/>
@@ -10,7 +10,7 @@
       </visual>
       <collision>
-        <origin xyz="0 0 0.041"/>
+		<origin xyz="0 0 0.041"/>
         <geometry>
-          <box size="0.065 0.25 0.082"/>
+		  <box size="0.065 0.25 0.082"/>
         </geometry>
       </collision>
@@ -18,25 +18,8 @@
         <mass value="0.935"/>
         <inertia ixx="0.0053937" ixy="0" ixz="0"
-                 iyy="0.00085311" iyz="0"
-                 izz="0.00519899" />
+				 iyy="0.00085311" iyz="0"
+				 izz="0.00519899" />
       </inertial>
     </link>
-  </xacro:macro>
-  <xacro:macro name="kinect_joints" params="suffix rpy xyz">
-    <xacro:kinect2_link_box_v0 name="${suffix}/kinect2_link"/>
-    <link name="${suffix}/kinect2_rgb_optical_frame"/>
-    <!-- Joint -->
-    <joint name="${suffix}/joint_kinect2" type="fixed">
-      <origin rpy="${rpy}" xyz="${xyz}"/>
-      <parent link="base_link"/>
-      <child link="${suffix}/kinect2_link"/>
-    </joint>
-    <joint name="${suffix}/joint_rgb_kinect2" type="fixed">
-      <origin rpy="${M_PI/2} ${M_PI} ${M_PI/2}"/>
-      <parent link="${suffix}/kinect2_link"/>
-      <child link="${suffix}/kinect2_rgb_optical_frame"/>
-    </joint>
-    <!-- Gazebo -->
-    <xacro:kinect_gazebo name="${suffix}/kinect2" suffix="${suffix}"/>
-  </xacro:macro>
+</xacro:macro>
 </robot>

Commit message: [Fix] 複数のKinectを想定した部分の仕様変更に対応 launchからpointcloud2のsubscribeするトピック名を変更することができなくなっています． 問題解決中．..

File: robots/sia5/sia5_with_multi_kinectv2.urdf.xacro (robot description, xacro)
@@ -23,5 +23,4 @@
   <!-- Gazebo -->
   <xacro:kinect_gazebo name="kinect_first"/>
-  <!-- Kinect_second -->
   <!-- Link -->
   <xacro:kinect2_link_box_v0 name="kinect_second_link"/>
@@ -34,7 +33,7 @@
   </joint>
   <joint name="joint_rgb_kinect_second" type="fixed">
-	<origin rpy="${M_PI/2} ${M_PI} ${M_PI/2}"/>
-	<parent link="kinect_second_link"/>
-	<child link="kinect_second_rgb_optical_frame"/>
+    <origin rpy="${M_PI/2} ${M_PI} ${M_PI/2}"/>
+    <parent link="kinect_second_link"/>
+    <child link="kinect_second_rgb_optical_frame"/>
   </joint>
   <!-- Gazebo -->

File: urdf/sensor/kinect.gazebo.xacro (robot description, xacro)
@@ -3,30 +3,30 @@
   <xacro:include filename="$(find motoman_description)/urdf/common.xacro" />
   <xacro:macro name="kinect_gazebo" params="name">
-	<gazebo reference="${name}_link">
-	  <mu1>0.2</mu1>
-	  <mu2>0.2</mu2>
-	  <material>Gazebo/Black</material>
-	  <!-- hd -->
+    <gazebo reference="${name}_link">
+      <mu1>0.2</mu1>
+      <mu2>0.2</mu2>
+      <material>Gazebo/Black</material>
+      <!-- hd -->
       <sensor type="depth" name="${name}">
-		<always_on>true</always_on>
-		<update_rate>30.0</update_rate>
-		<camera>
+        <always_on>true</always_on>
+        <update_rate>30.0</update_rate>
+        <camera>
           <horizontal_fov>${84.1*M_PI/180.0}</horizontal_fov>
           <image>
-			<format>R8G8B8</format>
-			<width>512</width>
-			<height>424</height>
+            <format>R8G8B8</format>
+            <width>512</width>
+            <height>424</height>
           </image>
           <clip>
-			<near>0.05</near>
-			<far>4.5</far>
+            <near>0.05</near>
+            <far>4.5</far>
           </clip>
-		  <noise>
-			<type>gaussian</type>
-			<mean>0.0</mean>
-			<stddev>0.005</stddev>
-		  </noise>
-		</camera>
-		<plugin name="${name}_camera_controller" filename="libgazebo_ros_openni_kinect.so">
+          <noise>
+            <type>gaussian</type>
+            <mean>0.0</mean>
+            <stddev>0.005</stddev>
+          </noise>
+        </camera>
+        <plugin name="${name}_camera_controller" filename="libgazebo_ros_openni_kinect.so">
           <cameraName>${name}/hd</cameraName>
           <alwaysOn>true</alwaysOn>
@@ -45,29 +45,29 @@
           <distortion_t2>0.0</distortion_t2>
           <pointCloudCutoff>0.05</pointCloudCutoff>
-		  <pointCloudCutoffMax>4.5</pointCloudCutoffMax>
-		</plugin>
+          <pointCloudCutoffMax>4.5</pointCloudCutoffMax>
+        </plugin>
       </sensor>
-	  <!-- qhd -->
+      <!-- qhd -->
       <sensor type="depth" name="${name}">
-		<always_on>true</always_on>
-		<update_rate>30.0</update_rate>
-		<camera>
+        <always_on>true</always_on>
+        <update_rate>30.0</update_rate>
+        <camera>
           <horizontal_fov>${84.1*M_PI/180.0}</horizontal_fov>
           <image>
-			<format>R8G8B8</format>
-			<width>512</width>
-			<height>424</height>
+            <format>R8G8B8</format>
+            <width>512</width>
+            <height>424</height>
           </image>
           <clip>
-			<near>0.05</near>
-			<far>4.5</far>
+            <near>0.05</near>
+            <far>4.5</far>
           </clip>
-		  <noise>
-			<type>gaussian</type>
-			<mean>0.0</mean>
-			<stddev>0.005</stddev>
-		  </noise>
-		</camera>
-		<plugin name="${name}_camera_controller" filename="libgazebo_ros_openni_kinect.so">
+          <noise>
+            <type>gaussian</type>
+            <mean>0.0</mean>
+            <stddev>0.005</stddev>
+          </noise>
+        </camera>
+        <plugin name="${name}_camera_controller" filename="libgazebo_ros_openni_kinect.so">
           <cameraName>${name}/qhd</cameraName>
           <alwaysOn>true</alwaysOn>
@@ -86,29 +86,29 @@
           <distortion_t2>0.0</distortion_t2>
           <pointCloudCutoff>0.05</pointCloudCutoff>
-		  <pointCloudCutoffMax>4.5</pointCloudCutoffMax>
-		</plugin>
+          <pointCloudCutoffMax>4.5</pointCloudCutoffMax>
+        </plugin>
       </sensor>
-	  <!-- sd -->
+      <!-- sd -->
       <sensor type="depth" name="${name}">
-		<always_on>true</always_on>
-		<update_rate>30.0</update_rate>
-		<camera>
+        <always_on>true</always_on>
+        <update_rate>30.0</update_rate>
+        <camera>
           <horizontal_fov>${84.1*M_PI/180.0}</horizontal_fov>
           <image>
-			<format>R8G8B8</format>
-			<width>512</width>
-			<height>424</height>
+            <format>R8G8B8</format>
+            <width>512</width>
+            <height>424</height>
           </image>
           <clip>
-			<near>0.05</near>
-			<far>4.5</far>
+            <near>0.05</near>
+            <far>4.5</far>
           </clip>
-		  <noise>
-			<type>gaussian</type>
-			<mean>0.0</mean>
-			<stddev>0.005</stddev>
-		  </noise>
-		</camera>
-		<plugin name="${name}_camera_controller" filename="libgazebo_ros_openni_kinect.so">
+          <noise>
+            <type>gaussian</type>
+            <mean>0.0</mean>
+            <stddev>0.005</stddev>
+          </noise>
+        </camera>
+        <plugin name="${name}_camera_controller" filename="libgazebo_ros_openni_kinect.so">
           <cameraName>${name}/sd</cameraName>
           <alwaysOn>true</alwaysOn>
@@ -127,8 +127,8 @@
           <distortion_t2>0.0</distortion_t2>
           <pointCloudCutoff>0.05</pointCloudCutoff>
-		  <pointCloudCutoffMax>4.5</pointCloudCutoffMax>
-		</plugin>
+          <pointCloudCutoffMax>4.5</pointCloudCutoffMax>
+        </plugin>
       </sensor>
-	</gazebo>
+    </gazebo>
   </xacro:macro>
 </robot>

Commit message: [Fix] 2台めのkinectの位置を移動させました．

File: robots/sia5/sia5_with_multi_kinectv2.urdf.xacro (robot description, xacro)
@@ -17,7 +17,7 @@
   </joint>
   <joint name="joint_rgb_kinect_first" type="fixed">
-	<origin rpy="${M_PI/2} ${M_PI} ${M_PI/2}"/>
-	<parent link="kinect_first_link"/>
-	<child link="kinect_first_rgb_optical_frame"/>
+    <origin rpy="${M_PI/2} ${M_PI} ${M_PI/2}"/>
+    <parent link="kinect_first_link"/>
+    <child link="kinect_first_rgb_optical_frame"/>
   </joint>
   <!-- Gazebo -->
@@ -28,5 +28,5 @@
   <!-- Joint -->
   <joint name="joint_kinect_second" type="fixed">
-    <origin rpy="0 ${10*M_PI/180} ${M_PI}" xyz="1.05024 -1 0.3195"/>
+    <origin rpy="0 ${29*M_PI/180} -${114/180*M_PI}" xyz="0.86 0.78 0.75"/>
     <parent link="base_link"/>
     <child link="kinect_second_link"/>

Commit message: [Fix] 2台のキネクトからoctomap生成のための位置調整

File: robots/sia5/sia5_with_multi_kinectv2.urdf.xacro (robot description, xacro)
@@ -23,11 +23,18 @@
   <!-- Gazebo -->
   <xacro:kinect_gazebo name="kinect_first"/>
+  <!-- Kinect_second -->
   <!-- Link -->
-  <xacro:kinect2_link_box_v0 name="camera_link"/>
+  <xacro:kinect2_link_box_v0 name="kinect_second_link"/>
+  <link name="kinect_second_rgb_optical_frame"/>
   <!-- Joint -->
   <joint name="joint_kinect_second" type="fixed">
-    <origin rpy="0 ${20*M_PI/180} -${125/180*M_PI}" xyz="0.92 1.02 0.68"/>
+    <origin xyz="0.9685 1.203 0.7466" rpy="0.0029 0.2681 -2.1377" />
     <parent link="base_link"/>
-    <child link="camera_link"/>
+    <child link="kinect_second_link"/>
+  </joint>
+  <joint name="joint_rgb_kinect_second" type="fixed">
+    <origin rpy="${M_PI/2} ${M_PI} ${M_PI/2}"/>
+    <parent link="kinect_second_link"/>
+    <child link="kinect_second_rgb_optical_frame"/>
   </joint>
   <!-- Gazebo -->

Commit message: [Fix] 実機のkinectの位置修正

File: robots/sia5/sia5_with_multi_kinectv2.urdf.xacro (robot description, xacro)
@@ -29,5 +29,5 @@
   <!-- Joint -->
   <joint name="joint_kinect_second" type="fixed">
-    <origin xyz="0.9685 1.203 0.7466" rpy="0.0029 0.2681 -2.1377" />
+    <origin xyz="0.9636 1.2007 0.7466" rpy="0.0029 0.2681 -2.0649" />
     <parent link="base_link"/>
     <child link="kinect_second_link"/>

Commit message: [Fix] kinectの位置修正

File: robots/sia5/sia5_with_multi_kinectv2.urdf.xacro (robot description, xacro)
@@ -12,5 +12,5 @@
   <!-- Joint -->
   <joint name="joint_kinect_first" type="fixed">
-    <origin xyz="0.8863 -0.7398 0.7912" rpy="0.0 0.5061 1.9897" />
+    <origin xyz="0.8625 -0.7818 0.7662" rpy="-0.0209 0.5976 1.9579" />
     <parent link="base_link"/>
     <child link="kinect_first_link"/>

Commit message: [modify] kinectの位置合わせ
毎回ずれるのでなんとかしたい...

File: robots/sia5/sia5_with_multi_kinectv2.urdf.xacro (robot description, xacro)
@@ -12,5 +12,5 @@
   <!-- Joint -->
   <joint name="joint_kinect_first" type="fixed">
-    <origin xyz="0.8625 -0.7818 0.7662" rpy="-0.0209 0.5976 1.9579" />
+    <origin xyz="0.8625 -0.7708 0.7662" rpy="-0.0209 0.5976 1.9287" />
     <parent link="base_link"/>
     <child link="kinect_first_link"/>

Commit message: [modify] クラスタリングのパラメータを変更

File: robots/sia5/sia5_with_multi_kinectv2.urdf.xacro (robot description, xacro)
@@ -12,5 +12,5 @@
   <!-- Joint -->
   <joint name="joint_kinect_first" type="fixed">
-    <origin xyz="0.8625 -0.7708 0.7662" rpy="-0.0209 0.5976 1.9287" />
+    <origin xyz="0.8932 -0.6831 0.5095" rpy="0.0046 0.5044 1.9714" />
     <parent link="base_link"/>
     <child link="kinect_first_link"/>
@@ -29,5 +29,5 @@
   <!-- Joint -->
   <joint name="joint_kinect_second" type="fixed">
-    <origin xyz="0.9636 1.2007 0.7466" rpy="0.0029 0.2681 -2.0649" />
+    <origin xyz="1.0211 1.2502 0.5335" rpy="0.0029 0.2681 -2.1162" />
     <parent link="base_link"/>
     <child link="kinect_second_link"/>
