Commit message: [modify] kinectの位置を修正

File: robots/sia5/sia5_with_dhand_and_multi_kinect.urdf.xacro (robot description, xacro)
@@ -12,5 +12,5 @@
   <!-- Joint -->
   <joint name="joint_kinect_first" type="fixed">
-    <origin xyz="0.8625 -0.7708 0.7662" rpy="-0.0209 0.5976 1.9287" />
+	<origin xyz="0.8932 -0.6831 0.5095" rpy="0.0046 0.5044 1.9714" />
     <parent link="base_link"/>
     <child link="kinect_first_link"/>
@@ -29,5 +29,5 @@
   <!-- Joint -->
   <joint name="joint_kinect_second" type="fixed">
-    <origin xyz="0.9636 1.2007 0.7466" rpy="0.0029 0.2681 -2.0649" />
+	<origin xyz="1.0211 1.2502 0.5335" rpy="0.0029 0.2681 -2.1162" />
     <parent link="base_link"/>
     <child link="kinect_second_link"/>

Commit message: [modify] kinectの位置を修正

File: robots/sia5/sia5_with_dhand_and_multi_kinect.urdf.xacro (robot description, xacro)
@@ -12,5 +12,5 @@
   <!-- Joint -->
   <joint name="joint_kinect_first" type="fixed">
-	<origin xyz="0.8932 -0.6831 0.5095" rpy="0.0046 0.5044 1.9714" />
+	<origin xyz="0.8958 -0.6453 0.5866" rpy="-0.0204 0.5757 1.986" />
     <parent link="base_link"/>
     <child link="kinect_first_link"/>
@@ -29,5 +29,5 @@
   <!-- Joint -->
   <joint name="joint_kinect_second" type="fixed">
-	<origin xyz="1.0211 1.2502 0.5335" rpy="0.0029 0.2681 -2.1162" />
+	<origin xyz="1.0281 1.2353 0.5207" rpy="-0.0202 0.2594 -1.943" />
     <parent link="base_link"/>
     <child link="kinect_second_link"/>

Commit message: [Fix] 微調整

File: robots/sia5/sia5_with_dhand_and_multi_kinect.urdf.xacro (robot description, xacro)
@@ -12,5 +12,5 @@
   <!-- Joint -->
   <joint name="joint_kinect_first" type="fixed">
-	<origin xyz="0.8958 -0.6453 0.5866" rpy="-0.0204 0.5757 1.986" />
+    <origin xyz="0.8989 -0.6288 0.5766" rpy="-0.0102 0.5201 1.9827" />
     <parent link="base_link"/>
     <child link="kinect_first_link"/>

Commit message: [modify] kinectの位置を変更

File: robots/sia5/sia5_with_dhand_and_multi_kinect.urdf.xacro (robot description, xacro)
@@ -12,5 +12,5 @@
   <!-- Joint -->
   <joint name="joint_kinect_first" type="fixed">
-    <origin xyz="0.8989 -0.6288 0.5766" rpy="-0.0102 0.5201 1.9827" />
+    <origin xyz="0.9394 -0.6455 0.5172" rpy="0.0257 0.5551 2.0027" />
     <parent link="base_link"/>
     <child link="kinect_first_link"/>
@@ -29,5 +29,5 @@
   <!-- Joint -->
   <joint name="joint_kinect_second" type="fixed">
-	<origin xyz="1.0281 1.2353 0.5207" rpy="-0.0202 0.2594 -1.943" />
+    <origin xyz="1.0281 1.2353 0.5207" rpy="-0.0202 0.2594 -1.943" />
     <parent link="base_link"/>
     <child link="kinect_second_link"/>

File: robots/sia5/sia5_with_multi_kinectv2.urdf.xacro (robot description, xacro)
@@ -12,5 +12,5 @@
   <!-- Joint -->
   <joint name="joint_kinect_first" type="fixed">
-    <origin xyz="0.8932 -0.6831 0.5095" rpy="0.0046 0.5044 1.9714" />
+    <origin xyz="0.9394 -0.6455 0.5172" rpy="0.0257 0.5551 2.0027" />
     <parent link="base_link"/>
     <child link="kinect_first_link"/>
@@ -29,5 +29,5 @@
   <!-- Joint -->
   <joint name="joint_kinect_second" type="fixed">
-    <origin xyz="1.0211 1.2502 0.5335" rpy="0.0029 0.2681 -2.1162" />
+    <origin xyz="1.0281 1.2353 0.5207" rpy="-0.0202 0.2594 -1.943" />
     <parent link="base_link"/>
     <child link="kinect_second_link"/>

Commit message: [modify] demo-multiとkinectの位置を変更

File: robots/sia5/sia5_with_dhand_and_multi_kinect.urdf.xacro (robot description, xacro)
@@ -12,5 +12,5 @@
   <!-- Joint -->
   <joint name="joint_kinect_first" type="fixed">
-	<origin xyz="0.8958 -0.6453 0.5866" rpy="-0.0204 0.5757 1.986" />
+	<origin xyz=" 0.921276974256 -0.647838792922 0.553282433796 " rpy=" -0.0106089945569 0.55569160821 1.95680104985 "/>
     <parent link="base_link"/>
     <child link="kinect_first_link"/>
@@ -29,5 +29,5 @@
   <!-- Joint -->
   <joint name="joint_kinect_second" type="fixed">
-	<origin xyz="1.0281 1.2353 0.5207" rpy="-0.0202 0.2594 -1.943" />
+	<origin xyz=" 1.00328565606 1.28042806877 0.54831861169 " rpy=" -0.0301801280519 0.618375792511 -2.09530002388 "/>
     <parent link="base_link"/>
     <child link="kinect_second_link"/>

Commit message: [modify] コンフリクトを解消

File: robots/sia5/sia5_with_dhand_and_multi_kinect.urdf.xacro (robot description, xacro)
@@ -12,9 +12,5 @@
   <!-- Joint -->
   <joint name="joint_kinect_first" type="fixed">
-<<<<<<< HEAD
 	<origin xyz=" 0.921276974256 -0.647838792922 0.553282433796 " rpy=" -0.0106089945569 0.55569160821 1.95680104985 "/>
-=======
-    <origin xyz="0.9394 -0.6455 0.5172" rpy="0.0257 0.5551 2.0027" />
->>>>>>> c6aa6b887cd80afd4c9f0fdba25d93214c5b5e08
     <parent link="base_link"/>
     <child link="kinect_first_link"/>
@@ -33,9 +29,5 @@
   <!-- Joint -->
   <joint name="joint_kinect_second" type="fixed">
-<<<<<<< HEAD
 	<origin xyz=" 1.00328565606 1.28042806877 0.54831861169 " rpy=" -0.0301801280519 0.618375792511 -2.09530002388 "/>
-=======
-    <origin xyz="1.0281 1.2353 0.5207" rpy="-0.0202 0.2594 -1.943" />
->>>>>>> c6aa6b887cd80afd4c9f0fdba25d93214c5b5e08
     <parent link="base_link"/>
     <child link="kinect_second_link"/>

Commit message: [modify] kinectの位置を修正

File: robots/sia5/sia5_with_dhand_and_multi_kinect.urdf.xacro (robot description, xacro)
@@ -12,5 +12,5 @@
   <!-- Joint -->
   <joint name="joint_kinect_first" type="fixed">
-	<origin xyz=" 0.921276974256 -0.647838792922 0.553282433796 " rpy=" -0.0106089945569 0.55569160821 1.95680104985 "/>
+	<origin xyz="1.0966 0.8845 0.4916" rpy="-0.0023 0.4544 -2.3328" />
     <parent link="base_link"/>
     <child link="kinect_first_link"/>
@@ -29,5 +29,5 @@
   <!-- Joint -->
   <joint name="joint_kinect_second" type="fixed">
-	<origin xyz=" 1.00328565606 1.28042806877 0.54831861169 " rpy=" -0.0301801280519 0.618375792511 -2.09530002388 "/>
+	<origin xyz="1.3967 -0.7631 0.5403" rpy="-0.0286 0.4706 2.4854" />
     <parent link="base_link"/>
     <child link="kinect_second_link"/>

Commit message: [Fix] 実験室でのKinectの位置に修正

File: robots/sia5/sia5_with_dhand_and_multi_kinect.urdf.xacro (robot description, xacro)
@@ -12,5 +12,5 @@
   <!-- Joint -->
   <joint name="joint_kinect_first" type="fixed">
-	<origin xyz="1.0966 0.8845 0.4916" rpy="-0.0023 0.4544 -2.3328" />
+	<origin xyz=" 0.91881506129 -0.63904840004 0.547199354356 " rpy=" 0.00586550918238 0.572600688929 2.07762026701 "/>
     <parent link="base_link"/>
     <child link="kinect_first_link"/>
@@ -29,5 +29,5 @@
   <!-- Joint -->
   <joint name="joint_kinect_second" type="fixed">
-	<origin xyz="1.3967 -0.7631 0.5403" rpy="-0.0286 0.4706 2.4854" />
+	<origin xyz="1.0335 1.2465 0.5252" rpy="-0.0249 0.2883 -2.1046" />
     <parent link="base_link"/>
     <child link="kinect_second_link"/>

Commit message: [modify] kinectのキャレイブレーションをやった

File: robots/sia5/sia5_with_dhand_and_multi_kinect.urdf.xacro (robot description, xacro)
@@ -12,5 +12,5 @@
   <!-- Joint -->
   <joint name="joint_kinect_first" type="fixed">
-	<origin xyz=" 0.91881506129 -0.63904840004 0.547199354356 " rpy=" 0.00586550918238 0.572600688929 2.07762026701 "/>
+  <origin xyz="0.8872 -0.6445 0.5718" rpy="-0.0087 0.5501 2.0698" />
     <parent link="base_link"/>
     <child link="kinect_first_link"/>
@@ -29,5 +29,5 @@
   <!-- Joint -->
   <joint name="joint_kinect_second" type="fixed">
-	<origin xyz="1.0335 1.2465 0.5252" rpy="-0.0249 0.2883 -2.1046" />
+	<origin xyz="1.0013 1.2696 0.5348" rpy="-0.0249 0.2883 -2.0823" />
     <parent link="base_link"/>
     <child link="kinect_second_link"/>

Commit message: [Update] TFの位置更新

File: robots/sia5/sia5_with_dhand_and_multi_kinect.urdf.xacro (robot description, xacro)
@@ -29,5 +29,5 @@
   <!-- Joint -->
   <joint name="joint_kinect_second" type="fixed">
-	<origin xyz="1.0335 1.2465 0.5252" rpy="-0.0249 0.2883 -2.1046" />
+  <origin xyz="0.9992 1.2708 0.5301" rpy="-0.0145 0.3292 -2.017" />
     <parent link="base_link"/>
     <child link="kinect_second_link"/>

Commit message: [modify] kinectの位置を修正

File: robots/sia5/sia5_with_dhand_and_multi_kinect.urdf.xacro (robot description, xacro)
@@ -29,5 +29,5 @@
   <!-- Joint -->
   <joint name="joint_kinect_second" type="fixed">
-	<origin xyz="1.0013 1.2696 0.5348" rpy="-0.0249 0.2883 -2.0823" />
+	<origin xyz="1.0305 1.245 0.4908" rpy="-0.0547 0.3049 -2.063" />
     <parent link="base_link"/>
     <child link="kinect_second_link"/>

Commit message: [Fix] 検証中

File: robots/sia5/sia5_with_dhand_and_multi_kinect.urdf.xacro (robot description, xacro)
@@ -12,5 +12,5 @@
   <!-- Joint -->
   <joint name="joint_kinect_first" type="fixed">
-    <origin xyz="0.8872 -0.6445 0.5718" rpy="-0.0087 0.5501 2.0698" />
+    <origin xyz="0.8794 -0.6445 0.5804" rpy="-0.035 0.3421 2.0509" />
     <parent link="base_link"/>
     <child link="kinect_first_link"/>
@@ -29,5 +29,5 @@
   <!-- Joint -->
   <joint name="joint_kinect_second" type="fixed">
-    <origin xyz="1.0305 1.245 0.4908" rpy="-0.0547 0.3049 -2.063" />
+    <origin xyz="0.9639 1.286 0.5372" rpy="0.0053 0.3332 -1.9757" />
     <parent link="base_link"/>
     <child link="kinect_second_link"/>

Commit message: [modify] kinect のいち修正

File: robots/sia5/sia5_with_dhand_and_multi_kinect.urdf.xacro (robot description, xacro)
@@ -29,5 +29,5 @@
   <!-- Joint -->
   <joint name="joint_kinect_second" type="fixed">
-    <origin xyz="0.9639 1.286 0.5372" rpy="0.0053 0.3332 -1.9757" />
+	<origin xyz="1.4552 0.2663 0.4009" rpy="0.0327 0.4283 -2.9288" />
     <parent link="base_link"/>
     <child link="kinect_second_link"/>

Commit message: [modify] kinectの位置修正

File: robots/sia5/sia5_with_dhand_and_multi_kinect.urdf.xacro (robot description, xacro)
@@ -29,5 +29,5 @@
   <!-- Joint -->
   <joint name="joint_kinect_second" type="fixed">
-	<origin xyz="1.4552 0.2663 0.4009" rpy="0.0327 0.4283 -2.9288" />
+	<origin xyz="1.451 0.2935 0.4009" rpy="0.0327 0.4283 -2.9288" />
     <parent link="base_link"/>
     <child link="kinect_second_link"/>

Commit message: [modify] kinect position

File: robots/sia5/sia5_with_dhand_and_multi_kinect.urdf.xacro (robot description, xacro)
@@ -29,5 +29,5 @@
   <!-- Joint -->
   <joint name="joint_kinect_second" type="fixed">
-	<origin xyz="1.451 0.2935 0.4009" rpy="0.0327 0.4283 -2.9288" />
+	<origin xyz="1.4421 0.2935 0.3909" rpy="0.023 0.3795 -2.9326" />
     <parent link="base_link"/>
     <child link="kinect_second_link"/>

Commit message: [modify] position & pose

File: robots/sia5/sia5_with_dhand_and_multi_kinect.urdf.xacro (robot description, xacro)
@@ -29,5 +29,5 @@
   <!-- Joint -->
   <joint name="joint_kinect_second" type="fixed">
-	<origin xyz="1.4421 0.2935 0.3909" rpy="0.023 0.3795 -2.9326" />
+	<origin xyz="1.448 0.3215 0.3881" rpy="0.0666 0.381 -2.898" />
     <parent link="base_link"/>
     <child link="kinect_second_link"/>

Commit message: [modify] tmp

File: robots/sia5/sia5_with_dhand_and_multi_kinect.urdf.xacro (robot description, xacro)
@@ -6,21 +6,4 @@
   <xacro:include filename="$(find motoman_description)/robots/sia5/sia5_with_dhand.urdf.xacro"/>
   <!-- add Kinect V2 -->
-  <!-- Kinect_first -->
-  <!-- Link -->
-  <xacro:kinect2_link_box_v0 name="kinect_first_link"/>
-  <link name="kinect_first_rgb_optical_frame"/>
-  <!-- Joint -->
-  <joint name="joint_kinect_first" type="fixed">
-    <origin xyz="0.8794 -0.6445 0.5804" rpy="-0.035 0.3421 2.0509" />
-    <parent link="base_link"/>
-    <child link="kinect_first_link"/>
-  </joint>
-  <joint name="joint_rgb_kinect_first" type="fixed">
-    <origin rpy="${M_PI/2} ${M_PI} ${M_PI/2}"/>
-    <parent link="kinect_first_link"/>
-    <child link="kinect_first_rgb_optical_frame"/>
-  </joint>
-  <!-- Gazebo -->
-  <xacro:kinect_gazebo name="kinect_first"/>
   <!-- Kinect_second -->
   <!-- Link -->
@@ -29,5 +12,5 @@
   <!-- Joint -->
   <joint name="joint_kinect_second" type="fixed">
-	<origin xyz="1.448 0.3215 0.3881" rpy="0.0666 0.381 -2.898" />
+	<origin xyz="1.4828 0.0827 0.3932" rpy="-0.0031 0.4431 3.14" />
     <parent link="base_link"/>
     <child link="kinect_second_link"/>
@@ -40,3 +23,20 @@
   <!-- Gazebo -->
   <xacro:kinect_gazebo name="kinect_second"/>
+  <!-- Kinect_hand -->
+  <!-- Link -->
+  <xacro:kinect2_link_box_v0 name="kinect_hand_link"/>
+  <link name="kinect_hand_rgb_optical_frame"/>
+  <!-- Joint -->
+  <joint name="joint_kinect_hand" type="fixed">
+	<origin xyz="0.09 0 -0.035" rpy="${M_PI} 0 0" />
+    <parent link="link_t"/>
+    <child link="kinect_hand_link"/>
+  </joint>
+  <joint name="joint_rgb_kinect_hand" type="fixed">
+    <origin rpy="${M_PI/2} ${M_PI} ${M_PI/2}"/>
+    <parent link="kinect_hand_link"/>
+    <child link="kinect_hand_rgb_optical_frame"/>
+  </joint>
+  <!-- Gazebo -->
+  <xacro:kinect_gazebo name="kinect_hand"/>
 </robot>
