Commit message: [modify] left kinect's position into calibrated position

File: robots/sia5/sia5_with_dhand_and_4_kinects.urdf.xacro (robot description, xacro)
@@ -64,9 +64,9 @@
   <joint name="joint_left_right" type="fixed">
   <!-- Calibrated position -->
-  <!-- <origin xyz="-0.513 1.0085 0.756" rpy="0.0126 0.2924 -0.634" /> -->
+  <origin xyz="-0.513 1.0085 0.756" rpy="0.0126 0.2924 -0.634" />
   <!-- Test positions -->
   <!-- <origin xyz="-0.600 0.800 0.600" rpy="-0.01 0.3206 -0.4815" /> -->
   <!-- <origin xyz="-0.500 0.800 0.600" rpy="-0.01 0.3206 -0.4815" /> -->
-  <origin xyz="-0.4835 1.0027 0.7524" rpy="0.0126 0.2424 -0.6279" />
+  <!-- <origin xyz="-0.4835 1.0027 0.7524" rpy="0.0126 0.2424 -0.6279" /> -->
     <parent link="base_link"/>
     <child link="kinect_left_link"/>
