Commit message: [rename] urdfの名前変更

File: robots/sia5/urdf/sia5_no_tool.urdf (robot description, URDF)
Before this commit: robot sia5, 10 links, 9 joints
Links:
- added link table_link, mass 40.0; collision mesh filename=package://motoman_description/meshes/sia5/collision/STL/tab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; visual mesh filename=package://motoman_description/meshes/sia5/visual/COLLADA/ta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
- link base_link: mass 20.1477501679 -> 9.23913043478
- link link_b: mass 0.0805910006716 -> 0.869565217391
- link link_e: mass 0.604432505037 -> 1.30434782609
- link link_l: mass 4.02955003358 -> 7.60869565217
- link link_r: mass 0.0805910006716 -> 0.978260869565
- link link_s: mass 4.8354600403 -> 8.36956521739
- link link_t: mass 0.0201477501679 -> 0.54347826087
- link link_u: mass 0.201477501679 -> 1.08695652174
Joints:
- added joint joint_base: type fixed, parent table_link, child base_link
- joint world: child base_link -> table_link; origin (none) -> xyz=0 0 0.53

Commit message: [modify] tool0の位置を変更したurdfを作成

File: robots/sia5/urdf/sia5_no_tool.urdf (robot description, URDF)
Before this commit: robot sia5, 11 links, 10 joints
Links:
- link table_link: geometry collision box size=1.116 0.676 0.53; visual mesh filename=package://motoman_description/meshes/sia5/visual/COLLADA/ta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
Joints:
- joint joint_tool0: origin xyz=0.0115 0 -0.040 rpy=0 0 0 -> xyz=0.0115 0 0 rpy=0 0 0
