Commit message: [modify] kinectv2の色変更に伴うxacroの変更

File: urdf/sensor/kinect.gazebo.xacro (robot description, xacro)
@@ -4,4 +4,7 @@
   <xacro:macro name="kinect_gazebo" params="name">
 	<gazebo reference="${name}_link">
+	  <mu1>0.2</mu1>
+	  <mu2>0.2</mu2>
+	  <material>Gazebo/Black</material>
 	  <!-- hd -->
       <sensor type="depth" name="${name}">

File: urdf/sensor/kinect.urdf.xacro (robot description, xacro)
@@ -4,6 +4,7 @@
     <link name="${name}">
       <visual>
+		<material name="black"/>
         <geometry>
-          <mesh filename="package://motoman_description/meshes/sensor/visual/COLLADA/kinect2.dae"/>
+          <mesh filename="package://motoman_description/meshes/sensor/visual/COLLADA/kinectv2.stl"/>
         </geometry>
       </visual>
