Commit message: [modify] joint limits

File: robots/sda5/sda5_basic.urdf.xacro (robot description, xacro)
@@ -11,5 +11,5 @@
   <xacro:property name="joint_s_upper_limit" value="${270*M_PI/180}"/>
   <xacro:property name="joint_s_lower_limit" value="${-90*M_PI/180}"/>
-  <xacro:property name="joint_l_upper_limit" value="${110*M_PI/180*0.95}"/>
+  <xacro:property name="joint_l_upper_limit" value="${110*M_PI/180}"/>
   <xacro:property name="joint_l_lower_limit" value="-${joint_l_upper_limit}"/>
   <xacro:property name="joint_e_upper_limit" value="${170*M_PI/180}"/>
@@ -17,9 +17,9 @@
   <xacro:property name="joint_u_upper_limit" value="${115*M_PI/180}"/>
   <xacro:property name="joint_u_lower_limit" value="${-90*M_PI/180}"/>
-  <xacro:property name="joint_r_upper_limit" value="${180*0.95*M_PI/180.0}"/>
+  <xacro:property name="joint_r_upper_limit" value="${180*M_PI/180}"/>
   <xacro:property name="joint_r_lower_limit" value="-${joint_r_upper_limit}"/>
   <xacro:property name="joint_b_upper_limit" value="${110*M_PI/180}"/>
   <xacro:property name="joint_b_lower_limit" value="-${joint_b_upper_limit}"/>
-  <xacro:property name="joint_t_upper_limit" value="${180*0.95*M_PI/180}"/>
+  <xacro:property name="joint_t_upper_limit" value="${180*M_PI/180}"/>
   <xacro:property name="joint_t_lower_limit" value="-${joint_t_upper_limit}"/>
   <!-- Velocity limits -->

Commit message: [modify] inertial info

File: robots/sda5/sda5_basic.urdf.xacro (robot description, xacro)
@@ -42,5 +42,5 @@
   <!-- TORSO Link -->
   <xacro:torso_link_v0 parent="base_link">
-    <origin xyz="0.045 0 0.6646"/>
+    <origin xyz="0.045 0 0.6696"/>
     <limit effort="30.0" lower="${torso_joint_lower_limit}"
            upper="${torso_joint_upper_limit}" velocity="${torso_joint_velocity_limit}"/>
@@ -48,5 +48,5 @@
   <!-- Link Left Parts -->
   <!-- Link LS -->
-  <xacro:link_v2 prefix="l" suffix="s" parent="torso_link" mass="8.36956521739">
+  <xacro:link_v2 prefix="l" suffix="s" parent="torso_link" mass="5.00">
     <origin xyz="0 0 0" rpy="0 0 0"/>
     <inertia ixx="0.1285284" ixy="0" ixz="0"
@@ -57,8 +57,8 @@
   </xacro:link_v2>
   <!-- Link LL -->
-  <xacro:link_v2 prefix="l" suffix="l" parent="link_l_s" mass="8.36956521739">
-    <origin xyz="0 0 0" rpy="0 0 0"/>
-    <inertia ixx="0.1285284" ixy="0" ixz="0"
-             iyy="0.127697251956" iyz="0" izz="0.0186623672464"/>
+  <xacro:link_v2 prefix="l" suffix="l" parent="link_l_s" mass="5.00">
+    <origin rpy="3.14159274 0 0" xyz="0 -0.006 0.15"/>
+    <inertia ixx="0.12248884058" ixy="0" ixz="0"
+             iyy="0.117554616667" iyz="0" izz="0.0177495804348"/>
     <origin xyz="0 0.03575 0.13" rpy="${-M_PI/2} 0 0"/>
     <limit effort="30.0" lower="${joint_l_lower_limit}"
@@ -66,8 +66,8 @@
   </xacro:link_v2>
   <!-- Link LE -->
-  <xacro:link_v2 prefix="l" suffix="e" parent="link_l_l" mass="8.36956521739">
-    <origin xyz="0 0 0" rpy="0 0 0"/>
-    <inertia ixx="0.1285284" ixy="0" ixz="0"
-             iyy="0.127697251956" iyz="0" izz="0.0186623672464"/>
+  <xacro:link_v2 prefix="l" suffix="e" parent="link_l_l" mass="3.00">
+    <origin rpy="0 0 -1.57079637" xyz="0 0 0"/>
+    <inertia ixx="0.0122899381739" ixy="0" ixz="0"
+             iyy="0.0117127787826" iyz="0" izz="0.00344401234783"/>
     <origin xyz="0 -0.18225 -0.0365" rpy="${M_PI/2} 0 0"/>
     <limit effort="30.0" lower="${joint_e_lower_limit}"
@@ -75,8 +75,8 @@
   </xacro:link_v2>
   <!-- Link LU -->
-  <xacro:link_v2 prefix="l" suffix="u" parent="link_l_e" mass="8.36956521739">
-    <origin xyz="0 0 0" rpy="0 0 0"/>
-    <inertia ixx="0.1285284" ixy="0" ixz="0"
-             iyy="0.127697251956" iyz="0" izz="0.0186623672464"/>
+  <xacro:link_v2 prefix="l" suffix="u" parent="link_l_e" mass="2.00">
+    <origin rpy="-3.14159274 1.57079637 0" xyz="0.008 -0.06 -0.131"/>
+    <inertia ixx="0.0110207115768" ixy="0" ixz="0"
+             iyy="0.00996803594202" iyz="0" izz="0.00214043853333"/>
     <origin xyz="0.085 -0.02928 0.087" rpy="0 ${M_PI/2} ${-M_PI/2}"/>
     <limit effort="30.0" lower="${joint_u_lower_limit}"
@@ -84,8 +84,8 @@
   </xacro:link_v2>
   <!-- Link LR -->
-  <xacro:link_v2 prefix="l" suffix="r" parent="link_l_u" mass="8.36956521739">
-    <origin xyz="0 0 0" rpy="0 0 0"/>
-    <inertia ixx="0.1285284" ixy="0" ixz="0"
-             iyy="0.127697251956" iyz="0" izz="0.0186623672464"/>
+  <xacro:link_v2 prefix="l" suffix="r" parent="link_l_u" mass="2.00">
+    <origin rpy="0 0 -1.57079637" xyz="0 0 0"/>
+    <inertia ixx="0.0108400832201" ixy="0" ixz="0"
+             iyy="0.010708873981" iyz="0" izz="0.00140456861413"/>
     <origin xyz="-0.06 0.14428 -0.03" rpy="${M_PI/2} 0 0"/>
     <limit effort="30.0" lower="${joint_r_lower_limit}"
@@ -93,8 +93,8 @@
   </xacro:link_v2>
   <!-- Link LB -->
-  <xacro:link_v2 prefix="l" suffix="b" parent="link_l_r" mass="8.36956521739">
-    <origin xyz="0 0 0" rpy="0 0 0"/>
-    <inertia ixx="0.1285284" ixy="0" ixz="0"
-             iyy="0.127697251956" iyz="0" izz="0.0186623672464"/>
+  <xacro:link_v2 prefix="l" suffix="b" parent="link_l_r" mass="2.00">
+    <origin rpy="1.57079637 -1.57079637 0" xyz="0 0.0045 0.1365"/>
+    <inertia ixx="0.00814341869565" ixy="0" ixz="0"
+             iyy="0.00709473869565" iyz="0" izz="0.000736577391304"/>
     <origin xyz="0 -0.0392 -0.125" rpy="${-M_PI/2} 0 0"/>
     <limit effort="30.0" lower="${joint_b_lower_limit}"
@@ -102,8 +102,7 @@
   </xacro:link_v2>
   <!-- Link LT -->
-  <xacro:link_v2 prefix="l" suffix="t" parent="link_l_b" mass="8.36956521739">
-    <origin xyz="0 0 0" rpy="0 0 0"/>
-    <inertia ixx="0.1285284" ixy="0" ixz="0"
-             iyy="0.127697251956" iyz="0" izz="0.0186623672464"/>
+  <xacro:link_v2 prefix="l" suffix="t" parent="link_l_b" mass="1.00">
+    <origin xyz="0 0 0" rpy="0 0 0"/>
+    <inertia ixx="0.003" ixy="0" ixz="0" iyy="0.003" iyz="0" izz="0.001"/>
     <origin xyz="0 0.1365 0.0392" rpy="${M_PI/2} 0 0"/>
     <limit effort="30.0" lower="${joint_t_lower_limit}"
@@ -112,5 +111,5 @@
   <!-- Link Right Parts -->
   <!-- Link RS -->
-  <xacro:link_v2 prefix="r" suffix="s" parent="torso_link" mass="8.36956521739">
+  <xacro:link_v2 prefix="r" suffix="s" parent="torso_link" mass="5.00">
     <origin xyz="0 0 0" rpy="0 0 0"/>
     <inertia ixx="0.1285284" ixy="0" ixz="0"
@@ -121,8 +120,8 @@
   </xacro:link_v2>
   <!-- Link RL -->
-  <xacro:link_v2 prefix="r" suffix="l" parent="link_r_s" mass="8.36956521739">
-    <origin xyz="0 0 0" rpy="0 0 0"/>
-    <inertia ixx="0.1285284" ixy="0" ixz="0"
-             iyy="0.127697251956" iyz="0" izz="0.0186623672464"/>
+  <xacro:link_v2 prefix="r" suffix="l" parent="link_r_s" mass="5.00">
+    <origin rpy="3.14159274 0 0" xyz="0 -0.006 0.15"/>
+    <inertia ixx="0.12248884058" ixy="0" ixz="0"
+             iyy="0.117554616667" iyz="0" izz="0.0177495804348"/>
     <origin xyz="0 0.03575 0.13" rpy="${-M_PI/2} 0 0"/>
     <limit effort="30.0" lower="${joint_l_lower_limit}"
@@ -130,8 +129,8 @@
   </xacro:link_v2>
   <!-- Link RE -->
-  <xacro:link_v2 prefix="r" suffix="e" parent="link_r_l" mass="8.36956521739">
-    <origin xyz="0 0 0" rpy="0 0 0"/>
-    <inertia ixx="0.1285284" ixy="0" ixz="0"
-             iyy="0.127697251956" iyz="0" izz="0.0186623672464"/>
+  <xacro:link_v2 prefix="r" suffix="e" parent="link_r_l" mass="3.00">
+    <origin rpy="0 0 -1.57079637" xyz="0 0 0"/>
+    <inertia ixx="0.0122899381739" ixy="0" ixz="0"
+             iyy="0.0117127787826" iyz="0" izz="0.00344401234783"/>
     <origin xyz="0 -0.18225 -0.0365" rpy="${M_PI/2} 0 0"/>
     <limit effort="30.0" lower="${joint_e_lower_limit}"
@@ -139,8 +138,8 @@
   </xacro:link_v2>
   <!-- Link RU -->
-  <xacro:link_v2 prefix="r" suffix="u" parent="link_r_e" mass="8.36956521739">
-    <origin xyz="0 0 0" rpy="0 0 0"/>
-    <inertia ixx="0.1285284" ixy="0" ixz="0"
-             iyy="0.127697251956" iyz="0" izz="0.0186623672464"/>
+  <xacro:link_v2 prefix="r" suffix="u" parent="link_r_e" mass="2.00">
+    <origin rpy="-3.14159274 1.57079637 0" xyz="0.008 -0.06 -0.131"/>
+    <inertia ixx="0.0110207115768" ixy="0" ixz="0"
+             iyy="0.00996803594202" iyz="0" izz="0.00214043853333"/>
     <origin xyz="0.085 -0.02928 0.087" rpy="0 ${M_PI/2} ${-M_PI/2}"/>
     <limit effort="30.0" lower="${joint_u_lower_limit}"
@@ -148,8 +147,8 @@
   </xacro:link_v2>
   <!-- Link RR -->
-  <xacro:link_v2 prefix="r" suffix="r" parent="link_r_u" mass="8.36956521739">
-    <origin xyz="0 0 0" rpy="0 0 0"/>
-    <inertia ixx="0.1285284" ixy="0" ixz="0"
-             iyy="0.127697251956" iyz="0" izz="0.0186623672464"/>
+  <xacro:link_v2 prefix="r" suffix="r" parent="link_r_u" mass="2.00">
+    <origin rpy="0 0 -1.57079637" xyz="0 0 0"/>
+    <inertia ixx="0.0108400832201" ixy="0" ixz="0"
+             iyy="0.010708873981" iyz="0" izz="0.00140456861413"/>
     <origin xyz="-0.06 0.14428 -0.03" rpy="${M_PI/2} 0 0"/>
     <limit effort="30.0" lower="${joint_r_lower_limit}"
@@ -157,8 +156,8 @@
   </xacro:link_v2>
   <!-- Link RB -->
-  <xacro:link_v2 prefix="r" suffix="b" parent="link_r_r" mass="8.36956521739">
-    <origin xyz="0 0 0" rpy="0 0 0"/>
-    <inertia ixx="0.1285284" ixy="0" ixz="0"
-             iyy="0.127697251956" iyz="0" izz="0.0186623672464"/>
+  <xacro:link_v2 prefix="r" suffix="b" parent="link_r_r" mass="2.00">
+    <origin rpy="1.57079637 -1.57079637 0" xyz="0 0.0045 0.1365"/>
+    <inertia ixx="0.00814341869565" ixy="0" ixz="0"
+             iyy="0.00709473869565" iyz="0" izz="0.000736577391304"/>
     <origin xyz="0 -0.0392 -0.125" rpy="${-M_PI/2} 0 0"/>
     <limit effort="30.0" lower="${joint_b_lower_limit}"
@@ -166,8 +165,7 @@
   </xacro:link_v2>
   <!-- Link RT -->
-  <xacro:link_v2 prefix="r" suffix="t" parent="link_r_b" mass="8.36956521739">
-    <origin xyz="0 0 0" rpy="0 0 0"/>
-    <inertia ixx="0.1285284" ixy="0" ixz="0"
-             iyy="0.127697251956" iyz="0" izz="0.0186623672464"/>
+  <xacro:link_v2 prefix="r" suffix="t" parent="link_r_b" mass="1.00">
+    <origin xyz="0 0 0" rpy="0 0 0"/>
+    <inertia ixx="0.003" ixy="0" ixz="0" iyy="0.003" iyz="0" izz="0.001"/>
     <origin xyz="0 0.1365 0.0392" rpy="${M_PI/2} 0 0"/>
     <limit effort="30.0" lower="${joint_t_lower_limit}"
@@ -178,16 +176,16 @@
   <xacro:trans_v0 prefix="l" suffix="s" reduction="300"/>
   <xacro:trans_v0 prefix="l" suffix="l" reduction="300"/>
-  <xacro:trans_v0 prefix="l" suffix="e" reduction="300"/>
-  <xacro:trans_v0 prefix="l" suffix="u" reduction="300"/>
-  <xacro:trans_v0 prefix="l" suffix="r" reduction="300"/>
-  <xacro:trans_v0 prefix="l" suffix="b" reduction="300"/>
-  <xacro:trans_v0 prefix="l" suffix="t" reduction="300"/>
+  <xacro:trans_v0 prefix="l" suffix="e" reduction="100"/>
+  <xacro:trans_v0 prefix="l" suffix="u" reduction="50"/>
+  <xacro:trans_v0 prefix="l" suffix="r" reduction="30"/>
+  <xacro:trans_v0 prefix="l" suffix="b" reduction="30"/>
+  <xacro:trans_v0 prefix="l" suffix="t" reduction="10"/>
   <xacro:trans_v0 prefix="r" suffix="s" reduction="300"/>
   <xacro:trans_v0 prefix="r" suffix="l" reduction="300"/>
-  <xacro:trans_v0 prefix="r" suffix="e" reduction="300"/>
-  <xacro:trans_v0 prefix="r" suffix="u" reduction="300"/>
-  <xacro:trans_v0 prefix="r" suffix="r" reduction="300"/>
-  <xacro:trans_v0 prefix="r" suffix="b" reduction="300"/>
-  <xacro:trans_v0 prefix="r" suffix="t" reduction="300"/>
+  <xacro:trans_v0 prefix="r" suffix="e" reduction="100"/>
+  <xacro:trans_v0 prefix="r" suffix="u" reduction="50"/>
+  <xacro:trans_v0 prefix="r" suffix="r" reduction="30"/>
+  <xacro:trans_v0 prefix="r" suffix="b" reduction="30"/>
+  <xacro:trans_v0 prefix="r" suffix="t" reduction="10"/>
   <!-- Add Gazebo -->
   <xacro:torso_gazebo_v1/>
