Commit message: [update] add hole links

File: motoman_description/urdf/sia20/link.urdf.xacro (robot description, xacro)
@@ -7,5 +7,4 @@
     <link name="link_${suffix}">
       <visual>
-        <origin rpy="${M_PI/2} 0 0"/>
         <geometry>
           <mesh filename="package://motoman_description/meshes/sia20/link_${suffix}/visual.dae"/>
@@ -13,5 +12,4 @@
       </visual>
       <collision>
-        <origin rpy="${M_PI/2} 0 0"/>
         <geometry>
           <mesh filename="package://motoman_description/meshes/sia20/link_${suffix}/collision.stl"/>

Commit message: [update] add inertial params for the link

File: motoman_description/urdf/sia20/link.urdf.xacro (robot description, xacro)
@@ -1,8 +1,13 @@
 <?xml version="1.0"?>
 <robot xmlns:xacro="http://ros.org/wiki/xacro">
-  <xacro:macro name="link_v0" params="suffix
+  <xacro:macro name="link_v1" params="suffix
                                       parent
+                                      mass
+                                      height
+                                      width
+                                      depth
                                       *joint_origin
-                                      *joint_limit">
+                                      *joint_limit
+                                      *inertial_origin">
     <link name="link_${suffix}">
       <visual>
@@ -16,4 +21,9 @@
         </geometry>
       </collision>
+      <inertial>
+        <xacro:box_inertial mass="${mass}" height="${height}" width="${width}" depth="${depth}">
+          <insert_block name="inertial_origin"/>
+        </xacro:box_inertial>
+      </inertial>
     </link>
     <joint name="joint_${suffix}" type="revolute">
