Commit message: [update] mesh models

File: motoman_description/robots/sia20/sia20_basic.urdf.xacro (robot description, xacro)
@@ -53,32 +53,37 @@
   <!-- Link L -->
   <xacro:link_v0 suffix="l" parent="link_s">
-    <origin xyz="0 0 0.298"/>
+    <origin xyz="0 0 0.298" rpy="${M_PI/2} 0 0"/>
     <limit effort="100.0" lower="${joint_l_lower_limit}"
            upper="${joint_l_upper_limit}" velocity="${joint_l_velocity_limit}"/>
   </xacro:link_v0>
-  <!-- <xacro:link_v0 suffix="s" parent="base_link"> -->
-  <!--   <origin xyz="0 0 0.112"/> -->
-  <!--   <limit effort="100.0" lower="${joint_s_lower_limit}" -->
-  <!--          upper="${joint_s_upper_limit}" velocity="${joint_s_velocity_limit}"/> -->
-  <!-- </xacro:link_v0> -->
-  <!-- <xacro:link_v0 suffix="s" parent="base_link"> -->
-  <!--   <origin xyz="0 0 0.112"/> -->
-  <!--   <limit effort="100.0" lower="${joint_s_lower_limit}" -->
-  <!--          upper="${joint_s_upper_limit}" velocity="${joint_s_velocity_limit}"/> -->
-  <!-- </xacro:link_v0> -->
-  <!-- <xacro:link_v0 suffix="s" parent="base_link"> -->
-  <!--   <origin xyz="0 0 0.112"/> -->
-  <!--   <limit effort="100.0" lower="${joint_s_lower_limit}" -->
-  <!--          upper="${joint_s_upper_limit}" velocity="${joint_s_velocity_limit}"/> -->
-  <!-- </xacro:link_v0> -->
-  <!-- <xacro:link_v0 suffix="s" parent="base_link"> -->
-  <!--   <origin xyz="0 0 0.112"/> -->
-  <!--   <limit effort="100.0" lower="${joint_s_lower_limit}" -->
-  <!--          upper="${joint_s_upper_limit}" velocity="${joint_s_velocity_limit}"/> -->
-  <!-- </xacro:link_v0> -->
-  <!-- <xacro:link_v0 suffix="s" parent="base_link"> -->
-  <!--   <origin xyz="0 0 0.112"/> -->
-  <!--   <limit effort="100.0" lower="${joint_s_lower_limit}" -->
-  <!--          upper="${joint_s_upper_limit}" velocity="${joint_s_velocity_limit}"/> -->
-  <!-- </xacro:link_v0> -->
+  <!-- Link E -->
+  <xacro:link_v0 suffix="e" parent="link_l">
+    <origin xyz="0 0.266 0" rpy="${-M_PI/2} 0 0"/>
+    <limit effort="100.0" lower="${joint_e_lower_limit}"
+           upper="${joint_e_upper_limit}" velocity="${joint_e_velocity_limit}"/>
+  </xacro:link_v0>
+  <!-- Link U -->
+  <xacro:link_v0 suffix="u" parent="link_e">
+    <origin xyz="0 0 0.224" rpy="${M_PI/2} 0 0"/>
+    <limit effort="100.0" lower="${joint_u_lower_limit}"
+           upper="${joint_u_upper_limit}" velocity="${joint_u_velocity_limit}"/>
+  </xacro:link_v0>
+  <!-- Link R -->
+  <xacro:link_v0 suffix="r" parent="link_u">
+    <origin xyz="0 0.264 0" rpy="${-M_PI/2} 0 0"/>
+    <limit effort="100.0" lower="${joint_r_lower_limit}"
+           upper="${joint_r_upper_limit}" velocity="${joint_r_velocity_limit}"/>
+  </xacro:link_v0>
+  <!-- Link B -->
+  <xacro:link_v0 suffix="b" parent="link_r">
+    <origin xyz="0 0 0.156" rpy="${M_PI/2} 0 0"/>
+    <limit effort="100.0" lower="${joint_b_lower_limit}"
+           upper="${joint_b_upper_limit}" velocity="${joint_b_velocity_limit}"/>
+  </xacro:link_v0>
+  <!-- Link T -->
+  <xacro:link_v0 suffix="t" parent="link_b">
+    <origin xyz="0 0.167 0" rpy="${-M_PI/2} 0 0"/>
+    <limit effort="100.0" lower="${joint_t_lower_limit}"
+           upper="${joint_t_upper_limit}" velocity="${joint_t_velocity_limit}"/>
+  </xacro:link_v0>
 </robot>

Commit message: [update] add inertial info

File: motoman_description/robots/sia20/sia20_basic.urdf.xacro (robot description, xacro)
@@ -5,28 +5,5 @@
   <xacro:include filename="$(find motoman_description)/urdf/materials.xacro"/>
   <xacro:include filename="$(find motoman_description)/urdf/sia20/link.urdf.xacro" />
-  <!-- Hard ware limits -->
-  <!-- Range limits -->
-  <xacro:property name="joint_s_upper_limit" value="${180*M_PI/180}"/>
-  <xacro:property name="joint_s_lower_limit" value="-${joint_s_upper_limit}"/>
-  <xacro:property name="joint_l_upper_limit" value="${110*M_PI/180}"/>
-  <xacro:property name="joint_l_lower_limit" value="-${joint_l_upper_limit}"/>
-  <xacro:property name="joint_e_upper_limit" value="${170*M_PI/180}"/>
-  <xacro:property name="joint_e_lower_limit" value="-${joint_e_upper_limit}"/>
-  <xacro:property name="joint_u_upper_limit" value="${130*M_PI/180}"/>
-  <xacro:property name="joint_u_lower_limit" value="-${joint_u_upper_limit}"/>
-  <xacro:property name="joint_r_upper_limit" value="${180*M_PI/180}"/>
-  <xacro:property name="joint_r_lower_limit" value="-${joint_r_upper_limit}"/>
-  <xacro:property name="joint_b_upper_limit" value="${110*M_PI/180}"/>
-  <xacro:property name="joint_b_lower_limit" value="-${joint_b_upper_limit}"/>
-  <xacro:property name="joint_t_upper_limit" value="${180*M_PI/180}"/>
-  <xacro:property name="joint_t_lower_limit" value="-${joint_t_upper_limit}"/>
-  <!-- Velocity limits -->
-  <xacro:property name="joint_s_velocity_limit" value="${130*M_PI/180}"/>
-  <xacro:property name="joint_l_velocity_limit" value="${130*M_PI/180}"/>
-  <xacro:property name="joint_e_velocity_limit" value="${170*M_PI/180}"/>
-  <xacro:property name="joint_u_velocity_limit" value="${170*M_PI/180}"/>
-  <xacro:property name="joint_r_velocity_limit" value="${200*M_PI/180}"/>
-  <xacro:property name="joint_b_velocity_limit" value="${200*M_PI/180}"/>
-  <xacro:property name="joint_t_velocity_limit" value="${400*M_PI/180}"/>
+  <xacro:include filename="$(find motoman_description)/robots/sia20/property.xacro"/>
   <!-- Add Link & Joint -->
   <!-- base_link -->
@@ -44,46 +21,65 @@
       </geometry>
     </collision>
+    <inertial>
+      <xacro:box_inertial mass="30" height="0.34" width="0.175" depth="0.28">
+        <origin xyz="0 0 ${0.28/2}" rpy="${M_PI/2} 0 0"/>
+      </xacro:box_inertial>
+    </inertial>
   </link>
   <!-- Link S -->
-  <xacro:link_v0 suffix="s" parent="base_link">
+  <xacro:link_v1 suffix="s" parent="base_link"
+                 mass="20" height="0.22" width="0.22" depth="0.407">
     <origin xyz="0 0 0.112"/>
     <limit effort="100.0" lower="${joint_s_lower_limit}"
            upper="${joint_s_upper_limit}" velocity="${joint_s_velocity_limit}"/>
-  </xacro:link_v0>
+    <origin xyz="0 0 ${0.407/2}"/>
+  </xacro:link_v1>
   <!-- Link L -->
-  <xacro:link_v0 suffix="l" parent="link_s">
+  <xacro:link_v1 suffix="l" parent="link_s"
+                 mass="20" height="0.24" width="0.388" depth="0.206">
     <origin xyz="0 0 0.298" rpy="${M_PI/2} 0 0"/>
     <limit effort="100.0" lower="${joint_l_lower_limit}"
            upper="${joint_l_upper_limit}" velocity="${joint_l_velocity_limit}"/>
-  </xacro:link_v0>
+    <origin xyz="0 ${0.388/4} 0"/>
+  </xacro:link_v1>
   <!-- Link E -->
-  <xacro:link_v0 suffix="e" parent="link_l">
+  <xacro:link_v1 suffix="e" parent="link_l"
+                 mass="15" height="0.18" width="0.195" depth="0.327">
     <origin xyz="0 0.266 0" rpy="${-M_PI/2} 0 0"/>
     <limit effort="100.0" lower="${joint_e_lower_limit}"
            upper="${joint_e_upper_limit}" velocity="${joint_e_velocity_limit}"/>
-  </xacro:link_v0>
+    <origin xyz="0 0 ${0.327/2}"/>
+  </xacro:link_v1>
   <!-- Link U -->
-  <xacro:link_v0 suffix="u" parent="link_e">
+  <xacro:link_v1 suffix="u" parent="link_e"
+                 mass="15" height="0.18" width="0.355" depth="0.16">
     <origin xyz="0 0 0.224" rpy="${M_PI/2} 0 0"/>
     <limit effort="100.0" lower="${joint_u_lower_limit}"
            upper="${joint_u_upper_limit}" velocity="${joint_u_velocity_limit}"/>
-  </xacro:link_v0>
+    <origin xyz="0 ${0.355/4} 0"/>
+  </xacro:link_v1>
   <!-- Link R -->
-  <xacro:link_v0 suffix="r" parent="link_u">
+  <xacro:link_v1 suffix="r" parent="link_u"
+                 mass="7.5" height="0.14" width="0.153" depth="0.247">
     <origin xyz="0 0.264 0" rpy="${-M_PI/2} 0 0"/>
     <limit effort="100.0" lower="${joint_r_lower_limit}"
            upper="${joint_r_upper_limit}" velocity="${joint_r_velocity_limit}"/>
-  </xacro:link_v0>
+    <origin xyz="0 0 ${0.247/2}"/>
+  </xacro:link_v1>
   <!-- Link B -->
-  <xacro:link_v0 suffix="b" parent="link_r">
+  <xacro:link_v1 suffix="b" parent="link_r"
+                 mass="7.5" height="0.14" width="0.237" depth="0.146">
     <origin xyz="0 0 0.156" rpy="${M_PI/2} 0 0"/>
     <limit effort="100.0" lower="${joint_b_lower_limit}"
            upper="${joint_b_upper_limit}" velocity="${joint_b_velocity_limit}"/>
-  </xacro:link_v0>
+    <origin xyz="0 ${0.237/4} 0"/>
+  </xacro:link_v1>
   <!-- Link T -->
-  <xacro:link_v0 suffix="t" parent="link_b">
+  <xacro:link_v1 suffix="t" parent="link_b"
+                 mass="5" height="0.0998" width="0.0998" depth="0.0158">
     <origin xyz="0 0.167 0" rpy="${-M_PI/2} 0 0"/>
     <limit effort="100.0" lower="${joint_t_lower_limit}"
            upper="${joint_t_upper_limit}" velocity="${joint_t_velocity_limit}"/>
-  </xacro:link_v0>
+    <origin xyz="0 0 ${0.0158/2}"/>
+  </xacro:link_v1>
 </robot>

Commit message: [update] to use macros

File: motoman_description/robots/sia20/sia20_basic.urdf.xacro (robot description, xacro)
@@ -4,27 +4,10 @@
   <xacro:include filename="$(find motoman_description)/urdf/common.xacro" />
   <xacro:include filename="$(find motoman_description)/urdf/materials.xacro"/>
-  <xacro:include filename="$(find motoman_description)/urdf/sia20/link.urdf.xacro" />
+  <xacro:include filename="$(find motoman_description)/urdf/sia20/base_link/base_link.urdf.xacro" />
+  <xacro:include filename="$(find motoman_description)/urdf/sia20/link/link.urdf.xacro" />
   <xacro:include filename="$(find motoman_description)/robots/sia20/property.xacro"/>
   <!-- Add Link & Joint -->
   <!-- base_link -->
-  <link name="base_link">
-    <visual>
-      <origin rpy="${M_PI/2} 0 0"/>
-      <geometry>
-        <mesh filename="package://motoman_description/meshes/sia20/base_link/visual.dae"/>
-      </geometry>
-    </visual>
-    <collision>
-      <origin rpy="${M_PI/2} 0 0"/>
-      <geometry>
-        <mesh filename="package://motoman_description/meshes/sia20/base_link/collision.stl"/>
-      </geometry>
-    </collision>
-    <inertial>
-      <xacro:box_inertial mass="30" height="0.34" width="0.175" depth="0.28">
-        <origin xyz="0 0 ${0.28/2}" rpy="${M_PI/2} 0 0"/>
-      </xacro:box_inertial>
-    </inertial>
-  </link>
+  <xacro:base_link_v0/>
   <!-- Link S -->
   <xacro:link_v1 suffix="s" parent="base_link"

Commit message: [update] add tool0 link

File: motoman_description/robots/sia20/sia20_basic.urdf.xacro (robot description, xacro)
@@ -66,4 +66,11 @@
     <origin xyz="0 0 ${0.0158/2}"/>
   </xacro:link_v1>
+  <!-- Tool Link -->
+  <link name="tool0"/>
+  <joint name="joint_tool0" type="fixed">
+    <origin xyz="0 0 0.01286" rpy="0 ${-M_PI/2} 0"/>
+    <parent link="link_t"/>
+    <child link="tool0"/>
+  </joint>
   <!-- Add Gazebo plugin -->
   <gazebo>
