Commit message: Add CAD files

File: motoman_description/urdf/motomini/body.urdf.xacro (robot description, xacro)
@@ -5,5 +5,5 @@
       <visual>
         <geometry>
-          <mesh filename="package://motoman_motomini_support/meshes/motomini/visual/${link_name}.stl"/>
+          <mesh filename="package://motoman_description/meshes/motomini/visual/${link_name}.stl"/>
         </geometry>
         <material name="yaskawa_blue"/>
@@ -11,5 +11,5 @@
       <collision>
         <geometry>
-          <mesh filename="package://motoman_motomini_support/meshes/motomini/collision/${link_name}.stl"/>
+          <mesh filename="package://motoman_description/meshes/motomini/collision/${link_name}.stl"/>
         </geometry>
       </collision>
