Commit message: Fix gazebo config for motomini

File: motoman_description/robots/motomini/motomini.xacro (robot description, xacro)
@@ -4,3 +4,6 @@
   <xacro:include filename="$(find motoman_description)/robots/motomini/motomini_basic.urdf.xacro" />
   <xacro:motoman_motomini prefix=""/>
+  <xacro:add_world>
+    <origin xyz="0 0 0" rpy="0 0 0"/>
+  </xacro:add_world>
 </robot>

File: motoman_description/robots/motomini/motomini_basic.urdf.xacro (robot description, xacro)
@@ -1,4 +1,4 @@
 <?xml version="1.0" ?>
-<robot xmlns:xacro="http://ros.org/wiki/xacro">
+<robot name="motomini" xmlns:xacro="http://ros.org/wiki/xacro">
   <!-- File Include -->
   <xacro:include filename="$(find motoman_description)/urdf/common.xacro"/>
@@ -9,4 +9,5 @@
   <!-- Configuration -->
   <xacro:macro name="motoman_motomini" params="prefix">
+    <property name="whole_mass" value="7.00" />
     <property name="base_link_volume" value="0.00030" />
     <property name="link_1_s_volume"  value="0.00030" />
@@ -20,25 +21,44 @@
                                        + link_3_u_volume  + link_4_r_volume
                                        + link_5_b_volume  + link_6_t_volume}" />
+    <!-- Add macro -->
+    <xacro:macro name="add_world" params="*origin">
+      <link name="world"/>
+      <joint name="world" type="fixed">
+        <insert_block name="origin"/>
+        <parent link="world"/>
+        <child link="base_link"/>
+      </joint>
+    </xacro:macro>
     <!-- link list -->
-    <!--xacro:link_v0 link_name="${prefix}base_link" color="yaskawa_blue" /-->
-    <xacro:link_box_v0 link_name="${prefix}base_link" mass="${base_link_volume/sum_volume}"
+    <!--
+    <xacro:link_v0 link_name="${prefix}base_link" color="yaskawa_blue" />
+    <xacro:link_v0 link_name="${prefix}link_1_s" color="yaskawa_blue" />
+    <xacro:link_v0 link_name="${prefix}link_2_l" color="yaskawa_blue" />
+    <xacro:link_v0 link_name="${prefix}link_3_u" color="yaskawa_blue" />
+    <xacro:link_v0 link_name="${prefix}link_4_r" color="yaskawa_blue" />
+    <xacro:link_v0 link_name="${prefix}link_5_b" color="yaskawa_blue" />
+    <xacro:link_v0 link_name="${prefix}link_6_t" color="yaskawa_blue" />
+    -->
+    <!--
+    -->
+    <xacro:link_box_v0 link_name="${prefix}base_link" mass="${whole_mass*base_link_volume/sum_volume}"
         width="0.124" depth="0.2246" height="0.1005"
         origin_xyz="0 0 0" origin_rpy="0 0 0" color="yaskawa_blue" />
-    <xacro:link_box_v0 link_name="${prefix}link_1_s" mass="${link_1_s_volume/sum_volume}"
+    <xacro:link_box_v0 link_name="${prefix}link_1_s" mass="${whole_mass*link_1_s_volume/sum_volume}"
         width="0.119" depth="0.1205" height="0.1435"
         origin_xyz="0 0 0" origin_rpy="0 0 0" color="yaskawa_blue"/>
-    <xacro:link_box_v0 link_name="${prefix}link_2_l" mass="${link_2_l_volume/sum_volume}"
+    <xacro:link_box_v0 link_name="${prefix}link_2_l" mass="${whole_mass*link_2_l_volume/sum_volume}"
         width="0.1072" depth="0.2430" height="0.1338"
         origin_xyz="0 0 0" origin_rpy="0 0 0" color="yaskawa_blue"/>
-    <xacro:link_box_v0 link_name="${prefix}link_3_u" mass="${link_3_u_volume/sum_volume}"
+    <xacro:link_box_v0 link_name="${prefix}link_3_u" mass="${whole_mass*link_3_u_volume/sum_volume}"
         width="0.0730" depth="0.1078" height="0.0855"
         origin_xyz="0 0 0" origin_rpy="0 0 0" color="yaskawa_blue"/>
-    <xacro:link_box_v0 link_name="${prefix}link_4_r" mass="${link_4_r_volume/sum_volume}"
+    <xacro:link_box_v0 link_name="${prefix}link_4_r" mass="${whole_mass*link_4_r_volume/sum_volume}"
         width="0.0943" depth="0.0930" height="0.1885"
         origin_xyz="0 0 0" origin_rpy="0 0 0" color="yaskawa_blue"/>
-    <xacro:link_box_v0 link_name="${prefix}link_5_b" mass="${link_5_b_volume/sum_volume}"
+    <xacro:link_box_v0 link_name="${prefix}link_5_b" mass="${whole_mass*link_5_b_volume/sum_volume}"
         width="0.0700" depth="0.0797" height="0.0571"
         origin_xyz="0 0 0" origin_rpy="0 0 0" color="yaskawa_blue"/>
-    <xacro:link_box_v0 link_name="${prefix}link_6_t" mass="${link_6_t_volume/sum_volume}"
+    <xacro:link_box_v0 link_name="${prefix}link_6_t" mass="${whole_mass*link_6_t_volume/sum_volume}"
         width="0.0300" depth="0.0300" height="0.0190"
         origin_xyz="0 0 0" origin_rpy="0 0 0" color="yaskawa_blue"/>
@@ -83,40 +103,36 @@
       <child link="base"/>
     </joint>
-  <!-- transmission -->
-  <xacro:simple_jp_trans_v0 name="transmission_s"
-                            joint_name="joint_s" actuator_name="motor_s"
-                            reduction="300"/>
-  <xacro:simple_jp_trans_v0 name="transmission_l"
-                            joint_name="joint_l" actuator_name="motor_l"
-                            reduction="300"/>
-  <xacro:simple_jp_trans_v0 name="transmission_e"
-                            joint_name="joint_e" actuator_name="motor_e"
-                            reduction="100"/>
-  <xacro:simple_jp_trans_v0 name="transmission_u"
-                            joint_name="joint_u" actuator_name="motor_u"
-                            reduction="50"/>
-  <xacro:simple_jp_trans_v0 name="transmission_r"
-                            joint_name="joint_r" actuator_name="motor_r"
-                            reduction="30"/>
-  <xacro:simple_jp_trans_v0 name="transmission_b"
-                            joint_name="joint_b" actuator_name="motor_b"
-                            reduction="30"/>
-  <xacro:simple_jp_trans_v0 name="transmission_t"
-                            joint_name="joint_t" actuator_name="motor_t"
-                            reduction="10"/>
-  <!-- gazebo -->
-  <gazebo>
-    <plugin name="gazebo_ros_control" filename="libgazebo_ros_control.so">
-      <robotSimType>gazebo_ros_control/DefaultRobotHWSim</robotSimType>
-    </plugin>
-  </gazebo>
-  <xacro:gazebo_link_v1 name="base_link"/>
-  <xacro:gazebo_link_v1 name="link_s"/>
-  <xacro:gazebo_link_v1 name="link_l"/>
-  <xacro:gazebo_link_v1 name="link_e"/>
-  <xacro:gazebo_link_v1 name="link_u"/>
-  <xacro:gazebo_link_v1 name="link_r"/>
-  <xacro:gazebo_link_v1 name="link_b"/>
-  <xacro:gazebo_link_v1 name="link_t"/>
+    <!-- transmission -->
+    <xacro:simple_jp_trans_v0 name="transmission_1_s"
+                              joint_name="${prefix}joint_1_s" actuator_name="${prefix}motor_1_s"
+                              reduction="300"/>
+    <xacro:simple_jp_trans_v0 name="transmission_2_l"
+                              joint_name="${prefix}joint_2_l" actuator_name="${prefix}motor_2_l"
+                              reduction="300"/>
+    <xacro:simple_jp_trans_v0 name="transmission_3_u"
+                              joint_name="${prefix}joint_3_u" actuator_name="${prefix}motor_3_u"
+                              reduction="50"/>
+    <xacro:simple_jp_trans_v0 name="transmission_4_r"
+                              joint_name="${prefix}joint_4_r" actuator_name="${prefix}motor_4_r"
+                              reduction="30"/>
+    <xacro:simple_jp_trans_v0 name="transmission_5_b"
+                              joint_name="${prefix}joint_5_b" actuator_name="${prefix}motor_5_b"
+                              reduction="30"/>
+    <xacro:simple_jp_trans_v0 name="transmission_6_t"
+                              joint_name="${prefix}joint_6_t" actuator_name="${prefix}motor_6_t"
+                              reduction="10"/>
+    <!-- gazebo -->
+    <gazebo>
+      <plugin name="gazebo_ros_control" filename="libgazebo_ros_control.so">
+        <robotSimType>gazebo_ros_control/DefaultRobotHWSim</robotSimType>
+      </plugin>
+    </gazebo>
+    <xacro:gazebo_link_v1 name="${prefix}base_link"/>
+    <xacro:gazebo_link_v1 name="${prefix}link_1_s"/>
+    <xacro:gazebo_link_v1 name="${prefix}link_2_l"/>
+    <xacro:gazebo_link_v1 name="${prefix}link_3_u"/>
+    <xacro:gazebo_link_v1 name="${prefix}link_4_r"/>
+    <xacro:gazebo_link_v1 name="${prefix}link_5_b"/>
+    <xacro:gazebo_link_v1 name="${prefix}link_6_t"/>
   </xacro:macro>
 </robot>

File: motoman_description/urdf/motomini/body.gazebo.xacro (robot description, xacro)
@@ -6,4 +6,5 @@
       <mu2>0.2</mu2>
       <selfCollide>true</selfCollide>
+      <material>Gazebo/Blue</material>
     </gazebo>
   </xacro:macro>

File: motoman_description/urdf/motomini/body.transmission.xacro (robot description, xacro)
@@ -7,8 +7,8 @@
       <type>transmission_interface/SimpleTransmission</type>
       <joint name="${joint_name}">
-      <hardwareInterface>PositionJointInterface</hardwareInterface>
+        <hardwareInterface>hardware_interface/PositionJointInterface</hardwareInterface>
       </joint>
       <actuator name="${actuator_name}">
-      <hardwareInterface>PositionJointInterface</hardwareInterface>
+      <hardwareInterface>hardware_interface/PositionJointInterface</hardwareInterface>
       <mechanicalReduction>${reduction}</mechanicalReduction>
       </actuator>

Commit message: [fix] z offset

File: motoman_description/robots/motomini/motomini.xacro (robot description, xacro)
@@ -5,5 +5,5 @@
   <xacro:motoman_motomini prefix=""/>
   <xacro:add_world>
-    <origin xyz="0 0 0" rpy="0 0 0"/>
+    <origin xyz="0 0 0.067" rpy="0 0 0"/>
   </xacro:add_world>
 </robot>
