Commit message: Modify misc config

File: motoman_description/robots/motomini/motomini_with_gripper_kinectv2.urdf.xacro (robot description, xacro)
@@ -1,4 +1,4 @@
 <?xml version="1.0"?>
-<robot name="sia5" xmlns:xacro="http://ros.org/wiki/xacro">
+<robot name="motoman_motomini" xmlns:xacro="http://ros.org/wiki/xacro">
   <!-- File Include -->
   <xacro:include filename="$(find motoman_description)/urdf/sensor/kinect.urdf.xacro"/>
@@ -8,5 +8,5 @@
   <!-- add gripper -->
   <xacro:gripper name="gripper" parent="tool0">
-    <origin xyz="0 0 0.03" rpy="0 0 0" />
+    <origin xyz="0 0 0.035" rpy="0 0 0" />
   </xacro:gripper>
   <!-- add Kinect V2 -->

File: motoman_description/robots/motomini/motomini_with_kinectv2.urdf.xacro (robot description, xacro)
@@ -1,4 +1,4 @@
 <?xml version="1.0"?>
-<robot name="sia5" xmlns:xacro="http://ros.org/wiki/xacro">
+<robot name="motoman_motomini" xmlns:xacro="http://ros.org/wiki/xacro">
   <!-- File Include -->
   <xacro:include filename="$(find motoman_description)/urdf/sensor/kinect.urdf.xacro"/>
