Commit message: Fix indent

File: motoman_description/urdf/tool/gripper.urdf.xacro (robot description, xacro)
@@ -4,98 +4,98 @@
        xmlns:interface="http://playerstage.sourceforge.net/gazebo/xmlschema/#interface"
        xmlns:xacro="http://ros.org/wiki/xacro">
-	<xacro:include filename="$(find motoman_description)/urdf/tool/gripper.gazebo.xacro" />
-	<xacro:include filename="$(find motoman_description)/urdf/tool/gripper.transmission.xacro" />
-	<xacro:include filename="$(find motoman_description)/urdf/tool/limits.urdf.xacro" />
-	<xacro:macro name="gripper" params="parent name *origin">
-		<!-- joint between arm_7_link and sdh_palm_link -->
-		<joint name="${name}_palm_joint" type="fixed" >
-			<insert_block name="origin" />
-			<parent link="${parent}" />
-			<child link="${name}_palm_link" />
-		</joint>
-		<link name="${name}_palm_link">
-			<inertial>
-				<origin xyz="0 0 0" rpy="0 0 0"/>
-				<mass value="0.1"/>
-				<inertia ixx="0.01" ixy="0" ixz="0" iyy="0.01" iyz="0" izz="0.01" />
-			</inertial>
-			<visual>
-				<origin xyz="0 0 0" rpy="0 0 0" />
-				<geometry>
-					<mesh filename="package://motoman_description/meshes/tool/palm.dae" />
-				</geometry>
-				<material name="Black" />
-			</visual>
-			<collision>
-				<origin xyz="0 0 0" rpy="0 0 0" />
-				<geometry>
-					<!--<box size="0.050 0.094 0.054"/>-->
-					<mesh filename="package://motoman_description/meshes/tool/palm_convex.dae" />
-				</geometry>
-			</collision>
-		</link>
-		<joint name="${name}_finger_joint_l" type="prismatic">
-			<origin xyz="0.004 0.008 0.046" rpy="0 0 ${M_PI}" />
-			<parent link="${name}_palm_link"/>
-			<child link="${name}_finger_link_l"/>
-			<axis xyz="0 -1 0" />
-			<dynamics damping="1.0" friction="1.0" />
-			<limit effort="2" velocity="0.1" lower="0" upper="${finger_joint}"/>
-                        <safety_controller k_position="20" k_velocity="25" soft_lower_limit="${threshold}" soft_upper_limit="${finger_joint_soft}" />
-		</joint>
-		<link name="${name}_finger_link_l">
-			<inertial>
-				<origin xyz="0 -0.001 0" rpy="0 0 0" />
-				<mass value="0.01"/>
-				<inertia ixx="0.01" ixy="0" ixz="0" iyy="0.01" iyz="0" izz="0.01" />
-			</inertial>
-			<visual>
-				<origin xyz="0 0 0" rpy="0 0 0" />
-				<geometry>
-					<mesh filename="package://motoman_description/meshes/tool/finger.dae" />
-				</geometry>
-				<material name="Black" />
-			</visual>
-			<collision>
-				<origin xyz="0 0 0" rpy="0 0 0" />
-				<geometry>
-					<!--<box size="0.014 0.020 0.046"/>-->
-					<mesh filename="package://motoman_description/meshes/tool/finger_convex.dae" />
-				</geometry>
-			</collision>
-		</link>
-               <joint name="${name}_finger_joint_r" type="prismatic">
-			<origin xyz="0.004 -0.008 0.046" rpy="0 0 0" />
-			<parent link="${name}_palm_link"/>
-			<child link="${name}_finger_link_r"/>
-			<axis xyz="0 -1 0" />
-			<dynamics damping="1.0" friction="1.0" />
-			<limit effort="2" velocity="0.1" lower="0" upper="${finger_joint}"/>
-                        <safety_controller k_position="20" k_velocity="25" soft_lower_limit="${threshold}" soft_upper_limit="${finger_joint_soft}" />
-		</joint>
-		<link name="${name}_finger_link_r">
-			<inertial>
-				<origin xyz="0.000 -0.001 0" rpy="0 0 0" />
-				<mass value="0.01"/>
-				<inertia ixx="0.01" ixy="0" ixz="0" iyy="0.01" iyz="0" izz="0.01" />
-			</inertial>
-			<visual>
-				<origin xyz="0 0 0" rpy="0 0 0" />
-				<geometry>
-					<mesh filename="package://motoman_description/meshes/tool/finger.dae" />
-				</geometry>
-				<material name="Black" />
-			</visual>
-			<collision>
-				<origin xyz="0.000 0 0" rpy="0 0 0" />
-				<geometry>
-					<!--<box size="0.014 0.020 0.046"/>-->
-					<mesh filename="package://motoman_description/meshes/tool/finger_convex.dae" />
-				</geometry>
-			</collision>
-		</link>
-		<!-- extensions -->
-		<xacro:gripper_gazebo name="${name}" />
-		<xacro:gripper_transmission name="${name}" />
-	</xacro:macro>
+  <xacro:include filename="$(find motoman_description)/urdf/tool/gripper.gazebo.xacro" />
+  <xacro:include filename="$(find motoman_description)/urdf/tool/gripper.transmission.xacro" />
+  <xacro:include filename="$(find motoman_description)/urdf/tool/limits.urdf.xacro" />
+  <xacro:macro name="gripper" params="parent name *origin">
+    <!-- joint between arm_7_link and sdh_palm_link -->
+    <joint name="${name}_palm_joint" type="fixed" >
+      <insert_block name="origin" />
+      <parent link="${parent}" />
+      <child link="${name}_palm_link" />
+    </joint>
+    <link name="${name}_palm_link">
+      <inertial>
+        <origin xyz="0 0 0" rpy="0 0 0"/>
+        <mass value="0.1"/>
+        <inertia ixx="0.01" ixy="0" ixz="0" iyy="0.01" iyz="0" izz="0.01" />
+      </inertial>
+      <visual>
+        <origin xyz="0 0 0" rpy="0 0 0" />
+        <geometry>
+          <mesh filename="package://motoman_description/meshes/tool/palm.dae" />
+        </geometry>
+        <material name="Black" />
+      </visual>
+      <collision>
+        <origin xyz="0 0 0" rpy="0 0 0" />
+        <geometry>
+          <!--<box size="0.050 0.094 0.054"/>-->
+          <mesh filename="package://motoman_description/meshes/tool/palm_convex.dae" />
+        </geometry>
+      </collision>
+    </link>
+    <joint name="${name}_finger_joint_l" type="prismatic">
+      <origin xyz="0.004 0.008 0.046" rpy="0 0 ${M_PI}" />
+      <parent link="${name}_palm_link"/>
+      <child link="${name}_finger_link_l"/>
+      <axis xyz="0 -1 0" />
+      <dynamics damping="1.0" friction="1.0" />
+      <limit effort="2" velocity="0.1" lower="0" upper="${finger_joint}"/>
+      <safety_controller k_position="20" k_velocity="25" soft_lower_limit="${threshold}" soft_upper_limit="${finger_joint_soft}" />
+    </joint>
+    <link name="${name}_finger_link_l">
+      <inertial>
+        <origin xyz="0 -0.001 0" rpy="0 0 0" />
+        <mass value="0.01"/>
+        <inertia ixx="0.01" ixy="0" ixz="0" iyy="0.01" iyz="0" izz="0.01" />
+      </inertial>
+      <visual>
+        <origin xyz="0 0 0" rpy="0 0 0" />
+        <geometry>
+          <mesh filename="package://motoman_description/meshes/tool/finger.dae" />
+        </geometry>
+        <material name="Black" />
+      </visual>
+      <collision>
+        <origin xyz="0 0 0" rpy="0 0 0" />
+        <geometry>
+          <!--<box size="0.014 0.020 0.046"/>-->
+          <mesh filename="package://motoman_description/meshes/tool/finger_convex.dae" />
+        </geometry>
+      </collision>
+    </link>
+    <joint name="${name}_finger_joint_r" type="prismatic">
+      <origin xyz="0.004 -0.008 0.046" rpy="0 0 0" />
+      <parent link="${name}_palm_link"/>
+      <child link="${name}_finger_link_r"/>
+      <axis xyz="0 -1 0" />
+      <dynamics damping="1.0" friction="1.0" />
+      <limit effort="2" velocity="0.1" lower="0" upper="${finger_joint}"/>
+      <safety_controller k_position="20" k_velocity="25" soft_lower_limit="${threshold}" soft_upper_limit="${finger_joint_soft}" />
+    </joint>
+    <link name="${name}_finger_link_r">
+      <inertial>
+        <origin xyz="0.000 -0.001 0" rpy="0 0 0" />
+        <mass value="0.01"/>
+        <inertia ixx="0.01" ixy="0" ixz="0" iyy="0.01" iyz="0" izz="0.01" />
+      </inertial>
+      <visual>
+        <origin xyz="0 0 0" rpy="0 0 0" />
+        <geometry>
+          <mesh filename="package://motoman_description/meshes/tool/finger.dae" />
+        </geometry>
+        <material name="Black" />
+      </visual>
+      <collision>
+        <origin xyz="0.000 0 0" rpy="0 0 0" />
+        <geometry>
+          <!--<box size="0.014 0.020 0.046"/>-->
+          <mesh filename="package://motoman_description/meshes/tool/finger_convex.dae" />
+        </geometry>
+      </collision>
+    </link>
+    <!-- extensions -->
+    <xacro:gripper_gazebo name="${name}" />
+    <xacro:gripper_transmission name="${name}" />
+  </xacro:macro>
 </robot>
