Commit message: Fix indent

File: motoman_description/urdf/tool/gripper.gazebo.xacro (robot description, xacro)
@@ -4,26 +4,26 @@
        xmlns:interface="http://playerstage.sourceforge.net/gazebo/xmlschema/#interface"
        xmlns:xacro="http://ros.org/wiki/xacro">
-	<xacro:macro name="gripper_gazebo" params="name">
-		<gazebo reference="${name}_palm_link">
-			<material>Gazebo/Black</material>
-			<turnGravityOff>false</turnGravityOff>
-			<selfCollide>true</selfCollide>
-		</gazebo>
-		<gazebo reference="${name}_finger_l_link">
-			<material>Gazebo/Black</material>
-			<turnGravityOff>false</turnGravityOff>
-			<selfCollide>true</selfCollide>
+  <xacro:macro name="gripper_gazebo" params="name">
+    <gazebo reference="${name}_palm_link">
+      <material>Gazebo/Black</material>
+      <turnGravityOff>false</turnGravityOff>
+      <selfCollide>true</selfCollide>
+    </gazebo>
+    <gazebo reference="${name}_finger_l_link">
+      <material>Gazebo/Black</material>
+      <turnGravityOff>false</turnGravityOff>
+      <selfCollide>true</selfCollide>
       <mu1>1.0</mu1>
       <mu2>1.0</mu2>
       <maxContacts>100</maxContacts>
-		</gazebo>
-		<gazebo reference="${name}_finger_r_link">
-			<material>Gazebo/Black</material>
-			<turnGravityOff>false</turnGravityOff>
-			<selfCollide>true</selfCollide>
+    </gazebo>
+    <gazebo reference="${name}_finger_r_link">
+      <material>Gazebo/Black</material>
+      <turnGravityOff>false</turnGravityOff>
+      <selfCollide>true</selfCollide>
       <mu1>1.0</mu1>
       <mu2>1.0</mu2>
       <maxContacts>100</maxContacts>
-		</gazebo>
-	</xacro:macro>
+    </gazebo>
+  </xacro:macro>
 </robot>

File: motoman_description/urdf/tool/gripper.transmission.xacro (robot description, xacro)
@@ -4,25 +4,25 @@
        xmlns:interface="http://playerstage.sourceforge.net/gazebo/xmlschema/#interface"
        xmlns:xacro="http://ros.org/wiki/xacro">
-	<xacro:macro name="gripper_transmission" params="name">
-		<transmission name="${name}_finger_l_trans">
+  <xacro:macro name="gripper_transmission" params="name">
+    <transmission name="${name}_finger_l_trans">
       <type>transmission_interface/SimpleTransmission</type>
-			<actuator name="${name}_finger_l_motor">
+      <actuator name="${name}_finger_l_motor">
         <hardwareInterface>EffortJointInterface</hardwareInterface>
         <mechanicalReduction>1</mechanicalReduction>
       </actuator>
-			<joint name="${name}_finger_joint_l">
+      <joint name="${name}_finger_joint_l">
         <hardwareInterface>EffortJointInterface</hardwareInterface>
       </joint>
-		</transmission>
-		<transmission name="${name}_finger_r_trans">
+    </transmission>
+    <transmission name="${name}_finger_r_trans">
       <type>transmission_interface/SimpleTransmission</type>
-			<actuator name="${name}_finger_r_motor">
+      <actuator name="${name}_finger_r_motor">
         <hardwareInterface>EffortJointInterface</hardwareInterface>
         <mechanicalReduction>1</mechanicalReduction>
       </actuator>
-			<joint name="${name}_finger_joint_r">
+      <joint name="${name}_finger_joint_r">
         <hardwareInterface>EffortJointInterface</hardwareInterface>
       </joint>
-		</transmission>
-	</xacro:macro>
+    </transmission>
+  </xacro:macro>
 </robot>

File: motoman_description/urdf/tool/limits.urdf.xacro (robot description, xacro)
@@ -1,11 +1,11 @@
 <?xml version="1.0"?>
 <robot>
-	<!-- common properties -->
-	<property name="M_PI" value="3.1415926535897931" />
-        <property name="threshold" value="0.001" />
-	<!-- fingers limits, values are in meters -->
-	<!--cs:  <property name="finger_joint" value="${0.023 / 2.0}" />	-->
-	<!--cs:  <property name="finger_joint_soft" value="${(0.023 - threshold) / 2.0}" />	  -->
+  <!-- common properties -->
+  <property name="M_PI" value="3.1415926535897931" />
+  <property name="threshold" value="0.001" />
+  <!-- fingers limits, values are in meters -->
+  <!--cs:  <property name="finger_joint" value="${0.023 / 2.0}" />	-->
+  <!--cs:  <property name="finger_joint_soft" value="${(0.023 - threshold) / 2.0}" />	  -->
   <property name="finger_joint" value="${0.06 / 2.0}" />
-	<property name="finger_joint_soft" value="${(0.06 - threshold) / 2.0}" />
+  <property name="finger_joint_soft" value="${(0.06 - threshold) / 2.0}" />
 </robot>
