Commit message: Modify transmission config for motomini

File: motoman_description/urdf/tool/gripper.transmission.xacro (robot description, xacro)
@@ -4,25 +4,25 @@
        xmlns:interface="http://playerstage.sourceforge.net/gazebo/xmlschema/#interface"
        xmlns:xacro="http://ros.org/wiki/xacro">
-	<xacro:macro name="gripper_transmission" params="name">
-		<transmission name="${name}_finger_l_trans">
+  <xacro:macro name="gripper_transmission" params="name">
+    <transmission name="${name}_finger_l_trans">
       <type>transmission_interface/SimpleTransmission</type>
-			<actuator name="${name}_finger_l_motor">
-        <hardwareInterface>EffortJointInterface</hardwareInterface>
+      <actuator name="${name}_finger_l_motor">
+        <hardwareInterface>hardware_interface/EffortJointInterface</hardwareInterface>
         <mechanicalReduction>1</mechanicalReduction>
       </actuator>
-			<joint name="${name}_finger_joint_l">
-        <hardwareInterface>EffortJointInterface</hardwareInterface>
+      <joint name="${name}_finger_joint_l">
+        <hardwareInterface>hardware_interface/EffortJointInterface</hardwareInterface>
       </joint>
-		</transmission>
-		<transmission name="${name}_finger_r_trans">
+    </transmission>
+    <transmission name="${name}_finger_r_trans">
       <type>transmission_interface/SimpleTransmission</type>
-			<actuator name="${name}_finger_r_motor">
-        <hardwareInterface>EffortJointInterface</hardwareInterface>
+      <actuator name="${name}_finger_r_motor">
+        <hardwareInterface>hardware_interface/EffortJointInterface</hardwareInterface>
         <mechanicalReduction>1</mechanicalReduction>
       </actuator>
-			<joint name="${name}_finger_joint_r">
-        <hardwareInterface>EffortJointInterface</hardwareInterface>
+      <joint name="${name}_finger_joint_r">
+        <hardwareInterface>hardware_interface/EffortJointInterface</hardwareInterface>
       </joint>
-		</transmission>
-	</xacro:macro>
+    </transmission>
+  </xacro:macro>
 </robot>
