Commit message: Modify mass

File: motoman_description/robots/hc10dt/hc10dt_basic.urdf.xacro (robot description, xacro)
@@ -51,8 +51,8 @@
       <origin xyz="0 0 0.167" rpy="0 0 0"/>
       <axis xyz="0 0 1"/>
-      <limit effort="30.0" lower="${joint_s_lower_limit}" upper="${joint_s_upper_limit}" velocity="${joint_s_velocity_limit}"/>
+      <limit effort="100.0" lower="${joint_s_lower_limit}" upper="${joint_s_upper_limit}" velocity="${joint_s_velocity_limit}"/>
     </xacro:link_v1>
     <xacro:link_v1 name="link_l"
-                   mass="9.260846"
+                   mass="14.232"
                    parent_link_name="link_s" child_link_name="link_l" joint_name="joint_l">
       <inertia ixx="2.518" ixy="0.000" ixz="0.000"
@@ -61,8 +61,8 @@
       <origin xyz="0 -0.107 0.108" rpy="${M_PI/2} 0 0"/>
       <axis xyz="0 0 1"/>
-      <limit effort="30.0" lower="${joint_l_lower_limit}" upper="${joint_l_upper_limit}" velocity="${joint_l_velocity_limit}"/>
+      <limit effort="100.0" lower="${joint_l_lower_limit}" upper="${joint_l_upper_limit}" velocity="${joint_l_velocity_limit}"/>
     </xacro:link_v1>
     <xacro:link_v1 name="link_u"
-                   mass="9.260846"
+                   mass="5.964"
                    parent_link_name="link_l" child_link_name="link_u" joint_name="joint_u">
       <inertia ixx="0.070" ixy="0.001" ixz="-0.004"
@@ -71,8 +71,8 @@
       <origin xyz="0 0.7 -0.01" rpy="0 0 0"/>
       <axis xyz="0 0 1"/>
-      <limit effort="30.0" lower="${joint_u_lower_limit}" upper="${joint_u_upper_limit}" velocity="${joint_u_velocity_limit}"/>
+      <limit effort="100.0" lower="${joint_u_lower_limit}" upper="${joint_u_upper_limit}" velocity="${joint_u_velocity_limit}"/>
     </xacro:link_v1>
     <xacro:link_v1 name="link_r"
-                   mass="9.260846"
+                   mass="4.849"
                    parent_link_name="link_u" child_link_name="link_r" joint_name="joint_r">
       <inertia ixx="0.347" ixy="0.000" ixz="0.000"
@@ -81,8 +81,8 @@
       <origin xyz="0 -0.106 -0.097" rpy="-${M_PI/2} 0 0"/>
       <axis xyz="0 0 1"/>
-      <limit effort="30.0" lower="${joint_r_lower_limit}" upper="${joint_r_upper_limit}" velocity="${joint_r_velocity_limit}"/>
+      <limit effort="100.0" lower="${joint_r_lower_limit}" upper="${joint_r_upper_limit}" velocity="${joint_r_velocity_limit}"/>
     </xacro:link_v1>
       <xacro:link_v1 name="link_b"
-                   mass="9.260846"
+                   mass="5.454"
                    parent_link_name="link_r" child_link_name="link_b" joint_name="joint_b">
       <inertia ixx="0.074" ixy="0.060" ixz="0.028"
@@ -91,8 +91,8 @@
       <origin xyz="0 0.064 -0.393" rpy="${M_PI/2} 0 0"/>
       <axis xyz="0 0 1"/>
-      <limit effort="30.0" lower="${joint_b_lower_limit}" upper="${joint_b_upper_limit}" velocity="${joint_b_velocity_limit}"/>
+      <limit effort="100.0" lower="${joint_b_lower_limit}" upper="${joint_b_upper_limit}" velocity="${joint_b_velocity_limit}"/>
     </xacro:link_v1>
     <xacro:link_v1 name="link_t"
-                   mass="9.260846"
+                   mass="0.705"
                    parent_link_name="link_b" child_link_name="link_t" joint_name="joint_t">
       <inertia ixx="0.001" ixy="0.000" ixz="0.000"
@@ -101,12 +101,11 @@
       <origin xyz="0 -0.1 -0.098" rpy="${M_PI/2} 0 0"/>
       <axis xyz="0 0 1"/>
-      <limit effort="30.0" lower="${joint_t_lower_limit}" upper="${joint_t_upper_limit}" velocity="${joint_t_velocity_limit}"/>
+      <limit effort="100.0" lower="${joint_t_lower_limit}" upper="${joint_t_upper_limit}" velocity="${joint_t_velocity_limit}"/>
     </xacro:link_v1>
-  <!--   <joint name="joint_tool0" type="fixed">
+    <!--joint name="joint_tool0" type="fixed">
       <origin rpy="0 0 0" xyz="0 0 0"/>
-      <parent link="link_6"/>
+      <parent link="link_t"/>
       <child link="tool0"/>
-    </joint>
-   -->
+    </joint-->
     <!-- transmission -->
     <xacro:simple_jp_trans_v0 name="transmission_1"

Commit message: Modify joint names for hc10dt

File: motoman_description/robots/hc10dt/hc10dt_basic.urdf.xacro (robot description, xacro)
@@ -2,31 +2,31 @@
 <robot name="hc10dt" xmlns:xacro="http://ros.org/wiki/xacro">
   <!-- Include -->
-  <xacro:include filename="$(find motoman_description)/urdf/hc10dt/common.xacro" />
-  <xacro:include filename="$(find motoman_description)/urdf/hc10dt/materials.xacro" />
-  <xacro:include filename="$(find motoman_description)/urdf/hc10dt/hc10dt/body.urdf.xacro" />
-  <xacro:include filename="$(find motoman_description)/urdf/hc10dt/hc10dt/body.gazebo.xacro"/>
-  <xacro:include filename="$(find motoman_description)/urdf/hc10dt/hc10dt/body.transmission.xacro"/>
+  <xacro:include filename="$(find motoman_description)/urdf/common.xacro" />
+  <xacro:include filename="$(find motoman_description)/urdf/materials.xacro" />
+  <xacro:include filename="$(find motoman_description)/urdf/hc10dt/body.urdf.xacro" />
+  <xacro:include filename="$(find motoman_description)/urdf/hc10dt/body.gazebo.xacro"/>
+  <xacro:include filename="$(find motoman_description)/urdf/hc10dt/body.transmission.xacro"/>
   <!-- Configuration -->
   <xacro:macro name="motoman_hc10dt" params="prefix">
     <!-- Radius Limits -->
-    <xacro:property name="joint_s_upper_limit" value="${180*M_PI/180.0}"/>
-    <xacro:property name="joint_s_lower_limit" value="-${joint_s_upper_limit}"/>
-    <xacro:property name="joint_l_upper_limit" value="${180*M_PI/180.0}"/>
-    <xacro:property name="joint_l_lower_limit" value="-${joint_l_upper_limit}"/>
-    <xacro:property name="joint_u_upper_limit" value="${355*M_PI/180.0}"/>
-    <xacro:property name="joint_u_lower_limit" value="${-5*M_PI/180.0}"/>
-    <xacro:property name="joint_r_upper_limit" value="${180*M_PI/180.0}"/>
-    <xacro:property name="joint_r_lower_limit" value="-${joint_r_upper_limit}"/>
-    <xacro:property name="joint_b_upper_limit" value="${180*M_PI/180.0}"/>
-    <xacro:property name="joint_b_lower_limit" value="-${joint_b_upper_limit}"/>
-    <xacro:property name="joint_t_upper_limit" value="${180*M_PI/180.0}"/>
-    <xacro:property name="joint_t_lower_limit" value="-${joint_t_upper_limit}"/>
+    <xacro:property name="joint_1_s_upper_limit" value="${180*M_PI/180.0}"/>
+    <xacro:property name="joint_1_s_lower_limit" value="-${joint_1_s_upper_limit}"/>
+    <xacro:property name="joint_2_l_upper_limit" value="${180*M_PI/180.0}"/>
+    <xacro:property name="joint_2_l_lower_limit" value="-${joint_2_l_upper_limit}"/>
+    <xacro:property name="joint_3_u_upper_limit" value="${355*M_PI/180.0}"/>
+    <xacro:property name="joint_3_u_lower_limit" value="${-5*M_PI/180.0}"/>
+    <xacro:property name="joint_4_r_upper_limit" value="${180*M_PI/180.0}"/>
+    <xacro:property name="joint_4_r_lower_limit" value="-${joint_4_r_upper_limit}"/>
+    <xacro:property name="joint_5_b_upper_limit" value="${180*M_PI/180.0}"/>
+    <xacro:property name="joint_5_b_lower_limit" value="-${joint_5_b_upper_limit}"/>
+    <xacro:property name="joint_6_t_upper_limit" value="${180*M_PI/180.0}"/>
+    <xacro:property name="joint_6_t_lower_limit" value="-${joint_6_t_upper_limit}"/>
     <!-- Velocity Limits -->
-    <xacro:property name="joint_s_velocity_limit" value="${130.0*M_PI/180.0}"/>
-    <xacro:property name="joint_l_velocity_limit" value="${130.0*M_PI/180.0}"/>
-    <xacro:property name="joint_u_velocity_limit" value="${180.0*M_PI/180.0}"/>
-    <xacro:property name="joint_r_velocity_limit" value="${180.0*M_PI/180.0}"/>
-    <xacro:property name="joint_b_velocity_limit" value="${250.0*M_PI/180.0}"/>
-    <xacro:property name="joint_t_velocity_limit" value="${250.0*M_PI/180.0}"/>
+    <xacro:property name="joint_1_s_velocity_limit" value="${130.0*M_PI/180.0}"/>
+    <xacro:property name="joint_2_l_velocity_limit" value="${130.0*M_PI/180.0}"/>
+    <xacro:property name="joint_3_u_velocity_limit" value="${180.0*M_PI/180.0}"/>
+    <xacro:property name="joint_4_r_velocity_limit" value="${180.0*M_PI/180.0}"/>
+    <xacro:property name="joint_5_b_velocity_limit" value="${250.0*M_PI/180.0}"/>
+    <xacro:property name="joint_6_t_velocity_limit" value="${250.0*M_PI/180.0}"/>
     <!-- Add macro -->
     <xacro:macro name="add_world" params="*origin">
@@ -43,7 +43,7 @@
                izz="0.052"/>
     </xacro:base_link_v1>
-    <xacro:link_v1 name="link_s"
+    <xacro:link_v1 name="link_1_s"
                    mass="8.913"
-                   parent_link_name="base_link" child_link_name="link_s" joint_name="joint_s">
+                   parent_link_name="base_link" child_link_name="link_1_s" joint_name="joint_1_s">
       <inertia ixx="0.132" ixy="-0.001" ixz="0.001"
                iyy="0.128" iyz="0.012"
@@ -51,9 +51,9 @@
       <origin xyz="0 0 0.167" rpy="0 0 0"/>
       <axis xyz="0 0 1"/>
-      <limit effort="100.0" lower="${joint_s_lower_limit}" upper="${joint_s_upper_limit}" velocity="${joint_s_velocity_limit}"/>
+      <limit effort="100.0" lower="${joint_1_s_lower_limit}" upper="${joint_1_s_upper_limit}" velocity="${joint_1_s_velocity_limit}"/>
     </xacro:link_v1>
-    <xacro:link_v1 name="link_l"
+    <xacro:link_v1 name="link_2_l"
                    mass="14.232"
-                   parent_link_name="link_s" child_link_name="link_l" joint_name="joint_l">
+                   parent_link_name="link_1_s" child_link_name="link_2_l" joint_name="joint_2_l">
       <inertia ixx="2.518" ixy="0.000" ixz="0.000"
                iyy="0.130" iyz="-0.328"
@@ -61,9 +61,9 @@
       <origin xyz="0 -0.107 0.108" rpy="${M_PI/2} 0 0"/>
       <axis xyz="0 0 1"/>
-      <limit effort="100.0" lower="${joint_l_lower_limit}" upper="${joint_l_upper_limit}" velocity="${joint_l_velocity_limit}"/>
+      <limit effort="100.0" lower="${joint_2_l_lower_limit}" upper="${joint_2_l_upper_limit}" velocity="${joint_2_l_velocity_limit}"/>
     </xacro:link_v1>
-    <xacro:link_v1 name="link_u"
+    <xacro:link_v1 name="link_3_u"
                    mass="5.964"
-                   parent_link_name="link_l" child_link_name="link_u" joint_name="joint_u">
+                   parent_link_name="link_2_l" child_link_name="link_3_u" joint_name="joint_3_u">
       <inertia ixx="0.070" ixy="0.001" ixz="-0.004"
                iyy="0.068" iyz="-0.007"
@@ -71,9 +71,9 @@
       <origin xyz="0 0.7 -0.01" rpy="0 0 0"/>
       <axis xyz="0 0 1"/>
-      <limit effort="100.0" lower="${joint_u_lower_limit}" upper="${joint_u_upper_limit}" velocity="${joint_u_velocity_limit}"/>
+      <limit effort="100.0" lower="${joint_3_u_lower_limit}" upper="${joint_3_u_upper_limit}" velocity="${joint_3_u_velocity_limit}"/>
     </xacro:link_v1>
-    <xacro:link_v1 name="link_r"
+    <xacro:link_v1 name="link_4_r"
                    mass="4.849"
-                   parent_link_name="link_u" child_link_name="link_r" joint_name="joint_r">
+                   parent_link_name="link_3_u" child_link_name="link_4_r" joint_name="joint_4_r">
       <inertia ixx="0.347" ixy="0.000" ixz="0.000"
                iyy="0.347" iyz="0.002"
@@ -81,9 +81,9 @@
       <origin xyz="0 -0.106 -0.097" rpy="-${M_PI/2} 0 0"/>
       <axis xyz="0 0 1"/>
-      <limit effort="100.0" lower="${joint_r_lower_limit}" upper="${joint_r_upper_limit}" velocity="${joint_r_velocity_limit}"/>
+      <limit effort="100.0" lower="${joint_4_r_lower_limit}" upper="${joint_4_r_upper_limit}" velocity="${joint_4_r_velocity_limit}"/>
     </xacro:link_v1>
-      <xacro:link_v1 name="link_b"
+      <xacro:link_v1 name="link_5_b"
                    mass="5.454"
-                   parent_link_name="link_r" child_link_name="link_b" joint_name="joint_b">
+                   parent_link_name="link_4_r" child_link_name="link_5_b" joint_name="joint_5_b">
       <inertia ixx="0.074" ixy="0.060" ixz="0.028"
                iyy="0.000" iyz="0.013"
@@ -91,9 +91,9 @@
       <origin xyz="0 0.064 -0.393" rpy="${M_PI/2} 0 0"/>
       <axis xyz="0 0 1"/>
-      <limit effort="100.0" lower="${joint_b_lower_limit}" upper="${joint_b_upper_limit}" velocity="${joint_b_velocity_limit}"/>
+      <limit effort="100.0" lower="${joint_5_b_lower_limit}" upper="${joint_5_b_upper_limit}" velocity="${joint_5_b_velocity_limit}"/>
     </xacro:link_v1>
-    <xacro:link_v1 name="link_t"
+    <xacro:link_v1 name="link_6_t"
                    mass="0.705"
-                   parent_link_name="link_b" child_link_name="link_t" joint_name="joint_t">
+                   parent_link_name="link_5_b" child_link_name="link_6_t" joint_name="joint_6_t">
       <inertia ixx="0.001" ixy="0.000" ixz="0.000"
                iyy="0.001" iyz="0.000"
@@ -101,5 +101,5 @@
       <origin xyz="0 -0.1 -0.098" rpy="${M_PI/2} 0 0"/>
       <axis xyz="0 0 1"/>
-      <limit effort="100.0" lower="${joint_t_lower_limit}" upper="${joint_t_upper_limit}" velocity="${joint_t_velocity_limit}"/>
+      <limit effort="100.0" lower="${joint_6_t_lower_limit}" upper="${joint_6_t_upper_limit}" velocity="${joint_6_t_velocity_limit}"/>
     </xacro:link_v1>
     <!--joint name="joint_tool0" type="fixed">
@@ -109,36 +109,37 @@
     </joint-->
     <!-- transmission -->
-    <xacro:simple_jp_trans_v0 name="transmission_1"
-                              joint_name="joint_s" actuator_name="motor_1"
+    <xacro:simple_jp_trans_v0 name="transmission_1_s"
+                              joint_name="joint_1_s" actuator_name="motor_1_s"
                               reduction="1"/>
-    <xacro:simple_jp_trans_v0 name="transmission_2"
-                              joint_name="joint_l" actuator_name="motor_2"
+    <xacro:simple_jp_trans_v0 name="transmission_2_l"
+                              joint_name="joint_2_l" actuator_name="motor_2_l"
                               reduction="1"/>
-    <xacro:simple_jp_trans_v0 name="transmission_3"
-                              joint_name="joint_u" actuator_name="motor_3"
+    <xacro:simple_jp_trans_v0 name="transmission_3_u"
+                              joint_name="joint_3_u" actuator_name="motor_3_u"
                               reduction="1"/>
-    <xacro:simple_jp_trans_v0 name="transmission_4"
-                              joint_name="joint_r" actuator_name="motor_4"
+    <xacro:simple_jp_trans_v0 name="transmission_4_r"
+                              joint_name="joint_4_r" actuator_name="motor_4_r"
                               reduction="1"/>
-    <xacro:simple_jp_trans_v0 name="transmission_5"
-                              joint_name="joint_b" actuator_name="motor_5"
+    <xacro:simple_jp_trans_v0 name="transmission_5_b"
+                              joint_name="joint_5_b" actuator_name="motor_5_b"
                               reduction="1"/>
-    <xacro:simple_jp_trans_v0 name="transmission_6"
-                              joint_name="joint_t" actuator_name="motor_6"
+    <xacro:simple_jp_trans_v0 name="transmission_6_t"
+                              joint_name="joint_6_t" actuator_name="motor_6_t"
                               reduction="1"/>
     <!-- gazebo -->
     <gazebo>
       <plugin name="gazebo_ros_control" filename="libgazebo_ros_control.so">
-        <robotNamespace>/hc10dt</robotNamespace>
+        <!--robotNamespace>/hc10dt</robotNamespace-->
         <robotSimType>gazebo_ros_control/DefaultRobotHWSim</robotSimType>
+        <legacyModeNS>true</legacyModeNS>
       </plugin>
     </gazebo>
     <xacro:gazebo_link_v1 name="base_link"/>
-    <xacro:gazebo_link_v1 name="link_s"/>
-    <xacro:gazebo_link_v1 name="link_l"/>
-    <xacro:gazebo_link_v1 name="link_u"/>
-    <xacro:gazebo_link_v1 name="link_b"/>
-    <xacro:gazebo_link_v1 name="link_r"/>
-    <xacro:gazebo_link_v1 name="link_t"/>
+    <xacro:gazebo_link_v1 name="link_1_s"/>
+    <xacro:gazebo_link_v1 name="link_2_l"/>
+    <xacro:gazebo_link_v1 name="link_3_u"/>
+    <xacro:gazebo_link_v1 name="link_4_b"/>
+    <xacro:gazebo_link_v1 name="link_5_r"/>
+    <xacro:gazebo_link_v1 name="link_6_t"/>
   </xacro:macro>
 </robot>
