Commit message: Update hc10dt.urdf

File: motoman_description/robots/hc10dt/hc10dt.urdf (robot description, URDF)
Before this commit: robot motoman_motomini, 8 links, 7 joints
Links:
- removed link link_b
- removed link link_l
- removed link link_r
- removed link link_s
- removed link link_t
- removed link link_u
- added link link_1_s, mass 8.913; collision mesh filename=package://motoman_description/meshes/hc10dt/collision/link_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; visual mesh filename=package://motoman_description/meshes/hc10dt/visual/link_1_s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
- added link link_2_l, mass 14.232; collision mesh filename=package://motoman_description/meshes/hc10dt/collision/link_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; visual mesh filename=package://motoman_description/meshes/hc10dt/visual/link_2_l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
- added link link_3_u, mass 5.964; collision mesh filename=package://motoman_description/meshes/hc10dt/collision/link_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; visual mesh filename=package://motoman_description/meshes/hc10dt/visual/link_3_u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
- added link link_4_r, mass 4.849; collision mesh filename=package://motoman_description/meshes/hc10dt/collision/link_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; visual mesh filename=package://motoman_description/meshes/hc10dt/visual/link_4_r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
- added link link_5_b, mass 5.454; collision mesh filename=package://motoman_description/meshes/hc10dt/collision/link_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; visual mesh filename=package://motoman_description/meshes/hc10dt/visual/link_5_b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
- added link link_6_t, mass 0.705; collision mesh filename=package://motoman_description/meshes/hc10dt/collision/link_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; visual mesh filename=package://motoman_description/meshes/hc10dt/visual/link_6_t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
Joints:
- removed joint joint_b
- removed joint joint_l
- removed joint joint_r
- removed joint joint_s
- removed joint joint_t
- removed joint joint_u
- added joint joint_1_s: type revolute, parent base_link, child link_1_s, origin xyz=0 0 0.167 rpy=0 0 0, axis 0 0 1, limit lower=-3.14159274 upper=3.14159274 effort=100.0 velocity=2.26892809
- added joint joint_2_l: type revolute, parent link_1_s, child link_2_l, origin xyz=0 -0.107 0.108 rpy=1.57079637 0 0, axis 0 0 1, limit lower=-3.14159274 upper=3.14159274 effort=100.0 velocity=2.26892809
- added joint joint_3_u: type revolute, parent link_2_l, child link_3_u, origin xyz=0 0.7 -0.01 rpy=0 0 0, axis 0 0 1, limit lower=-0.087266465 upper=6.195919015 effort=100.0 velocity=3.14159274
- added joint joint_4_r: type revolute, parent link_3_u, child link_4_r, origin xyz=0 -0.106 -0.097 rpy=-1.57079637 0 0, axis 0 0 1, limit lower=-3.14159274 upper=3.14159274 effort=100.0 velocity=3.14159274
- added joint joint_5_b: type revolute, parent link_4_r, child link_5_b, origin xyz=0 0.064 -0.393 rpy=1.57079637 0 0, axis 0 0 1, limit lower=-3.14159274 upper=3.14159274 effort=100.0 velocity=4.36332325
- added joint joint_6_t: type revolute, parent link_5_b, child link_6_t, origin xyz=0 -0.1 -0.098 rpy=1.57079637 0 0, axis 0 0 1, limit lower=-3.14159274 upper=3.14159274 effort=100.0 velocity=4.36332325
